File: hardware/slim4_r22_wip/board/SLIM4_R22.kicad_pcb (KiCad board)
At the start: 6 copper layers, 99.2 x 125 mm, 165 parts, among them J1 FH12-20S-0.5SH(55), J2 USB4105-GF-A-120, J3 SM03B-SRSS-TB(LF)(SN), J4 SM02B-SRSS-TB(LF)(SN), J5 SM02B-SRSS-TB(LF)(SN), Q1 2N7002, SW1 D2LS-21(20M), SW2 D2LS-21(20M), SW3 D2LS-11, SW4 D2LS-11, SW5 B3U-1000P, SW6 B3U-1000P, SW7 B3U-1000P, U1 ESP32-P4NRW32X, U10 BQ24074RGTR, U11 TPD2EUSB30DRTR, U12 TPD2EUSB30DRTR, U13 TUSB320LAIRWBR, U14 TPS3808G33DBVR, U2 W25Q512JVEIQ TR, U3 TLV62569DBVR, U4 TPS63070RNMR, U5 TLV75518PDBVR, U6 TLV75528PDBVR, U7 TPS61165DBVR, U8 MAX98357AETE+T, U9 MAX98357AETE+T, Y1 L327S400H11L

Commit message: PCB R22: display chosen, backlight fixed, JLCPCB order pack
- Display: Startek KD047HDFID001, 4.7 in 720x1280 IPS (ST7703, 450 nits).
  Its active area matches the case's screen opening, so the front
  controls stay where they are. J1 becomes a fixed display port; a small
  adapter maps it to the panel's 31-pin cable, so a pinout mistake can
  only land on the adapter (DISPLAY_PORT.md)
- Backlight: R309 5.1 ohm (39 mA for the panel's two 7-LED strings);
  C309 1 uF 50 V (the boost's open-LED limit is 38 V; it was 25 V)
- Panel VCI 3.0 V: U6 TLV75530; net LCD_2V8 renamed LCD_VCI_3V0
- scripts/build_r22_order_pack.py and ORDER/STRUTHIO_SLIM4_R22_PCB_ORDER.zip:
  Gerbers + drill, BOM (LCSC for all 165 parts), CPL, order options;
  KiCad 7.0.11 DRC 0/0/0, zone fills current, no mask openings at vias
- FIRMWARE_PINMAP.md: every GPIO, its default state and how to drive it

Co-Authored-By: Claude Opus 5.5 <noreply@anthropic.com>
Claude-Session: https://claude.ai/code/session_01AZXyynf2vqoA1qdTyQFbXM
Parts:
- C309: value CS1608X7R105K250NRB -> CL10A105KB8NNNC
- R309: value 0603WAF249KT5E -> 0603WAF510KT5E
- U6: value TLV75528PDBVR -> TLV75530PDBVR
Connections:
- net LCD_2V8 renamed LCD_VCI_3V0

Commit message: PCB R22: battery port takes any 2-wire cell; display flex documented
- J3: JST SH 3-pin -> 2-pin, the same part as the speaker sockets
  (pin 1 BAT+, pin 2 GND), so one cable type serves battery and speakers
- R424 10k from the BQ24074 TS pin to GND (the datasheet's no-thermistor
  connection); the NTC route is cut back to it, net BAT_NTC -> BQ_TS.
  Cell protection stays on the cell's PCM
- DISPLAY_PORT.md: the custom flex (31-pin ZIF on the panel end, 20 x
  0.5 mm gold fingers with stiffener to 0.30 mm at J1)
- Order pack regenerated: 166 parts, 51 BOM lines, LCSC for all; KiCad
  DRC 0/0/0; README states the battery polarity (no reverse protection)

Co-Authored-By: Claude Opus 5.5 <noreply@anthropic.com>
Claude-Session: https://claude.ai/code/session_01AZXyynf2vqoA1qdTyQFbXM
Parts:
- added R424: 0402WGF1002TCE, SLIM4:FP_R424, B.Cu at (-22.5, 59.0)
- J3: value SM03B-SRSS-TB(LF)(SN) -> SM02B-SRSS-TB(LF)(SN)
- moved J3 0.50 mm to (-23.5, 66.0)
Connections:
- J3 pad 2: BAT_NTC -> GND
- U10 pad 1: BAT_NTC -> BQ_TS
Routing:
- net BAT_NTC: track 92.3 -> 0.00 mm, vias 2 -> 0
- net BQ_TS: track 0.00 -> 88.3 mm, vias 0 -> 2
- net GND: track 653.6 -> 655.4 mm, vias 23 -> 24

Commit message: PCB R22: JLCPCB stock substitutions; U1 sourcing note
Stock checked against JLCPCB's parts search on 2026-10-07. Same package
and value for each:
- 10 uF 0805 -> CL21A106KAYNNNE (C15850); 22 uF 0805 -> CL21A226MQQNNNE
  (C5674); 4.7 uF 0603 -> CL10A475KO8NNNC (C19666); 499k -> C25793;
  4.02k -> C43251
- U6 -> ME6211C30M5G-N (C403651): SOT-23-5 IN/GND/EN/NC/OUT like TLV755
- SW1-SW4 -> Omron D2LS-21 (C3823622): D2LS-11 positions and land
  pattern, 0.6 N like the flap switches
- ESP32-P4NRW32X has no stock anywhere checked: README and order README
  give the pre-order / consign route and warn against the v1.x part

KiCad DRC 0/0/0; 50 BOM lines, LCSC for all 166 parts.

Co-Authored-By: Claude Opus 5.5 <noreply@anthropic.com>
Claude-Session: https://claude.ai/code/session_01AZXyynf2vqoA1qdTyQFbXM
Parts:
- C112, C311, C409, C410: value 0603X5R475K100NT -> CL10A475KO8NNNC
- C123, C126, C133, C411, C412: value C0805C106K8PAC7800 -> CL21A106KAYNNNE
- C135, C413, C414, C415: value C0805X5R6R3-226MNE -> CL21A226MQQNNNE
- R103: value RMCF0402FT4K02 -> 0402WGF4021TCE
- R104, R105: value RM04FTN4993 -> 0402WGF4993TCE
- SW1, SW2: value D2LS-21(20M) -> D2LS-21
- SW3, SW4: value D2LS-11 -> D2LS-21
- U6: value TLV75530PDBVR -> ME6211C30M5G-N
