File: hardware/arc1-compact/R08_WORK/cad/boot_nor.kicad_sch (KiCad schematic)
At the start: 19 parts, among them J2 LA SPI0, SW2 FEL (NOR reset), U16 W25Q256JVFIQ

Commit message: ARC-1 Compact R08: rule checker + negative tests, margin analysis, diagnostic boot0 image, runner, dossiers, ledger, risk register, status
Co-Authored-By: Claude Opus 5.5 <noreply@anthropic.com>
Claude-Session: https://claude.ai/code/session_01UkiuLdbjDvK75uDzAPKsGs
Parts:
- C61, C62, R32, R33, R34, R35, R36, R37, R38: Evidence VERIFIED_BY_VENDOR_DOC -> GENERIC_PASSIVE (value from design.py / analysis; MPN only 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
- J2, TP25, TP26, TP27, TP28, TP29, TP30, TP31: Evidence VERIFIED_BY_VENDOR_DOC -> GENERIC (no device-specific claim)
