File: hardware/arc1-compact/R08_WORK/cad/controls.kicad_sch (KiCad schematic)
At the start: 20 parts, among them J10 F133 UART0, SW10 Y, SW11 L, SW12 R, SW13 START, SW14 SELECT, SW15 HOME, SW3 UP, SW4 DOWN, SW5 LEFT, SW6 RIGHT, SW7 A, SW8 B, SW9 X

Commit message: ARC-1 Compact R08: rule checker + negative tests, margin analysis, diagnostic boot0 image, runner, dossiers, ledger, risk register, status
Co-Authored-By: Claude Opus 5.5 <noreply@anthropic.com>
Claude-Session: https://claude.ai/code/session_01UkiuLdbjDvK75uDzAPKsGs
Parts:
- D4, D5, D6: Evidence CANDIDATE -> GENERIC (no device-specific claim)
- J10: Evidence VERIFIED_BY_VENDOR_DOC -> GENERIC (no device-specific claim)
- R94, R95, R96: Evidence VERIFIED_BY_VENDOR_DOC -> GENERIC_PASSIVE (value from design.py / analysis; MPN only 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
