File: hardware/arc1-compact/R08_WORK/cad/mn820.kicad_sch (KiCad schematic)
At the start: 24 parts, among them J3 DF40C-100DS-0.4V(51), J4 LA SPI1, U17 MISO buffer

Commit message: ARC-1 Compact R08: rule checker + negative tests, margin analysis, diagnostic boot0 image, runner, dossiers, ledger, risk register, status
Co-Authored-By: Claude Opus 5.5 <noreply@anthropic.com>
Claude-Session: https://claude.ai/code/session_01UkiuLdbjDvK75uDzAPKsGs
Parts:
- C63, C64, C65, C66, R39, R40, R41, R42, R43, R44, R45, R46, R47, R48, R49: Evidence VERIFIED_BY_VENDOR_DOC -> GENERIC_PASSIVE (value from design.py / analysis; MPN only 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
- J4, TP32, TP33, TP34, TP35: Evidence VERIFIED_BY_VENDOR_DOC -> GENERIC (no device-specific claim)
