File: hardware/arc1-compact/R08_WORK/cad/power.kicad_sch (KiCad schematic)
At the start: 94 parts, among them SW1 RESET, U10 3V3_T35 switch, U11 3V3_MN switch, U12 PSRAM_VDD switch, U13 AND, U14 TPS3808G30, U3 3V3 2A, U4 TPS3808G33, U5 VDD_CORE 0.95V, U6 1V8_DRAM, U7 1V8_AN, U8 TPS3808G09, U9 1V2_T35

Commit message: ARC-1 Compact R08: rule checker + negative tests, margin analysis, diagnostic boot0 image, runner, dossiers, ledger, risk register, status
Co-Authored-By: Claude Opus 5.5 <noreply@anthropic.com>
Claude-Session: https://claude.ai/code/session_01UkiuLdbjDvK75uDzAPKsGs
Parts:
- C10, C11, C12, C13, C14, C15, C16, C17, C18, C19, C20, C21, C22, C23, C24, C25, C26, C27, C28, C29, C30, C31, C4, C5, C6, C7, C8, C9, L1, L2, L3, L4, R10, R11, R12, R13, R14, R15, R16, R17, R18, R19, R20, R21, R22, R23, R24, R25, R26, R27, R28, R29, R30, R8, R9: Evidence VERIFIED_BY_VENDOR_DOC -> GENERIC_PASSIVE (value from design.py / analysis; MPN only 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
- FID1, FID2, FID3, H1, H2, H3, H4, TP10, TP11, TP12, TP13, TP14, TP15, TP16, TP17, TP18, TP19, TP20, TP21, TP22, TP4, TP5, TP6, TP7, TP8, TP9: Evidence VERIFIED_BY_VENDOR_DOC -> GENERIC (no device-specific claim)
