File: hardware/arc1-compact/R08_WORK/cad/psram.kicad_sch (KiCad schematic)
At the start: 18 parts, among them U25 APS6404L-3SQR, U26 SN74LVC07A

Commit message: ARC-1 Compact R08: rule checker + negative tests, margin analysis, diagnostic boot0 image, runner, dossiers, ledger, risk register, status
Co-Authored-By: Claude Opus 5.5 <noreply@anthropic.com>
Claude-Session: https://claude.ai/code/session_01UkiuLdbjDvK75uDzAPKsGs
Parts:
- C106, C107, C108, R71, R72, R73, R74, R75, R76, R77, R78, R79, R80, R81, R82, R83: Evidence VERIFIED_BY_VENDOR_DOC -> GENERIC_PASSIVE (value from design.py / analysis; MPN only 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
