File: hardware/arc1-compact/R08_WORK/cad/sd_audio.kicad_sch (KiCad schematic)
At the start: 25 parts, among them J7 microSD, J8 SPK L, J9 SPK R, U27 SD power switch, U28 MAX98357A L, U29 MAX98357A R

Commit message: ARC-1 Compact R08: rule checker + negative tests, margin analysis, diagnostic boot0 image, runner, dossiers, ledger, risk register, status
Co-Authored-By: Claude Opus 5.5 <noreply@anthropic.com>
Claude-Session: https://claude.ai/code/session_01UkiuLdbjDvK75uDzAPKsGs
Parts:
- C109, C110, C111, C112, C113, C114, C115, R84, R85, R86, R87, R88, R89, R90, R91, R92, R93: Evidence VERIFIED_BY_VENDOR_DOC -> GENERIC_PASSIVE (value from design.py / analysis; MPN only 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
- TP40, TP41: Evidence VERIFIED_BY_VENDOR_DOC -> GENERIC (no device-specific claim)
