File: hardware/arc1-compact/R08_WORK/cad/t35.kicad_sch (KiCad schematic)
At the start: 77 parts, among them J5 T35 JTAG, J6 T35 UART, U18 T35F400C3, U19 W25Q32JVSSIQ, U20 Schmitt, U21 iso SCK, U22 iso MOSI, U23 iso SS, U24 iso MISO, X1 25MHz

Commit message: ARC-1 Compact R08: rule checker + negative tests, margin analysis, diagnostic boot0 image, runner, dossiers, ledger, risk register, status
Co-Authored-By: Claude Opus 5.5 <noreply@anthropic.com>
Claude-Session: https://claude.ai/code/session_01UkiuLdbjDvK75uDzAPKsGs
Parts:
- C100, C101, C102, C103, C104, C105, C67, C68, C69, C70, C71, C72, C73, C74, C75, C76, C77, C78, C79, C80, C81, C82, C83, C84, C85, C86, C87, C88, C89, C90, C91, C92, C93, C94, C95, C96, C97, C98, C99, FB1, R50, R51, R52, R53, R54, R55, R56, R57, R58, R59, R60, R61, R62, R63, R64, R65, R66, R67, R68, R69, R70: Evidence VERIFIED_BY_VENDOR_DOC -> GENERIC_PASSIVE (value from design.py / analysis; MPN only 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
- D2, D3: Evidence CANDIDATE -> GENERIC (no device-specific claim)
- J5, J6, TP36, TP37, TP38, TP39: Evidence VERIFIED_BY_VENDOR_DOC -> GENERIC (no device-specific claim)
