File: hardware/arc1-compact/R85_WORK/cad/boot_nor.kicad_sch (KiCad schematic)
At the start: 19 parts, among them J2 LA SPI0, SW2 FEL (NOR reset), U16 W25Q256JVFIQ

Commit message: ARC-1 Compact R8.5: ECP5 board sheet (power tree, sysCONFIG SSPI, JTAG), regenerated KiCad (ERC 0), R8.5 rule checker, pin matrices + generated LPF, routed reproducible bitstream
Co-Authored-By: Claude Opus 5.5 <noreply@anthropic.com>
Claude-Session: https://claude.ai/code/session_01UkiuLdbjDvK75uDzAPKsGs
Parts:
- removed C61: 100nF, Capacitor_SMD:C_0402_1005Metric, symbol ARC1_R08:C0402
- removed C62: 1uF, Capacitor_SMD:C_0402_1005Metric, symbol ARC1_R08:C0402
- removed R32: 22R, Resistor_SMD:R_0402_1005Metric, symbol ARC1_R08:R0402
- removed TP25: SPI0_CLK, TestPoint:TestPoint_Pad_D1.0mm, symbol ARC1_R08:TP
- removed TP26: SPI0_MOSI, TestPoint:TestPoint_Pad_D1.0mm, symbol ARC1_R08:TP
- added C63: 100nF, Capacitor_SMD:C_0402_1005Metric, symbol ARC1_R85:C0402
- added C64: 1uF, Capacitor_SMD:C_0402_1005Metric, symbol ARC1_R85:C0402
- added R39: 10k, Resistor_SMD:R_0402_1005Metric, symbol ARC1_R85:R0402
- added TP32: SPI0_IO2, TestPoint:TestPoint_Pad_D1.0mm, symbol ARC1_R85:TP
- added TP33: SPI0_IO3, TestPoint:TestPoint_Pad_D1.0mm, symbol ARC1_R85:TP
- J2: symbol ARC1_R08:HDR_2x5_127 -> ARC1_R85:HDR_2x5_127
- R33: value 3.3k -> 22R; symbol ARC1_R08:R0402 -> ARC1_R85:R0402; LCSC C25890 -> (none); MPN 0402WGF3301TCE -> (none); Manufacturer UNI-ROYAL -> (none); Note BOOT-SEL0 = 0 vs internal PU 12k min: 0.217*VCC < 0.3*VCC -> source series termination at F133; Reuse SLIM4_R26_BOM_LINE (re-validate) -> (none)
- R34: symbol ARC1_R08:R0402 -> ARC1_R85:R0402; Note BOOT-SEL1 = 0; NOR DO hi-Z (CS# high) and T35 buffer hi-Z a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 -> BOOT-SEL0 = 0 vs internal PU 12k min: 0.217*VCC < 0.3*VCC
- R35: value 10k -> 3.3k; symbol ARC1_R08:R0402 -> ARC1_R85:R0402; LCSC C25744 -> C25890; MPN 0402WGF1002TCE -> 0402WGF3301TCE; Note NOR deselected while F133 in reset -> BOOT-SEL1 = 0; NOR DO hi-Z (CS# high) and FPGA MISO buffer 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
- R36: symbol ARC1_R08:R0402 -> ARC1_R85:R0402; Note QE=1 (IQ): IO2 must not float; xfel drives only PC2-PC5 -> NOR deselected while F133 in reset
- R37: symbol ARC1_R08:R0402 -> ARC1_R85:R0402; Note (none) -> QE=1 (IQ): IO2 must not float; xfel drives only PC2-PC5
- R38: symbol ARC1_R08:R0402 -> ARC1_R85:R0402
- SW2: symbol ARC1_R08:SW_B3U -> ARC1_R85:SW_B3U
- TP27: value SPI0_MISO -> SPI0_CLK; symbol ARC1_R08:TP -> ARC1_R85:TP
- TP28: value SPI0_CS0_N -> SPI0_MOSI; symbol ARC1_R08:TP -> ARC1_R85:TP
- TP29: value NOR_RESET_N -> SPI0_MISO; symbol ARC1_R08:TP -> ARC1_R85:TP
- TP30: value SPI0_IO2 -> SPI0_CS0_N; symbol ARC1_R08:TP -> ARC1_R85:TP
- TP31: value SPI0_IO3 -> NOR_RESET_N; symbol ARC1_R08:TP -> ARC1_R85:TP
- U16: symbol ARC1_R08:W25Q256JVFIQ -> ARC1_R85:W25Q256JVFIQ
Connections:
- net 3V3: now also C63.1, C64.1, R39.2; no longer R35.2
- net GND: now also R35.2, C63.2, C64.2; no longer R33.2
- net NOR_RESET_N: now also TP31.1, R39.1; no longer R38.1, TP29.1
- net SPI0_CLK: now also R33.2, TP27.1
- net SPI0_CLK_F: now also R33.1
- net SPI0_CS0_N: now also R36.1, TP30.1; no longer R35.1, TP28.1
- net SPI0_IO2: now also R37.1, TP32.1; no longer R36.1, TP30.1
- net SPI0_IO3: now also R38.1, TP33.1; no longer R37.1, TP31.1
- net SPI0_MISO: now also R35.1, TP29.1; no longer R34.1, TP27.1
- net SPI0_MOSI: now also R34.1, TP28.1; no longer R33.1
- net T35_SS_N_F renamed FPGA_SS_N_F
Other:
- title: ARC-1 Compact R08: 32 MiB SPI NOR boot (BOOT-SEL 00), straps, FEL/clip recovery -> ARC-1 Compact R8.5: 32 MiB SPI NOR boot (BOOT-SEL 00), straps, FEL/clip recovery
- moved on the sheet: R33, R34, R35, R36, R37, R38, TP27, TP28, TP29, TP30, TP31
