File: hardware/arc1-compact/R85_WORK/cad/f133.kicad_sch (KiCad schematic)
At the start: 34 parts, among them U15 F133-B, Y1 24MHz

Commit message: ARC-1 Compact R8.5: ECP5 board sheet (power tree, sysCONFIG SSPI, JTAG), regenerated KiCad (ERC 0), R8.5 rule checker, pin matrices + generated LPF, routed reproducible bitstream
Co-Authored-By: Claude Opus 5.5 <noreply@anthropic.com>
Claude-Session: https://claude.ai/code/session_01UkiuLdbjDvK75uDzAPKsGs
Parts:
- removed C32, C33: 100nF, Capacitor_SMD:C_0402_1005Metric, symbol ARC1_R08:C0402
- removed R31: 240R, Resistor_SMD:R_0402_1005Metric, symbol ARC1_R08:R0402
- removed TP23: UART0_TX, TestPoint:TestPoint_Pad_D1.0mm, symbol ARC1_R08:TP
- removed TP24: UART0_RX, TestPoint:TestPoint_Pad_D1.0mm, symbol ARC1_R08:TP
- added C61, C62: 12pF, Capacitor_SMD:C_0402_1005Metric, symbol ARC1_R85:C0402
- added R32: 240R, Resistor_SMD:R_0402_1005Metric, symbol ARC1_R85:R0402
- added TP25: UART0_TX, TestPoint:TestPoint_Pad_D1.0mm, symbol ARC1_R85:TP
- added TP26: UART0_RX, TestPoint:TestPoint_Pad_D1.0mm, symbol ARC1_R85:TP
- C34, C35, C36, C37, C38, C39, C40, C41, C42, C43, C44, C45, C46, C47, C48, C49, C50, C51: symbol ARC1_R08:C0402 -> ARC1_R85:C0402
- C52, C53: value 10uF -> 100nF; footprint Capacitor_SMD:C_0603_1608Metric -> Capacitor_SMD:C_0402_1005Metric; symbol ARC1_R08:C0603 -> ARC1_R85:C0402; LCSC C19702 -> C1525; MPN CL10A106KP8NNNC -> CL05B104KO5NNNC
- C54, C55: value 4.7uF -> 10uF; symbol ARC1_R08:C0603 -> ARC1_R85:C0603; LCSC C19666 -> C19702; MPN CL10A475KO8NNNC -> CL10A106KP8NNNC
- C56: value 2.2uF -> 4.7uF; symbol ARC1_R08:C0603 -> ARC1_R85:C0603; LCSC (none) -> C19666; MPN (none) -> CL10A475KO8NNNC; Manufacturer (none) -> Samsung; Note LDOB-OUT unused (DRAM from buck), cap per MangoPi MQ -> (none); Reuse (none) -> SLIM4_R26_BOM_LINE (re-validate)
- C57: value 1uF -> 4.7uF; footprint Capacitor_SMD:C_0402_1005Metric -> Capacitor_SMD:C_0603_1608Metric; symbol ARC1_R08:C0402 -> ARC1_R85:C0603; LCSC C52923 -> C19666; MPN CL05A105KA5NQNC -> CL10A475KO8NNNC; Note value per reference design -- OPEN (no Allwinner reference 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 -> (none)
- C58: value 1uF -> 2.2uF; footprint Capacitor_SMD:C_0402_1005Metric -> Capacitor_SMD:C_0603_1608Metric; symbol ARC1_R08:C0402 -> ARC1_R85:C0603; LCSC C52923 -> (none); MPN CL05A105KA5NQNC -> (none); Manufacturer Samsung -> (none); Note value per reference design -- OPEN -> LDOB-OUT unused (DRAM from buck), cap per MangoPi MQ; Reuse SLIM4_R26_BOM_LINE (re-validate) -> (none)
- C59: value 12pF -> 1uF; symbol ARC1_R08:C0402 -> ARC1_R85:C0402; LCSC C1547 -> C52923; MPN 0402CG120J500NT -> CL05A105KA5NQNC; Manufacturer FH -> Samsung; Note CL match to crystal choice -- R09 -> value per reference design -- OPEN (no Allwinner reference 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
- C60: value 12pF -> 1uF; symbol ARC1_R08:C0402 -> ARC1_R85:C0402; LCSC C1547 -> C52923; MPN 0402CG120J500NT -> CL05A105KA5NQNC; Manufacturer FH -> Samsung; Note (none) -> value per reference design -- OPEN
- U15: footprint ARC1_R08:Allwinner_F133_eLQFP128_14x14_P0.4_EP5.72 -> ARC1_R85:Allwinner_F133_eLQFP128_14x14_P0.4_EP5.72; symbol ARC1_R08:F133 -> ARC1_R85:F133
- Y1: symbol ARC1_R08:XTAL_3225 -> ARC1_R85:XTAL_3225
Connections:
- net 1V8_AN: now also C52.1, C53.1; no longer C49.1, C50.1
- net 1V8_DRAM: now also C45.1, C46.1, C56.1; no longer C43.1, C44.1, C54.1
- net 1V8_LDOA: now also C49.1, C50.1, C57.1; no longer C45.1, C46.1, C55.1
- net 3V3: now also C43.1, C44.1, C55.1; no longer C37.1, C38.1, C53.1
- net F133_LDOB: now also C58.1; no longer C56.1
- net F133_PIN47_DZQ: now also R32.1
- net F133_VRA1: now also C59.1; no longer C57.1
- net F133_VRA2: now also C60.1; no longer C58.1
- net GND: now also C61.2, C62.2, R32.2
- net UART0_RX: now also TP26.1
- net UART0_TX: now also TP25.1
- net VDD_CORE: now also C37.1, C38.1, C54.1; no longer C52.1
- net XTAL24_IN: now also C61.1; no longer C59.1
- net XTAL24_OUT: now also C62.1; no longer C60.1
- net FPGA_INITN: now reaches U15.55 (PD0)
- net FPGA_VCC_PG: now reaches U15.56 (PD1)
- net T35_BUS_EN_N renamed FPGA_BUS_EN_N
- net T35_CDONE renamed FPGA_DONE
- net T35_CRESET_N_F renamed FPGA_PROGRAMN_F
- net T35_IRQ_N renamed FPGA_IRQ_N
- net T35_PWR_EN renamed FPGA_PWR_EN_F
- net T35_SS_N_F renamed FPGA_SS_N_F
- no-connect marks 44 -> 42
Other:
- title: ARC-1 Compact R08: F133-B SoC: supplies, clock, reset, pin assignment -> ARC-1 Compact R8.5: F133-B SoC: supplies, clock, reset, pin assignment
- moved on the sheet: C34, C35, C36, C37, C38, C39, C40, C41, C42, C43, C44, C45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
