File: hardware/arc1-compact/R85_WORK/cad/mn820.kicad_sch (KiCad schematic)
At the start: 24 parts, among them J3 DF40C-100DS-0.4V(51), J4 LA SPI1, U17 MISO buffer

Commit message: ARC-1 Compact R8.5: ECP5 board sheet (power tree, sysCONFIG SSPI, JTAG), regenerated KiCad (ERC 0), R8.5 rule checker, pin matrices + generated LPF, routed reproducible bitstream
Co-Authored-By: Claude Opus 5.5 <noreply@anthropic.com>
Claude-Session: https://claude.ai/code/session_01UkiuLdbjDvK75uDzAPKsGs
Parts:
- removed C63, C64: 100nF, Capacitor_SMD:C_0402_1005Metric, symbol ARC1_R08:C0402
- removed R39: 33R, Resistor_SMD:R_0402_1005Metric, symbol ARC1_R08:R0402
- removed TP32: BT_SCK, TestPoint:TestPoint_Pad_D1.0mm, symbol ARC1_R08:TP
- removed TP33: BT_MISO, TestPoint:TestPoint_Pad_D1.0mm, symbol ARC1_R08:TP
- added C67: 100nF, Capacitor_SMD:C_0402_1005Metric, symbol ARC1_R85:C0402
- added C68: 10uF, Capacitor_SMD:C_0603_1608Metric, symbol ARC1_R85:C0603
- added R50: 47k, Resistor_SMD:R_0402_1005Metric, symbol ARC1_R85:R0402
- added TP36: BT_INT_N, TestPoint:TestPoint_Pad_D1.0mm, symbol ARC1_R85:TP
- added TP37: BT_RST_N, TestPoint:TestPoint_Pad_D1.0mm, symbol ARC1_R85:TP
- C65: symbol ARC1_R08:C0402 -> ARC1_R85:C0402
- C66: value 10uF -> 100nF; footprint Capacitor_SMD:C_0603_1608Metric -> Capacitor_SMD:C_0402_1005Metric; symbol ARC1_R08:C0603 -> ARC1_R85:C0402; LCSC C19702 -> C1525; MPN CL10A106KP8NNNC -> CL05B104KO5NNNC
- H5, H6: symbol ARC1_R08:MH_NPTH -> ARC1_R85:MH_NPTH
- J3: footprint ARC1_R08:Hirose_DF40C-100DS-0.4V_51 -> ARC1_R85:Hirose_DF40C-100DS-0.4V_51; symbol ARC1_R08:MN820_RCPT -> ARC1_R85:MN820_RCPT
- J4: symbol ARC1_R08:HDR_2x5_127 -> ARC1_R85:HDR_2x5_127
- R40, R41, R42, R48: symbol ARC1_R08:R0402 -> ARC1_R85:R0402
- R43: value 10k -> 33R; symbol ARC1_R08:R0402 -> ARC1_R85:R0402; LCSC C25744 -> (none); MPN 0402WGF1002TCE -> (none); Manufacturer UNI-ROYAL -> (none); Note as VM820C; pull to module rail (no back-power) -> (none); Reuse SLIM4_R26_BOM_LINE (re-validate) -> (none)
- R44: symbol ARC1_R08:R0402 -> ARC1_R85:R0402; Note (none) -> as VM820C; pull to module rail (no back-power)
- R45: symbol ARC1_R08:R0402 -> ARC1_R85:R0402; Note BT820 held in reset until F133 drives it -> (none)
- R46: symbol ARC1_R08:R0402 -> ARC1_R85:R0402; Note BT820 DS 4.5.1: data lines need pull-downs (VM820C 10k) -> BT820 held in reset until F133 drives it
- R47: symbol ARC1_R08:R0402 -> ARC1_R85:R0402; Note (none) -> BT820 DS 4.5.1: data lines need pull-downs (VM820C 10k)
- R49: value 47k -> 10k; symbol ARC1_R08:R0402 -> ARC1_R85:R0402; LCSC (none) -> C25744; MPN (none) -> 0402WGF1002TCE; Manufacturer (none) -> UNI-ROYAL; Note F133 side: defined level while buffer hi-Z -> (none); Reuse (none) -> SLIM4_R26_BOM_LINE (re-validate)
- TP34: value BT_INT_N -> BT_SCK; symbol ARC1_R08:TP -> ARC1_R85:TP
- TP35: value BT_RST_N -> BT_MISO; symbol ARC1_R08:TP -> ARC1_R85:TP
- U17: symbol ARC1_R08:LVC1G125 -> ARC1_R85:LVC1G125
Connections:
- net 3V3: now also C65.1
- net 3V3_MN: now also R45.2, C67.1, C68.1; no longer C65.1, R43.2
- net BT_INT_N: now also R45.1, TP36.1; no longer R44.1, TP34.1
- net BT_IO2_M: now also R48.1; no longer R47.1
- net BT_IO3_M: now also R49.1; no longer R48.1
- net BT_MISO: now also TP35.1, R50.1; no longer R49.1
- net BT_MISO_M: now also R47.1; no longer R46.1
- net BT_MOSI: now also R41.2; no longer R40.2
- net BT_MOSI_F: now also R41.1; no longer R40.1
- net BT_RST_N: now also R43.2, R46.1, TP37.1; no longer R42.2, R45.1, TP35.1
- net BT_RST_N_F: now also R43.1; no longer R42.1
- net BT_SCK: now also R40.2, TP34.1
- net BT_SCK_F: now also R40.1
- net BT_SS_N: now also R42.1; no longer R41.1
- net BT_SS_N_M: now also R42.2, R44.1; no longer R41.2, R43.1
- net GND: now also C67.2, C68.2, R50.2; no longer R45.2
Other:
- title: ARC-1 Compact R08: MN820 (BT820B + 128 MiB DDR3L) module socket, host SPI1, LVDS to R09 panel -> ARC-1 Compact R8.5: MN820 (BT820B + 128 MiB DDR3L) module socket, host SPI1, LVDS to R09 panel
- moved on the sheet: C65, C66, R40, R41, R42, R43, R44, R45, R46, R47, R48, R49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
