File: hardware/arc1-compact/R85_WORK/cad/power.kicad_sch (KiCad schematic)
At the start: 94 parts, among them SW1 RESET, U10 3V3_T35 switch, U11 3V3_MN switch, U12 PSRAM_VDD switch, U13 AND, U14 TPS3808G30, U3 3V3 2A, U4 TPS3808G33, U5 VDD_CORE 0.95V, U6 1V8_DRAM, U7 1V8_AN, U8 TPS3808G09, U9 1V2_T35

Commit message: ARC-1 Compact R8.5: ECP5 board sheet (power tree, sysCONFIG SSPI, JTAG), regenerated KiCad (ERC 0), R8.5 rule checker, pin matrices + generated LPF, routed reproducible bitstream
Co-Authored-By: Claude Opus 5.5 <noreply@anthropic.com>
Claude-Session: https://claude.ai/code/session_01UkiuLdbjDvK75uDzAPKsGs
Parts:
- added C32: 1nF, Capacitor_SMD:C_0402_1005Metric, symbol ARC1_R85:C0402
- added C33: 100nF, Capacitor_SMD:C_0402_1005Metric, symbol ARC1_R85:C0402
- added FB2: ferrite 120R@100MHz, Inductor_SMD:L_0603_1608Metric, symbol ARC1_R85:FB0603
- added J11: FPGA power override, Connector_PinHeader_2.54mm:PinHeader_1x03_P2.54mm_Vertical, symbol ARC1_R85:HDR_1x3
- added R31: 10k, Resistor_SMD:R_0402_1005Metric, symbol ARC1_R85:R0402
- added TP23, TP24: GND, TestPoint:TestPoint_Pad_D1.0mm, symbol ARC1_R85:TP
- added U30: 2V5_FPGA_AUX, Package_TO_SOT_SMD:SOT-23-5, symbol ARC1_R85:TLV75525P
- C10, C11, C12, C13, C17, C18, C19, C4, C5, C6, C9: symbol ARC1_R08:C0805 -> ARC1_R85:C0805
- C14, C15, C16, C21, C24, C31, C7, C8: symbol ARC1_R08:C0402 -> ARC1_R85:C0402
- C20: symbol ARC1_R08:C0402 -> ARC1_R85:C0402; Note calc SR = 0.55*1000+30 us/V -> ~1.9 ms ramp = 1.7 V/ms (T35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 -> calc SR = 0.55*1000+30 us/V -> ~1.9 ms ramp = 1.7 V/ms (ECP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
- C22: symbol ARC1_R08:C0603 -> ARC1_R85:C0603
- C23, C26: value 1nF -> 1uF; symbol ARC1_R08:C0402 -> ARC1_R85:C0402; LCSC (none) -> C52923; MPN (none) -> CL05A105KA5NQNC; Manufacturer (none) -> Samsung; Reuse (none) -> SLIM4_R26_BOM_LINE (re-validate)
- C25: value 22uF -> 1nF; footprint Capacitor_SMD:C_0805_2012Metric -> Capacitor_SMD:C_0402_1005Metric; symbol ARC1_R08:C0805 -> ARC1_R85:C0402; LCSC C5674 -> (none); MPN CL21A226MQQNNNE -> (none); Manufacturer Samsung -> (none); Reuse SLIM4_R26_BOM_LINE (re-validate) -> (none)
- C27: value 1uF -> 22uF; footprint Capacitor_SMD:C_0402_1005Metric -> Capacitor_SMD:C_0805_2012Metric; symbol ARC1_R08:C0402 -> ARC1_R85:C0805; LCSC C52923 -> C5674; MPN CL05A105KA5NQNC -> CL21A226MQQNNNE
- C28: value 4.7uF -> 1nF; footprint Capacitor_SMD:C_0603_1608Metric -> Capacitor_SMD:C_0402_1005Metric; symbol ARC1_R08:C0603 -> ARC1_R85:C0402; LCSC C19666 -> (none); MPN CL10A475KO8NNNC -> (none); Manufacturer Samsung -> (none); Reuse SLIM4_R26_BOM_LINE (re-validate) -> (none)
- C29: value 100nF -> 1uF; symbol ARC1_R08:C0402 -> ARC1_R85:C0402; LCSC C1525 -> C52923; MPN CL05B104KO5NNNC -> CL05A105KA5NQNC
- C30: value 1nF -> 4.7uF; footprint Capacitor_SMD:C_0402_1005Metric -> Capacitor_SMD:C_0603_1608Metric; symbol ARC1_R08:C0402 -> ARC1_R85:C0603; LCSC (none) -> C19666; MPN (none) -> CL10A475KO8NNNC; Manufacturer (none) -> Samsung; Reuse (none) -> SLIM4_R26_BOM_LINE (re-validate)
- FID1, FID2, FID3: symbol ARC1_R08:FID -> ARC1_R85:FID
- H1, H2, H3, H4: symbol ARC1_R08:MH -> ARC1_R85:MH
- L1, L2, L3, L4: footprint ARC1_R08:SLIM4_FP_L2_ASWPA4035 -> ARC1_R85:SLIM4_FP_L2_ASWPA4035; symbol ARC1_R08:L4035 -> ARC1_R85:L4035
- R10, R12, R13, R14, R15, R17, R18, R19, R20, R28, R29, R8, R9: symbol ARC1_R08:R0402 -> ARC1_R85:R0402
- R11, R16: symbol ARC1_R08:R0603 -> ARC1_R85:R0603
- R21: value 100k -> 82.5k; symbol ARC1_R08:R0402 -> ARC1_R85:R0402; LCSC C25741 -> (none); MPN 0402WGF1003TCE -> (none); Manufacturer UNI-ROYAL -> (none); Note (none) -> 1 % (E96); Reuse SLIM4_R26_BOM_LINE (re-validate) -> (none)
- R22: symbol ARC1_R08:R0402 -> ARC1_R85:R0402; Note (none) -> 1 %
- R23: symbol ARC1_R08:R0603 -> ARC1_R85:R0603; Note staged power-on link / T35 isolation -> staged power-on link / ECP5 VCC current measurement
- R24: value 100k -> 1k; symbol ARC1_R08:R0402 -> ARC1_R85:R0402; LCSC C25741 -> (none); MPN 0402WGF1003TCE -> (none); Manufacturer UNI-ROYAL -> (none); Note T35 unpowered until F133 firmware enables it -> F133 PE0 drive; lets jumper J11 force the FPGA on for JTAG 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; Reuse SLIM4_R26_BOM_LINE (re-validate) -> (none)
- R25: symbol ARC1_R08:R0402 -> ARC1_R85:R0402; Note (none) -> FPGA unpowered until F133 firmware (or J11) enables it
- R26: symbol ARC1_R08:R0402 -> ARC1_R85:R0402; Note default ON even while F133 is in reset (graphics independen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 -> open-drain PG to F133 PD1 (rail-fault diagnosis)
- R27: symbol ARC1_R08:R0402 -> ARC1_R85:R0402; Note (none) -> default ON even while F133 is in reset (graphics independen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
- R30: value 10k -> 100k; symbol ARC1_R08:R0402 -> ARC1_R85:R0402; LCSC C25744 -> C25741; MPN 0402WGF1002TCE -> 0402WGF1003TCE
- SW1: symbol ARC1_R08:SW_B3U -> ARC1_R85:SW_B3U
- TP10, TP11, TP21, TP22, TP4, TP5, TP6, TP7, TP8, TP9: symbol ARC1_R08:TP -> ARC1_R85:TP
- TP12: value 1V2_T35 -> 1V1_FPGA; symbol ARC1_R08:TP -> ARC1_R85:TP
- TP13: value T35_1V2_PG -> FPGA_VCC_PG; symbol ARC1_R08:TP -> ARC1_R85:TP
- TP14: value 3V3_T35 -> FPGA_PWR_EN; symbol ARC1_R08:TP -> ARC1_R85:TP
- TP15: value 3V3_MN -> 3V3_FPGA; symbol ARC1_R08:TP -> ARC1_R85:TP
- TP16: value PSRAM_VDD -> 2V5_FPGA_AUX; symbol ARC1_R08:TP -> ARC1_R85:TP
- TP17: value PSRAM_PG -> 3V3_MN; symbol ARC1_R08:TP -> ARC1_R85:TP
- TP18: value PSRAM_EN -> PSRAM_VDD; symbol ARC1_R08:TP -> ARC1_R85:TP
- TP19: value GND -> PSRAM_PG; symbol ARC1_R08:TP -> ARC1_R85:TP
- TP20: value GND -> PSRAM_EN; symbol ARC1_R08:TP -> ARC1_R85:TP
- U10: value 3V3_T35 switch -> 3V3_FPGA switch; symbol ARC1_R08:TPS22918 -> ARC1_R85:TPS22918; Note T35 sequence: VCC first, VCCIO after (T35 DS) -> same enable as VCC: VCCIO with VCC/VCCAUX (TN-02038 s.4)
- U11, U12: symbol ARC1_R08:TPS22918 -> ARC1_R85:TPS22918
- U13: symbol ARC1_R08:LVC1G08 -> ARC1_R85:LVC1G08
- U14, U4, U8: symbol ARC1_R08:TPS3808 -> ARC1_R85:TPS3808
- U3: symbol ARC1_R08:TLV62569P -> ARC1_R85:TLV62569P
- U5, U6: symbol ARC1_R08:TLV62569 -> ARC1_R85:TLV62569
- U7: symbol ARC1_R08:TLV75518P -> ARC1_R85:TLV75518P
- U9: value 1V2_T35 -> 1V1_FPGA; symbol ARC1_R08:TLV62569P -> ARC1_R85:TLV62569P; Note calc: 0.6*(1+100k/100k)=1.20 V (T35 1.15/1.20/1.25) -> calc: 0.6*(1+82.5k/100k)=1.095 V (ECP5 VCC 1.045/1.10/1.155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
Connections:
- net 3V3: now also C26.1, C31.1, R27.2, J11.1; no longer C24.1, C29.1, R25.2
- net 3V3_MN: now also C27.1, TP17.1; no longer C25.1, TP15.1
- net GND: now also R25.2, R29.2, C32.2, C33.2, J11.3, TP23.1, TP24.1, U30.2 (GND); no longer R24.2, R27.2, TP19.1, TP20.1
- net MN_PWR_EN: now also R27.1; no longer R26.1
- net PSRAM_EN: now also R29.1, TP20.1; no longer R28.1, TP18.1
- net PSRAM_PG: now also TP19.1, R31.1; no longer R30.1, TP17.1
- net PSRAM_PWR_REQ: now also R28.1; no longer R27.1
- net PSRAM_SUP_CT: now also C32.1; no longer C30.1
- net PSRAM_SUP_MR_N: now also R30.1; no longer R29.1
- net PSRAM_VDD: now also C30.1, TP18.1; no longer C28.1, TP16.1
- net SW_MN_CT: now also C25.1; no longer C23.1
- net SW_PS_CT: now also C28.1; no longer C26.1
- net 1V2_T35 renamed 1V1_FPGA
- net 1V2_T35_REG renamed 1V1_FPGA_REG
- net 3V3_T35 renamed 3V3_FPGA
- net 3V3_FPGA: now also C23.1, C29.1, TP15.1, C33.1, R31.2, U30.1 (IN), U30.3 (EN); no longer C27.1, C31.1, R29.2, TP14.1
- net CDONE_DLY renamed DONE_DLY
- net FB_1V2 renamed FB_1V1
- net SW_1V2 renamed SW_1V1
- net SW_T35_CT renamed SW_FPGA_CT
- net T35_1V2_PG renamed FPGA_PWR_EN
- net FPGA_PWR_EN: now also R24.2, TP14.1, U9.1 (EN), J11.2; no longer TP13.1, U9.5 (PG)
- net T35_PWR_EN renamed FPGA_PWR_EN_F
- net FPGA_PWR_EN_F: no longer U9.1 (EN)
- new net 2V5_AUX_REG: C24.1, FB2.1, U30.5 (OUT)
- new net 2V5_FPGA_AUX: FB2.2, TP16.1
- new net FPGA_VCC_PG: R26.1, TP13.1, U9.5 (PG)
- no-connect marks 1 -> 2
Other:
- title: ARC-1 Compact R08: Regulators, rail order, supervisors, staged-power links -> ARC-1 Compact R8.5: Regulators, rail order, supervisors, staged-power links
- moved on the sheet: C10, C11, C12, C13, C14, C15, C16, C17, C18, C19, C20, C21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
