File: hardware/arc1-compact/R85_WORK/cad/psram.kicad_sch (KiCad schematic)
At the start: 18 parts, among them U25 APS6404L-3SQR, U26 SN74LVC07A

Commit message: ARC-1 Compact R8.5: ECP5 board sheet (power tree, sysCONFIG SSPI, JTAG), regenerated KiCad (ERC 0), R8.5 rule checker, pin matrices + generated LPF, routed reproducible bitstream
Co-Authored-By: Claude Opus 5.5 <noreply@anthropic.com>
Claude-Session: https://claude.ai/code/session_01UkiuLdbjDvK75uDzAPKsGs
Parts:
- removed C106, C108: 100nF, Capacitor_SMD:C_0402_1005Metric, symbol ARC1_R08:C0402
- removed C107: 1uF, Capacitor_SMD:C_0402_1005Metric, symbol ARC1_R08:C0402
- removed R71: 22R, Resistor_SMD:R_0402_1005Metric, symbol ARC1_R08:R0402
- removed R72: 10k, Resistor_SMD:R_0402_1005Metric, symbol ARC1_R08:R0402
- removed R73, R74: 100k, Resistor_SMD:R_0402_1005Metric, symbol ARC1_R08:R0402
- removed R82, R83: 1.5k, Resistor_SMD:R_0402_1005Metric, symbol ARC1_R08:R0402
- removed U26: SN74LVC07A, Package_SO:TSSOP-14_4.4x5mm_P0.65mm, symbol ARC1_R08:LVC07A
- added C129: 100nF, Capacitor_SMD:C_0402_1005Metric, symbol ARC1_R85:C0402
- added C130: 1uF, Capacitor_SMD:C_0402_1005Metric, symbol ARC1_R85:C0402
- R75: value 100k -> 22R; symbol ARC1_R08:R0402 -> ARC1_R85:R0402; LCSC C25741 -> (none); MPN 0402WGF1003TCE -> (none); Manufacturer UNI-ROYAL -> (none); Note static: idle level in user mode, load 34 uA << 0.2 mA VOH t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 -> source termination near the FPGA; Reuse SLIM4_R26_BOM_LINE (re-validate) -> (none)
- R76: value 100k -> 10k; symbol ARC1_R08:R0402 -> ARC1_R85:R0402; LCSC C25741 -> C25744; MPN 0402WGF1003TCE -> 0402WGF1002TCE; Note static: idle level in user mode, load 34 uA << 0.2 mA VOH t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 -> CE# tracks the switched VDD during the ramp (PULLMODE=NONE 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
- R77: symbol ARC1_R08:R0402 -> ARC1_R85:R0402
- R78, R79, R80, R81: value 1.5k -> 100k; symbol ARC1_R08:R0402 -> ARC1_R85:R0402; LCSC C25867 -> C25741; MPN 0402WGF1501TCE -> 0402WGF1003TCE; Note calc: vs T35 weak PU 27k min @3.40 V -> <= 0.38 V (VOL 0.2 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 -> static: idle level in user mode, load 34 uA << 0.2 mA VOH t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
- U25: symbol ARC1_R08:APS6404L -> ARC1_R85:APS6404L
Connections:
- net PD_CE is gone; now on net GND: R78.2
- net PD_SCLK is gone; now on net GND: R79.2
- net PD_SIO0 is gone; now on net GND: R80.2
- net PD_SIO1 is gone; now on net GND: R81.2
- net GND: now also C129.2, C130.2; no longer R75.2, R76.2
- net PSRAM_CE_N: now also R76.1; no longer R78.1
- net PSRAM_SCLK: now also R75.2, R77.1; no longer R79.1
- net PSRAM_SIO0: now also R78.1; no longer R80.1
- net PSRAM_SIO1: now also R79.1; no longer R75.1, R81.1
- net PSRAM_SIO2: now also R80.1; no longer R76.1
- net PSRAM_SIO3: now also R81.1; no longer R77.1
- net PSRAM_VDD: now also R76.2, C129.1, C130.1
- new net PSRAM_SCLK_F: R75.1
Other:
- note added: "APS6404L 8 MiB PSRAM: switched VDD (DONE-gated), static pulls Sheet generated from design.py; global labels carry every net."
- note removed: "APS6404L 8 MiB PSRAM: switched VDD, switched start-up pull-downs Sheet generated from design.py; global labels carry every net."
- title: ARC-1 Compact R08: APS6404L 8 MiB PSRAM: switched VDD, switched start-up pull-downs -> ARC-1 Compact R8.5: APS6404L 8 MiB PSRAM: switched VDD (DONE-gated), static pulls
- moved on the sheet: R75, R76, R77, R78, R79, R80, R81, U25
