File: hardware/arc1-compact/R85_WORK/cad/sd_audio.kicad_sch (KiCad schematic)
At the start: 25 parts, among them J7 microSD, J8 SPK L, J9 SPK R, U27 SD power switch, U28 MAX98357A L, U29 MAX98357A R

Commit message: ARC-1 Compact R8.5: ECP5 board sheet (power tree, sysCONFIG SSPI, JTAG), regenerated KiCad (ERC 0), R8.5 rule checker, pin matrices + generated LPF, routed reproducible bitstream
Co-Authored-By: Claude Opus 5.5 <noreply@anthropic.com>
Claude-Session: https://claude.ai/code/session_01UkiuLdbjDvK75uDzAPKsGs
Parts:
- removed C109: 1nF, Capacitor_SMD:C_0402_1005Metric, symbol ARC1_R08:C0402
- removed C110: 10uF, Capacitor_SMD:C_0603_1608Metric, symbol ARC1_R08:C0603
- removed C111, C113, C115: 100nF, Capacitor_SMD:C_0402_1005Metric, symbol ARC1_R08:C0402
- removed C112, C114: 10uF, Capacitor_SMD:C_0805_2012Metric, symbol ARC1_R08:C0805
- removed R92: 210k, Resistor_SMD:R_0402_1005Metric, symbol ARC1_R08:R0402
- removed R93: 100k, Resistor_SMD:R_0402_1005Metric, symbol ARC1_R08:R0402
- removed TP40: SD_VDD, TestPoint:TestPoint_Pad_D1.0mm, symbol ARC1_R08:TP
- removed TP41: SD_DET_N, TestPoint:TestPoint_Pad_D1.0mm, symbol ARC1_R08:TP
- added C131: 1nF, Capacitor_SMD:C_0402_1005Metric, symbol ARC1_R85:C0402
- added C132: 10uF, Capacitor_SMD:C_0603_1608Metric, symbol ARC1_R85:C0603
- added C133, C135, C137: 100nF, Capacitor_SMD:C_0402_1005Metric, symbol ARC1_R85:C0402
- added C134, C136: 10uF, Capacitor_SMD:C_0805_2012Metric, symbol ARC1_R85:C0805
- added R82: 100k, Resistor_SMD:R_0402_1005Metric, symbol ARC1_R85:R0402
- added R83: 33R, Resistor_SMD:R_0402_1005Metric, symbol ARC1_R85:R0402
- added TP44: SD_VDD, TestPoint:TestPoint_Pad_D1.0mm, symbol ARC1_R85:TP
- added TP45: SD_DET_N, TestPoint:TestPoint_Pad_D1.0mm, symbol ARC1_R85:TP
- J7: symbol ARC1_R08:MICROSD -> ARC1_R85:MICROSD
- J8, J9: symbol ARC1_R08:JST_PH2 -> ARC1_R85:JST_PH2
- R84: value 100k -> 47k; symbol ARC1_R08:R0402 -> ARC1_R85:R0402; LCSC C25741 -> (none); MPN 0402WGF1003TCE -> (none); Manufacturer UNI-ROYAL -> (none); Note (none) -> SD pull-ups to the card rail (no back-power when card power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; Reuse SLIM4_R26_BOM_LINE (re-validate) -> (none)
- R85: value 33R -> 47k; symbol ARC1_R08:R0402 -> ARC1_R85:R0402; Note (none) -> SD pull-ups to the card rail (no back-power when card power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
- R86, R87, R88: symbol ARC1_R08:R0402 -> ARC1_R85:R0402
- R89: value 47k -> 10k; symbol ARC1_R08:R0402 -> ARC1_R85:R0402; LCSC (none) -> C25744; MPN (none) -> 0402WGF1002TCE; Manufacturer (none) -> UNI-ROYAL; Note SD pull-ups to the card rail (no back-power when card power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 -> (none); Reuse (none) -> SLIM4_R26_BOM_LINE (re-validate)
- R90: value 47k -> 210k; symbol ARC1_R08:R0402 -> ARC1_R85:R0402; Note SD pull-ups to the card rail (no back-power when card power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 -> (none)
- R91: value 10k -> 100k; symbol ARC1_R08:R0402 -> ARC1_R85:R0402; LCSC C25744 -> C25741; MPN 0402WGF1002TCE -> 0402WGF1003TCE; Note (none) -> amps in shutdown while F133 in reset
- U27: symbol ARC1_R08:TPS22918 -> ARC1_R85:TPS22918
- U28, U29: symbol ARC1_R08:MAX98357A -> ARC1_R85:MAX98357A
Connections:
- net 3V3: now also R89.2; no longer R91.2
- net AMP_EN: now also R90.1, R91.1
- net AMP_R_SDMODE: now also R90.2
- net GND: now also R91.2, C131.2, C132.2, C133.2, C134.2, C135.2, C136.2, C137.2, R82.2; no longer R84.2
- net SD_CLK: now also R83.2; no longer R85.2
- net SD_CLK_F: now also R83.1; no longer R85.1
- net SD_CMD: now also R84.1; no longer R86.1
- net SD_D0: now also R85.1; no longer R87.1
- net SD_D1: now also R86.1; no longer R88.1
- net SD_D2: now also R87.1; no longer R89.1
- net SD_D3: now also R88.1; no longer R90.1
- net SD_DET_N: now also R89.1, TP45.1; no longer R91.1
- net SD_PWR_EN: now also R82.1; no longer R84.1
- net SD_VDD: now also R84.2, R85.2, C132.1, C133.1, TP44.1; no longer R89.2, R90.2
- net SW_SD_CT: now also C131.1
- net VBUS_5V: now also C134.1, C135.1, C136.1, C137.1
Other:
- title: ARC-1 Compact R08: microSD game media (not boot), 2x MAX98357A I2S speakers -> ARC-1 Compact R8.5: microSD game media (not boot), 2x MAX98357A I2S speakers
- moved on the sheet: R84, R85, R86, R87, R88, R89, R90, R91
