File: hardware/arc1-compact/R85_WORK/cad/usb_power.kicad_sch (KiCad schematic)
At the start: 18 parts, among them J1 USB-C receptacle, U1 TUSB320LAI, U2 TPD2EUSB30

Commit message: ARC-1 Compact R8.5: ECP5 board sheet (power tree, sysCONFIG SSPI, JTAG), regenerated KiCad (ERC 0), R8.5 rule checker, pin matrices + generated LPF, routed reproducible bitstream
Co-Authored-By: Claude Opus 5.5 <noreply@anthropic.com>
Claude-Session: https://claude.ai/code/session_01UkiuLdbjDvK75uDzAPKsGs
Parts:
- C1: symbol ARC1_R08:C0805 -> ARC1_R85:C0805
- C2, C3: symbol ARC1_R08:C0402 -> ARC1_R85:C0402
- D1: symbol ARC1_R08:TVS_SMF -> ARC1_R85:TVS_SMF
- F1: symbol ARC1_R08:F1812 -> ARC1_R85:F1812
- J1: symbol ARC1_R08:USB_C -> ARC1_R85:USB_C
- R1, R2, R3, R4, R5, R6, R7: symbol ARC1_R08:R0402 -> ARC1_R85:R0402
- TP1, TP2, TP3: symbol ARC1_R08:TP -> ARC1_R85:TP
- U1: footprint ARC1_R08:SLIM4_FP_U13_TUSB320LAI_RWB_X2QFN12 -> ARC1_R85:SLIM4_FP_U13_TUSB320LAI_RWB_X2QFN12; symbol ARC1_R08:TUSB320LAI -> ARC1_R85:TUSB320LAI
- U2: footprint ARC1_R08:SLIM4_FP_U11_TPD2EUSB30_DRT3 -> ARC1_R85:SLIM4_FP_U11_TPD2EUSB30_DRT3; symbol ARC1_R08:TPD2EUSB30 -> ARC1_R85:TPD2EUSB30
Other:
- title: ARC-1 Compact R08: USB-C sink (no host), VBUS protection, USB0 device/FEL -> ARC-1 Compact R8.5: USB-C sink (no host), VBUS protection, USB0 device/FEL
