File: hardware/arc1-compact/R85C_WORK/cad/controls.kicad_sch (KiCad schematic)
At the start: 20 parts, among them J10 F133 UART0, SW10 Y, SW11 L, SW12 R, SW13 START, SW14 SELECT, SW15 HOME, SW3 UP, SW4 DOWN, SW5 LEFT, SW6 RIGHT, SW7 A, SW8 B, SW9 X

Commit message: R85C C3: RGMII on F133 PG0-PG12 to ECP5 bank 0, buttons moved to PD2-9/PD14/PD15/PD22/PB2/PB3
- design.py: 12 RGMII nets with 22R series resistors at each driver, 100k CTL pull-downs; RXCK onto PCLKT0_0 (B11)
- F133 mux transcription extended from DS rev 2.3 Table 4-3 (PG0-PG12, PD2-PD9, PD14, PD15)
- pin matrix / LPF generated from the board plan (identical to the C2 provisional LPF, which is removed);
  bitstream unchanged (087cb5a2...12be)
- board rule rgmii_link + 7 negative tests (17/17 rules, 37 tests pass); KiCad ERC 0/0; crosscheck PASS
- RGMII timing budget from F133 DS Table 5-21 and ECP5 DS-02012 Table 3.22: 0.53 / 0.53 / 0.5 ns, CONDITIONAL
  (board skew and delay-chain centring are assumptions); docs/RGMII_LINK_R85C.md
- firmware host tests 799/0 and freestanding build pass with the new pin header

Co-Authored-By: Claude Opus 5.5 <noreply@anthropic.com>
Claude-Session: https://claude.ai/code/session_01UkiuLdbjDvK75uDzAPKsGs
Parts:
- removed R92, R93: 1k, Resistor_SMD:R_0402_1005Metric, symbol ARC1_R85:R0402
- removed R94: 2k, Resistor_SMD:R_0402_1005Metric, symbol ARC1_R85:R0402
- added R106, R107: 1k, Resistor_SMD:R_0402_1005Metric, symbol ARC1_R85:R0402
- added R108: 2k, Resistor_SMD:R_0402_1005Metric, symbol ARC1_R85:R0402
Connections:
- net 3V3: now also R108.1
- net LED_3V3_R: now also R108.2
- net LED_ERROR: now also R107.1
- net LED_ERROR_R: now also R107.2
- net LED_STATUS: now also R106.1
- net LED_STATUS_R: now also R106.2
