File: hardware/arc1-compact/R85C_WORK/cad/fpga_ecp5.kicad_sch (KiCad schematic)
At the start: 101 parts, among them J5 ECP5 JTAG, J6 FPGA UART, U18 LFE5U-45F-6BG381C, U20 Schmitt, U21 iso SCK, U22 iso MOSI, U23 iso SS, U24 iso MISO, X1 25MHz

Commit message: R85C C3: RGMII on F133 PG0-PG12 to ECP5 bank 0, buttons moved to PD2-9/PD14/PD15/PD22/PB2/PB3
- design.py: 12 RGMII nets with 22R series resistors at each driver, 100k CTL pull-downs; RXCK onto PCLKT0_0 (B11)
- F133 mux transcription extended from DS rev 2.3 Table 4-3 (PG0-PG12, PD2-PD9, PD14, PD15)
- pin matrix / LPF generated from the board plan (identical to the C2 provisional LPF, which is removed);
  bitstream unchanged (087cb5a2...12be)
- board rule rgmii_link + 7 negative tests (17/17 rules, 37 tests pass); KiCad ERC 0/0; crosscheck PASS
- RGMII timing budget from F133 DS Table 5-21 and ECP5 DS-02012 Table 3.22: 0.53 / 0.53 / 0.5 ns, CONDITIONAL
  (board skew and delay-chain centring are assumptions); docs/RGMII_LINK_R85C.md
- firmware host tests 799/0 and freestanding build pass with the new pin header

Co-Authored-By: Claude Opus 5.5 <noreply@anthropic.com>
Claude-Session: https://claude.ai/code/session_01UkiuLdbjDvK75uDzAPKsGs
Parts:
- added R75, R76, R77: 4.7k, Resistor_SMD:R_0402_1005Metric, symbol ARC1_R85:R0402
- added R78, R82: 33R, Resistor_SMD:R_0402_1005Metric, symbol ARC1_R85:R0402
- added R79, R83, R84: 10k, Resistor_SMD:R_0402_1005Metric, symbol ARC1_R85:R0402
- added R80: 470R, Resistor_SMD:R_0402_1005Metric, symbol ARC1_R85:R0402
- added R81, R85, R86: 100k, Resistor_SMD:R_0402_1005Metric, symbol ARC1_R85:R0402
- added R87, R88: 1k, Resistor_SMD:R_0402_1005Metric, symbol ARC1_R85:R0402
- added TP44: FPGA_OSC_25M, TestPoint:TestPoint_Pad_D1.0mm, symbol ARC1_R85:TP
- added TP45: FPGA_SCK, TestPoint:TestPoint_Pad_D1.0mm, symbol ARC1_R85:TP
- R51: value 4.7k -> 22R; Note TN-02038: 4.7k to VCCIO8 -> RGMII F133->ECP5 series R, place at F133 (TXCK)
- R52: value 470R -> 22R; Note F133 PE8 used open-drain (low or input only): worst case 0.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 -> RGMII F133->ECP5 series R, place at F133 (TXD0)
- R53: value 4.7k -> 22R; Note TN-02038: 4.7k; reads 0 at F133 PD0 while the FPGA is off -> RGMII F133->ECP5 series R, place at F133 (TXD1)
- R54: value 4.7k -> 22R; Note TN-02038: 4.7k; reads 0 at F133 PE9 while the FPGA is off -> RGMII F133->ECP5 series R, place at F133 (TXD2)
- R55: value 4.7k -> 22R; Note TN-02039 6.2: SN 4.7k pull-up to VCCIO8 -> RGMII F133->ECP5 series R, place at F133 (TXD3)
- R56: value 4.7k -> 22R; Note CFG_0 = 1 (1-10k); CFG_1/CFG_2 tied to GND -> 001 slave SPI -> RGMII F133->ECP5 series R, place at F133 (TXCTL)
- R57: value 10k -> 22R; LCSC C25744 -> (none); MPN 0402WGF1002TCE -> (none); Manufacturer UNI-ROYAL -> (none); Note HOLDN inactive (conservative: TN lists HOLDN as optional SS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 -> RGMII ECP5->F133 series R, place at ECP5 (RXCK); Reuse SLIM4_R26_BOM_LINE (re-validate) -> (none)
- R58: value 1k -> 22R; Note TN-02038 Table 6.2: CCLK 510R-1k pull-up -> RGMII ECP5->F133 series R, place at ECP5 (RXD0)
- R59: value 4.7k -> 22R; Note TCK pull-down 4.7k (no internal pull) -> RGMII ECP5->F133 series R, place at ECP5 (RXD1)
- R60: value 4.7k -> 22R; Note (none) -> RGMII ECP5->F133 series R, place at ECP5 (RXD2)
- R61: value 4.7k -> 22R; Note (none) -> RGMII ECP5->F133 series R, place at ECP5 (RXD3)
- R62: value 4.7k -> 22R; Note (none) -> RGMII ECP5->F133 series R, place at ECP5 (RXCTL)
- R63: value 4.7k -> 100k; LCSC (none) -> C25741; MPN (none) -> 0402WGF1003TCE; Manufacturer (none) -> UNI-ROYAL; Note open drain; 4.7k vs ECP5 config-time weak pull-down 150 uA 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 -> ECP5 RX idle while F133 PG12 is hi-Z (reset, FEL, before EM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; Reuse (none) -> SLIM4_R26_BOM_LINE (re-validate)
- R64: value 33R -> 100k; LCSC (none) -> C25741; MPN (none) -> 0402WGF1003TCE; Manufacturer (none) -> UNI-ROYAL; Note (none) -> F133 EMAC RX idle while the ECP5 is unpowered or unconfigur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; Reuse (none) -> SLIM4_R26_BOM_LINE (re-validate)
- R65: value 10k -> 4.7k; LCSC C25744 -> (none); MPN 0402WGF1002TCE -> (none); Manufacturer UNI-ROYAL -> (none); Note calc: tau = (4.7k+10k) * 100nF = 1.5 ms; delay >= 0.5 ms -> TN-02038: 4.7k to VCCIO8; Reuse SLIM4_R26_BOM_LINE (re-validate) -> (none)
- R66: Note (none) -> F133 PE8 used open-drain (low or input only): worst case 0.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
- R67: value 100k -> 4.7k; LCSC C25741 -> (none); MPN 0402WGF1003TCE -> (none); Manufacturer UNI-ROYAL -> (none); Note defined low while 3V3_FPGA is off -> TN-02038: 4.7k; reads 0 at F133 PD0 while the FPGA is off; Reuse SLIM4_R26_BOM_LINE (re-validate) -> (none)
- R68: value 33R -> 4.7k; Note CCLK series 22-80R near the driver (TN-02038 Table 6.2) -> TN-02038: 4.7k; reads 0 at F133 PE9 while the FPGA is off
- R69: value 10k -> 4.7k; LCSC C25744 -> (none); MPN 0402WGF1002TCE -> (none); Manufacturer UNI-ROYAL -> (none); Note isolation buffers disabled at reset -> TN-02039 6.2: SN 4.7k pull-up to VCCIO8; Reuse SLIM4_R26_BOM_LINE (re-validate) -> (none)
- R70: value 10k -> 4.7k; LCSC C25744 -> (none); MPN 0402WGF1002TCE -> (none); Manufacturer UNI-ROYAL -> (none); Note FPGA deselected and MISO buffer off at reset -> CFG_0 = 1 (1-10k); CFG_1/CFG_2 tied to GND -> 001 slave SPI; Reuse SLIM4_R26_BOM_LINE (re-validate) -> (none)
- R71: value 100k -> 10k; LCSC C25741 -> C25744; MPN 0402WGF1003TCE -> 0402WGF1002TCE; Note (none) -> HOLDN inactive (conservative: TN lists HOLDN as optional SS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
- R72: value 100k -> 1k; LCSC C25741 -> (none); MPN 0402WGF1003TCE -> (none); Manufacturer UNI-ROYAL -> (none); Note buffer input defined when the FPGA is off/unconfigured (MIS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 -> TN-02038 Table 6.2: CCLK 510R-1k pull-up; Reuse SLIM4_R26_BOM_LINE (re-validate) -> (none)
- R73: value 1k -> 4.7k; Note (none) -> TCK pull-down 4.7k (no internal pull)
- R74: value 1k -> 4.7k; Note limits injection from an external UART adapter into an unpo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 -> (none)
- TP38: value FPGA_DONE -> ETH_TXCK
- TP39: value DONE_DLY -> ETH_RXCK
- TP40: value FPGA_PROGRAMN -> FPGA_DONE
- TP41: value FPGA_INITN -> DONE_DLY
- TP42: value FPGA_OSC_25M -> FPGA_PROGRAMN
- TP43: value FPGA_SCK -> FPGA_INITN
Connections:
- net 3V3: now also R83.2, R84.2; no longer R69.2, R70.2
- net 3V3_FPGA: now also R65.2, R67.2, R68.2, R69.2, R70.2, R71.2, R72.2, R74.2, R75.2, R76.2, R77.2; no longer R51.2, R53.2, R54.2, R55.2, R56.2, R57.2, R58.2, R60.2, R61.2, R62.2, R63.2
- net DONE_DIS: now also R80.2; no longer R66.2
- net DONE_DLY: now also TP41.1, R81.1; no longer R67.1, TP39.1
- net DONE_RC: now also R79.2, R80.1; no longer R65.2, R66.1
- net FPGA_BUS_EN_N: now also R83.1; no longer R69.1
- net FPGA_CFG0: now also R70.1; no longer R56.1
- net FPGA_DBG_RX: now also R88.2; no longer R74.2
- net FPGA_DBG_RX_J: now also R88.1; no longer R74.1
- net FPGA_DONE: now also R68.1, TP40.1, R79.1; no longer R54.1, R65.1, TP38.1
- net FPGA_HOLDN: now also R71.1; no longer R57.1
- net FPGA_INITN: now also R67.1, TP43.1; no longer R53.1, TP41.1
- net FPGA_IRQ_N: now also R77.1; no longer R63.1
- net FPGA_LED0: now also R87.1; no longer R73.1
- net FPGA_LED0_R: now also R87.2; no longer R73.2
- net FPGA_MISO: now also R86.1; no longer R72.1
- net FPGA_MOSI: now also R85.1; no longer R71.1
- net FPGA_OSC_25M: now also R78.2, TP44.1; no longer R64.2, TP42.1
- net FPGA_OSC_25M_X: now also R78.1; no longer R64.1
- net FPGA_PROGRAMN: now also R65.1, R66.2, TP42.1; no longer R51.1, R52.2, TP40.1
- net FPGA_PROGRAMN_F: now also R66.1; no longer R52.1
- net FPGA_SCK: now also R72.1, R82.2, TP45.1; no longer R58.1, R68.2, TP43.1
- net FPGA_SCK_B: now also R82.1; no longer R68.1
- net FPGA_SS_N: now also R69.1; no longer R55.1
- net FPGA_SS_N_F: now also R84.1; no longer R70.1
- net FPGA_TCK: now also R73.1; no longer R59.1
- net FPGA_TDI: now also R75.1; no longer R61.1
- net FPGA_TDO: now also R76.1; no longer R62.1
- net FPGA_TMS: now also R74.1; no longer R60.1
- net GND: now also R63.2, R64.2, R73.2, R81.2, R85.2, R86.2; no longer R59.2, R67.2, R71.2, R72.2
- net ETH_TXCK: now reaches U18.B11 (PT38A/PCLKT0_0)
- net ETH_TXCK: now also R51.2, TP38.1
- net ETH_TXD1: now reaches U18.B9 (PT31A)
- net ETH_TXD1: now also R53.2
- net ETH_TXD0: now reaches U18.C10 (PT31B)
- net ETH_TXD0: now also R52.2
- net ETH_RXCTL_E: now reaches U18.C7 (PT11B)
- net ETH_RXCTL_E: now also R62.1
- net ETH_RXCK_E: now reaches U18.C8 (PT15A)
- net ETH_RXCK_E: now also R57.1
- net ETH_TXD2: now reaches U18.C9 (PT27A)
- net ETH_TXD2: now also R54.2
- net ETH_TXD3: now reaches U18.D10 (PT29A)
- net ETH_TXD3: now also R55.2
- net ETH_RXD2_E: now reaches U18.D8 (PT13B)
- net ETH_RXD2_E: now also R60.1
- net ETH_RXD0_E: now reaches U18.D9 (PT20A)
- net ETH_RXD0_E: now also R58.1
- net ETH_TXCTL: now reaches U18.E10 (PT29B)
- net ETH_TXCTL: now also R56.2, R63.1
- net ETH_RXD3_E: now reaches U18.E8 (PT13A)
- net ETH_RXD3_E: now also R61.1
- net ETH_RXD1_E: now reaches U18.E9 (PT20B)
- net ETH_RXD1_E: now also R59.1
- new net ETH_RXCK: R57.2, TP39.1
- new net ETH_RXCTL: R62.2, R64.1
- new net ETH_RXD0: R58.2
- new net ETH_RXD1: R59.2
- new net ETH_RXD2: R60.2
- new net ETH_RXD3: R61.2
- new net ETH_TXCK_F: R51.1
- new net ETH_TXCTL_F: R56.1
- new net ETH_TXD0_F: R52.1
- new net ETH_TXD1_F: R53.1
- new net ETH_TXD2_F: R54.1
- new net ETH_TXD3_F: R55.1
- no-connect marks 199 -> 187
Other:
- moved on the sheet: C100, C101, C102, C103, C104, C105, C106, C107, C108, C109, C110, C111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
