File: hardware/arc1-compact/R85C_WORK/cad/psram.kicad_sch (KiCad schematic)
At the start: 10 parts, among them U25 APS6404L-3SQR

Commit message: R85C C3: RGMII on F133 PG0-PG12 to ECP5 bank 0, buttons moved to PD2-9/PD14/PD15/PD22/PB2/PB3
- design.py: 12 RGMII nets with 22R series resistors at each driver, 100k CTL pull-downs; RXCK onto PCLKT0_0 (B11)
- F133 mux transcription extended from DS rev 2.3 Table 4-3 (PG0-PG12, PD2-PD9, PD14, PD15)
- pin matrix / LPF generated from the board plan (identical to the C2 provisional LPF, which is removed);
  bitstream unchanged (087cb5a2...12be)
- board rule rgmii_link + 7 negative tests (17/17 rules, 37 tests pass); KiCad ERC 0/0; crosscheck PASS
- RGMII timing budget from F133 DS Table 5-21 and ECP5 DS-02012 Table 3.22: 0.53 / 0.53 / 0.5 ns, CONDITIONAL
  (board skew and delay-chain centring are assumptions); docs/RGMII_LINK_R85C.md
- firmware host tests 799/0 and freestanding build pass with the new pin header

Co-Authored-By: Claude Opus 5.5 <noreply@anthropic.com>
Claude-Session: https://claude.ai/code/session_01UkiuLdbjDvK75uDzAPKsGs
Parts:
- removed R75: 22R, Resistor_SMD:R_0402_1005Metric, symbol ARC1_R85:R0402
- removed R76: 10k, Resistor_SMD:R_0402_1005Metric, symbol ARC1_R85:R0402
- removed R77, R78, R79, R80, R81: 100k, Resistor_SMD:R_0402_1005Metric, symbol ARC1_R85:R0402
- added R89: 22R, Resistor_SMD:R_0402_1005Metric, symbol ARC1_R85:R0402
- added R90: 10k, Resistor_SMD:R_0402_1005Metric, symbol ARC1_R85:R0402
- added R91, R92, R93, R94, R95: 100k, Resistor_SMD:R_0402_1005Metric, symbol ARC1_R85:R0402
Connections:
- net GND: now also R91.2, R92.2, R93.2, R94.2, R95.2
- net PSRAM_CE_N: now also R90.1
- net PSRAM_SCLK: now also R89.2, R91.1
- net PSRAM_SCLK_F: now also R89.1
- net PSRAM_SIO0: now also R92.1
- net PSRAM_SIO1: now also R93.1
- net PSRAM_SIO2: now also R94.1
- net PSRAM_SIO3: now also R95.1
- net PSRAM_VDD: now also R90.2
