File: hardware/arc1-compact/R85C_WORK/cad/sd_audio.kicad_sch (KiCad schematic)
At the start: 25 parts, among them J7 microSD, J8 SPK L, J9 SPK R, U27 SD power switch, U28 MAX98357A L, U29 MAX98357A R

Commit message: R85C C3: RGMII on F133 PG0-PG12 to ECP5 bank 0, buttons moved to PD2-9/PD14/PD15/PD22/PB2/PB3
- design.py: 12 RGMII nets with 22R series resistors at each driver, 100k CTL pull-downs; RXCK onto PCLKT0_0 (B11)
- F133 mux transcription extended from DS rev 2.3 Table 4-3 (PG0-PG12, PD2-PD9, PD14, PD15)
- pin matrix / LPF generated from the board plan (identical to the C2 provisional LPF, which is removed);
  bitstream unchanged (087cb5a2...12be)
- board rule rgmii_link + 7 negative tests (17/17 rules, 37 tests pass); KiCad ERC 0/0; crosscheck PASS
- RGMII timing budget from F133 DS Table 5-21 and ECP5 DS-02012 Table 3.22: 0.53 / 0.53 / 0.5 ns, CONDITIONAL
  (board skew and delay-chain centring are assumptions); docs/RGMII_LINK_R85C.md
- firmware host tests 799/0 and freestanding build pass with the new pin header

Co-Authored-By: Claude Opus 5.5 <noreply@anthropic.com>
Claude-Session: https://claude.ai/code/session_01UkiuLdbjDvK75uDzAPKsGs
Parts:
- removed R82, R91: 100k, Resistor_SMD:R_0402_1005Metric, symbol ARC1_R85:R0402
- removed R83: 33R, Resistor_SMD:R_0402_1005Metric, symbol ARC1_R85:R0402
- removed R84, R85, R86, R87, R88: 47k, Resistor_SMD:R_0402_1005Metric, symbol ARC1_R85:R0402
- removed R89: 10k, Resistor_SMD:R_0402_1005Metric, symbol ARC1_R85:R0402
- removed R90: 210k, Resistor_SMD:R_0402_1005Metric, symbol ARC1_R85:R0402
- removed TP44: SD_VDD, TestPoint:TestPoint_Pad_D1.0mm, symbol ARC1_R85:TP
- removed TP45: SD_DET_N, TestPoint:TestPoint_Pad_D1.0mm, symbol ARC1_R85:TP
- added R100, R101, R102, R98, R99: 47k, Resistor_SMD:R_0402_1005Metric, symbol ARC1_R85:R0402
- added R103: 10k, Resistor_SMD:R_0402_1005Metric, symbol ARC1_R85:R0402
- added R104: 210k, Resistor_SMD:R_0402_1005Metric, symbol ARC1_R85:R0402
- added R105, R96: 100k, Resistor_SMD:R_0402_1005Metric, symbol ARC1_R85:R0402
- added R97: 33R, Resistor_SMD:R_0402_1005Metric, symbol ARC1_R85:R0402
- added TP46: SD_VDD, TestPoint:TestPoint_Pad_D1.0mm, symbol ARC1_R85:TP
- added TP47: SD_DET_N, TestPoint:TestPoint_Pad_D1.0mm, symbol ARC1_R85:TP
Connections:
- net 3V3: now also R103.2
- net AMP_EN: now also R104.1, R105.1
- net AMP_R_SDMODE: now also R104.2
- net GND: now also R105.2, R96.2
- net SD_CLK: now also R97.2
- net SD_CLK_F: now also R97.1
- net SD_CMD: now also R98.1
- net SD_D0: now also R99.1
- net SD_D1: now also R100.1
- net SD_D2: now also R101.1
- net SD_D3: now also R102.1
- net SD_DET_N: now also R103.1, TP47.1
- net SD_PWR_EN: now also R96.1
- net SD_VDD: now also R100.2, R101.2, R102.2, R98.2, R99.2, TP46.1
