File: hardware/arc1-compact/R10_WORK/cad/boot_nor.kicad_sch (KiCad schematic)
At the start: 19 parts, among them J4 LA SPI0, SW2 FEL (NOR reset), U18 W25Q512JVFIQ

Commit message: R10 change order rev 1.1: HDMI audio (ADV7513), USB0 role mux + hub + 2x front USB-A, eMMC, buttonless board
Owner handoff ARC1_R10_Handoff rev 1.1 (spec/, SHA-256 recorded) implemented in the generated schematic:
- D8 ADV7513BSWZ replaces the TFP410 (supersedes D6): D213 RGB888 video, D213 I2C2 init,
  F133 I2S2 -> HDMI embedded audio; own 1.8 V buck + 3 filtered domains; R_EXT 887R.
  D[23:0] pin order verified from the datasheet glyph coordinates.
- D9 F133 USB0 -> TS3USB221A (default rear USB-C device/FEL) or USB2422 hub -> two
  TPS2051C-switched front USB-A ports; F133 USB1 remains the internal D213 link; the D213
  recovery USB-C becomes internal fixture pads.
- D10 Samsung KLMAG1JETD-B041 16 GB eMMC on F133 SMHC0 (CONDITIONAL: SMHC0 documented for SD).
- D11 no switches: fixture pad pairs; game buttons, microSD and speakers removed.
- crosscheck_r10 section I (handoff go/no-go: 4 exterior connectors, 0 switches, I2S wired
  to the HDMI transmitter, USB0/USB1 roles, eMMC wiring) PASS; ERC 0/0; pin review PASS.
Sources: ADV7513 DS Rev B (LCSC copy), ADI AN-1270, Linux adv7511 driver, USB2422
DS00001726A, TPS20xxC SLVSAU6I, Samsung eMMC DS (not committed: vendor-confidential mark).

Co-Authored-By: Claude Opus 5.5 <noreply@anthropic.com>
Claude-Session: https://claude.ai/code/session_01UkiuLdbjDvK75uDzAPKsGs
Parts:
- removed C70: 100nF, Capacitor_SMD:C_0402_1005Metric, symbol ARC1_R10:C0402
- removed C71: 1uF, Capacitor_SMD:C_0402_1005Metric, symbol ARC1_R10:C0402
- removed J4: LA SPI0, Connector_PinHeader_1.27mm:PinHeader_2x05_P1.27mm_Vertical_SMD, symbol ARC1_R10:HDR_2x5_127
- removed R41: 22R, Resistor_SMD:R_0402_1005Metric, symbol ARC1_R10:R0402
- removed R42, R43: 3.3k, Resistor_SMD:R_0402_1005Metric, symbol ARC1_R10:R0402
- removed SW2: FEL (NOR reset), Button_Switch_SMD:SW_SPST_B3U-1000P, symbol ARC1_R10:SW_B3U
- removed TP29: SPI0_CLK, TestPoint:TestPoint_Pad_D1.0mm, symbol ARC1_R10:TP
- removed U18: W25Q512JVFIQ, Package_SO:SOIC-16W_7.5x10.3mm_P1.27mm, symbol ARC1_R10:W25Q512JVFIQ
- added C73: 100nF, Capacitor_SMD:C_0402_1005Metric, symbol ARC1_R10:C0402
- added C74: 1uF, Capacitor_SMD:C_0402_1005Metric, symbol ARC1_R10:C0402
- added J5: FEL pads (NOR reset), TestPoint:TestPoint_2Pads_Pitch2.54mm_Drill0.8mm, symbol ARC1_R10:PADS_1x2
- added J6: LA SPI0, Connector_PinHeader_1.27mm:PinHeader_2x05_P1.27mm_Vertical_SMD, symbol ARC1_R10:HDR_2x5_127
- added R48, R49, R50: 10k, Resistor_SMD:R_0402_1005Metric, symbol ARC1_R10:R0402
- added TP36: SPI0_IO3, TestPoint:TestPoint_Pad_D1.0mm, symbol ARC1_R10:TP
- added U19: W25Q512JVFIQ, Package_SO:SOIC-16W_7.5x10.3mm_P1.27mm, symbol ARC1_R10:W25Q512JVFIQ
- R44: value 10k -> 22R; LCSC C25744 -> C25092; MPN 0402WGF1002TCE -> 0402WGF220JTCE; Note (none) -> source series termination at F133
- R45: value 10k -> 3.3k; LCSC C25744 -> (none); MPN 0402WGF1002TCE -> (none); Manufacturer UNI-ROYAL -> (none); Note (none) -> BOOT-SEL0 = 0; Reuse SLIM4_R26_BOM_LINE (re-validate) -> (none)
- R46: value 10k -> 3.3k; LCSC C25744 -> (none); MPN 0402WGF1002TCE -> (none); Manufacturer UNI-ROYAL -> (none); Note (none) -> BOOT-SEL1 = 0; Reuse SLIM4_R26_BOM_LINE (re-validate) -> (none)
- TP30: value SPI0_MOSI -> SPI0_CLK
- TP31: value SPI0_MISO -> SPI0_MOSI
- TP32: value SPI0_CS0_N -> SPI0_MISO
- TP33: value NOR_RESET_N -> SPI0_CS0_N
- TP34: value SPI0_IO2 -> NOR_RESET_N
- TP35: value SPI0_IO3 -> SPI0_IO2
Connections:
- net 3V3: now also C73.1, C74.1, R48.2, R49.2, R50.2, U19.2 (VCC); no longer R44.2, R45.2, R46.2
- net F133_RESET_N: now also J6.10
- net FPGA12_SS_N_F: now also J6.8
- net GND: now also R45.2, R46.2, C73.2, C74.2, J5.2, J6.2, J6.4, J6.6, U19.10 (GND)
- net NOR_RESET_N: now also TP34.1, J5.1, J6.9, R50.1, U19.3 (~{RESET}); no longer R47.1, TP33.1
- net SPI0_CLK: now also R44.2, TP30.1, J6.1, U19.16 (CLK)
- net SPI0_CLK_F: now also R44.1
- net SPI0_CS0_N: now also R47.1, TP33.1, J6.7, U19.7 (~{CS}); no longer R44.1, TP32.1
- net SPI0_IO2: now also TP35.1, R48.1, U19.9 (IO2); no longer R45.1, TP34.1
- net SPI0_IO3: now also R49.1, TP36.1, U19.1 (IO3); no longer R46.1, TP35.1
- net SPI0_MISO: now also R46.1, TP32.1, J6.5, U19.8 (DO_IO1); no longer TP31.1
- net SPI0_MOSI: now also R45.1, TP31.1, J6.3, U19.15 (DI_IO0); no longer TP30.1
Other:
- moved on the sheet: R44, R45, R46, R47, TP30, TP31, TP32, TP33, TP34, TP35
