File: hardware/arc1-compact/R10_WORK/cad/d213.kicad_sch (KiCad schematic)
At the start: 55 parts, among them J5 D213 UART0, SW3 D213 RESET, SW4 D213 BOOT (PA0), U19 D213ECV, U20 D213 ctl OD, U21 W25Q512JVFIQ, Y2 24MHz +-20ppm

Commit message: R10 change order rev 1.1: HDMI audio (ADV7513), USB0 role mux + hub + 2x front USB-A, eMMC, buttonless board
Owner handoff ARC1_R10_Handoff rev 1.1 (spec/, SHA-256 recorded) implemented in the generated schematic:
- D8 ADV7513BSWZ replaces the TFP410 (supersedes D6): D213 RGB888 video, D213 I2C2 init,
  F133 I2S2 -> HDMI embedded audio; own 1.8 V buck + 3 filtered domains; R_EXT 887R.
  D[23:0] pin order verified from the datasheet glyph coordinates.
- D9 F133 USB0 -> TS3USB221A (default rear USB-C device/FEL) or USB2422 hub -> two
  TPS2051C-switched front USB-A ports; F133 USB1 remains the internal D213 link; the D213
  recovery USB-C becomes internal fixture pads.
- D10 Samsung KLMAG1JETD-B041 16 GB eMMC on F133 SMHC0 (CONDITIONAL: SMHC0 documented for SD).
- D11 no switches: fixture pad pairs; game buttons, microSD and speakers removed.
- crosscheck_r10 section I (handoff go/no-go: 4 exterior connectors, 0 switches, I2S wired
  to the HDMI transmitter, USB0/USB1 roles, eMMC wiring) PASS; ERC 0/0; pin review PASS.
Sources: ADV7513 DS Rev B (LCSC copy), ADI AN-1270, Linux adv7511 driver, USB2422
DS00001726A, TPS20xxC SLVSAU6I, Samsung eMMC DS (not committed: vendor-confidential mark).

Co-Authored-By: Claude Opus 5.5 <noreply@anthropic.com>
Claude-Session: https://claude.ai/code/session_01UkiuLdbjDvK75uDzAPKsGs
Parts:
- removed C72, C73, C74: 100nF, Capacitor_SMD:C_0402_1005Metric, symbol ARC1_R10:C0402
- removed J5: D213 UART0, Connector_PinHeader_2.54mm:PinHeader_1x03_P2.54mm_Vertical, symbol ARC1_R10:HDR_1x3
- removed R48: 0R, Resistor_SMD:R_0402_1005Metric, symbol ARC1_R10:R0402
- removed R49, R50: 100k, Resistor_SMD:R_0402_1005Metric, symbol ARC1_R10:R0402
- removed SW3: D213 RESET, Button_Switch_SMD:SW_SPST_B3U-1000P, symbol ARC1_R10:SW_B3U
- removed SW4: D213 BOOT (PA0), Button_Switch_SMD:SW_SPST_B3U-1000P, symbol ARC1_R10:SW_B3U
- removed TP36: D213_NOR_CLK, TestPoint:TestPoint_Pad_D1.0mm, symbol ARC1_R10:TP
- removed U19: D213ECV, ARC1_R10:ArtInChip_QFN-128-1EP_12.3x12.3mm_P0.35mm_EP7.0x7.0mm, symbol ARC1_R10:D213ECV
- added C101, C102, C103: 100nF, Capacitor_SMD:C_0402_1005Metric, symbol ARC1_R10:C0402
- added J7: D213 RESET pads, TestPoint:TestPoint_2Pads_Pitch2.54mm_Drill0.8mm, symbol ARC1_R10:PADS_1x2
- added J8: D213 BOOT pads (PA0), TestPoint:TestPoint_2Pads_Pitch2.54mm_Drill0.8mm, symbol ARC1_R10:PADS_1x2
- added J9: D213 UART0, Connector_PinHeader_2.54mm:PinHeader_1x03_P2.54mm_Vertical, symbol ARC1_R10:HDR_1x3
- added R59, R60: 10k, Resistor_SMD:R_0402_1005Metric, symbol ARC1_R10:R0402
- added R61: 1k, Resistor_SMD:R_0402_1005Metric, symbol ARC1_R10:R0402
- added TP43: D213_XI, TestPoint:TestPoint_Pad_D1.0mm, symbol ARC1_R10:TP
- added U22: W25Q512JVFIQ, Package_SO:SOIC-16W_7.5x10.3mm_P1.27mm, symbol ARC1_R10:W25Q512JVFIQ
- C100: value 100nF -> 12pF; LCSC C1525 -> C1547; MPN CL05B104KO5NNNC -> 0402CG120J500NT; Manufacturer Samsung -> FH
- C78, C79, C85, C86, C92: value 10uF -> 100nF; footprint Capacitor_SMD:C_0603_1608Metric -> Capacitor_SMD:C_0402_1005Metric; symbol ARC1_R10:C0603 -> ARC1_R10:C0402; LCSC C19702 -> C1525; MPN CL10A106KP8NNNC -> CL05B104KO5NNNC
- C81, C82, C88, C89: value 100nF -> 10uF; footprint Capacitor_SMD:C_0402_1005Metric -> Capacitor_SMD:C_0603_1608Metric; symbol ARC1_R10:C0402 -> ARC1_R10:C0603; LCSC C1525 -> C19702; MPN CL05B104KO5NNNC -> CL10A106KP8NNNC
- C93, C94: value 1uF -> 100nF; LCSC C52923 -> C1525; MPN CL05A105KA5NQNC -> CL05B104KO5NNNC
- C95: value 1uF -> 10uF; footprint Capacitor_SMD:C_0402_1005Metric -> Capacitor_SMD:C_0603_1608Metric; symbol ARC1_R10:C0402 -> ARC1_R10:C0603; LCSC C52923 -> C19702; MPN CL05A105KA5NQNC -> CL10A106KP8NNNC
- C96: value 12pF -> 1uF; LCSC C1547 -> C52923; MPN 0402CG120J500NT -> CL05A105KA5NQNC; Manufacturer FH -> Samsung; Note CL match to crystal -> (none)
- C97: value 12pF -> 1uF; LCSC C1547 -> C52923; MPN 0402CG120J500NT -> CL05A105KA5NQNC; Manufacturer FH -> Samsung
- C98: value 100nF -> 1uF; LCSC C1525 -> C52923; MPN CL05B104KO5NNNC -> CL05A105KA5NQNC
- C99: value 100nF -> 12pF; LCSC C1525 -> C1547; MPN CL05B104KO5NNNC -> 0402CG120J500NT; Manufacturer Samsung -> FH; Note optional delay cap (<= 4.7 uF allowed) -> CL match to crystal; now fitted
- R51: value 100R -> 0R; LCSC (none) -> C17168; MPN (none) -> 0402WGF0000TCE; Manufacturer (none) -> UNI-ROYAL; Note EOS series R on an exposed pin (HW guide 4.7 item 1) -> HW guide 2.2.2: series 0R on PLL_XO to tune drive; Reuse (none) -> SLIM4_R26_BOM_LINE (re-validate)
- R52: Note PA0 idles high: normal boot unless the F133 or the BOOT key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 -> inactive while F133 PD11 is hi-Z
- R53: value 22R -> 100k; LCSC C25092 -> C25741; MPN 0402WGF220JTCE -> 0402WGF1003TCE; Note source series termination -> inactive while F133 PD10 is hi-Z
- R54: value 10k -> 100R; LCSC C25744 -> (none); MPN 0402WGF1002TCE -> (none); Manufacturer UNI-ROYAL -> (none); Note HW guide 2.3.1: CS/WP/HOLD must be pulled up -> EOS series R on an exposed pin (HW guide 4.7 item 1); Reuse SLIM4_R26_BOM_LINE (re-validate) -> (none)
- R55: value 10k -> 100k; LCSC C25744 -> C25741; MPN 0402WGF1002TCE -> 0402WGF1003TCE; Note HW guide 2.3.1: CS/WP/HOLD must be pulled up -> PA0 idles high: normal boot unless the F133 or the BOOT key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
- R56: value 10k -> 22R; LCSC C25744 -> C25092; MPN 0402WGF1002TCE -> 0402WGF220JTCE; Note HW guide 2.3.1: CS/WP/HOLD must be pulled up -> source series termination
- R58: value 1k -> 10k; LCSC C11702 -> C25744; MPN 0402WGF1001TCE -> 0402WGF1002TCE; Note (none) -> HW guide 2.3.1: CS/WP/HOLD must be pulled up
- TP37: value D213_NOR_MOSI -> D213_NOR_CLK
- TP38: value D213_NOR_MISO -> D213_NOR_MOSI
- TP39: value D213_NOR_CS_N -> D213_NOR_MISO
- TP40: value D213_RESET_N -> D213_NOR_CS_N; Note (none) -> SOIC-16 clip / probe
- TP41: value D213_UART0_TX -> D213_RESET_N
- TP42: value D213_XI -> D213_UART0_TX
- U20: value D213 ctl OD -> D213ECV; footprint Package_TO_SOT_SMD:SOT-23-6 -> ARC1_R10:ArtInChip_QFN-128-1EP_12.3x12.3mm_P0.35mm_EP7.0x7.0mm; symbol ARC1_R10:LVC2G07 -> ARC1_R10:D213ECV; Footprint_status STD_LIB -> GENERATED_DERIVED; MPN SN74LVC2G07DBVR -> D213ECV; Manufacturer Texas Instruments -> ArtInChip; Note 1Y holds PA0 (boot/upgrade pin, also UART0_TX) low across a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 -> EPAD = GND, many vias (HW guide 3.1); Source TI SCES308L DBV pin functions (sources/ti) -> D21x HW guide V2.0 Table 2-5; D21x DS v1.4 Fig 5-6 (package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
- U21: value W25Q512JVFIQ -> D213 ctl OD; footprint Package_SO:SOIC-16W_7.5x10.3mm_P1.27mm -> Package_TO_SOT_SMD:SOT-23-6; symbol ARC1_R10:W25Q512JVFIQ -> ARC1_R10:LVC2G07; MPN W25Q512JVFIQ -> SN74LVC2G07DBVR; Manufacturer Winbond -> Texas Instruments; Note prototype bring-up/recovery boot flash (D5); same part as t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 -> 1Y holds PA0 (boot/upgrade pin, also UART0_TX) low across a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; Source W25Q512JV DS Rev.B Figure 1b (hardware/gen_flash_pinmux.py;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 -> TI SCES308L DBV pin functions (sources/ti)
Connections:
- net 1V2_D213: now also C80.1, C81.1, C82.1, U20.128 (VDD11_SYS), U20.31 (VDD11_SYS), U20.34 (VDD11_SYS), U20.44 (VDD11_SYS), U20.74 (VDD11_SYS), U20.75 (VDD11_SYS)
- net 1V5_D213: now also C87.1, C88.1, C89.1, U20.30 (VCC_DRAM), U20.32 (VCC_DRAM), U20.33 (VCC_DRAM), U20.35 (VCC_DRAM), U20.36 (VCC_DRAM); no longer C80.1, C81.1, C82.1
- net 3V3: now also C93.1, C94.1, C95.1, R53.2, R58.2, U20.114 (VCC33_IO1), U20.27 (VCC33_IO1), U20.41 (VCC33_IO0), U20.57 (VCC33_IO0), U20.83 (VCC33_IO0), U21.5 (VCC), C101.1, C103.1, R59.2, R60.2, U22.2 (VCC); no longer C100.1, C87.1, C88.1, C89.1, C98.1, R54.2, R56.2, U20.5 (VCC), U21.2 (VCC)
- net D213_BOOT_REQ_N: now also R52.1, U21.1 (1A); no longer U20.1 (1A)
- net D213_LDO1X: now also C96.1, U20.28 (LDO1x); no longer C93.1
- net D213_LDO25: now also C97.1, U20.29 (LDO25); no longer C94.1
- net D213_LED: now also U20.46 (PB7), R61.1; no longer R58.1
- net D213_LED_R: now also R61.2; no longer R58.2
- net D213_NOR_CLK: now also R56.2, TP37.1, U22.16 (CLK); no longer R53.2, U21.16 (CLK)
- net D213_NOR_CLK_D: now also R56.1, U20.43 (PB5); no longer R53.1
- net D213_NOR_CS_N: now also R57.1, TP40.1, U20.39 (PB2), U22.7 (~{CS}); no longer R54.1, TP39.1, U21.7 (~{CS})
- net D213_NOR_IO2: now also R58.1, U20.38 (PB1), U22.9 (IO2); no longer R55.1, U21.9 (IO2)
- net D213_NOR_IO3: now also U20.37 (PB0), R59.1, U22.1 (IO3); no longer R56.1, U21.1 (IO3)
- net D213_NOR_MISO: now also TP39.1, U20.40 (PB3), U22.8 (DO_IO1); no longer TP38.1, U21.8 (DO_IO1)
- net D213_NOR_MOSI: now also TP38.1, U20.42 (PB4), U22.15 (DI_IO0); no longer TP37.1, U21.15 (DI_IO0)
- net D213_NOR_RESET_N: now also R60.1, U22.3 (~{RESET}); no longer R57.1, U21.3 (~{RESET})
- net D213_RDY: now also U20.45 (PB6)
- net D213_RESET_N: now also TP41.1, U20.76 (RESETN), U21.4 (2Y), C102.1, J7.1; no longer C99.1, TP40.1, U20.4 (2Y)
- net D213_RESET_REQ_N: now also R53.1, U21.3 (2A); no longer U20.3 (2A)
- net D213_UART0_RX: now also R54.2, U20.86 (PA1); no longer R51.2
- net D213_UART0_RX_J: now also R54.1, J9.3; no longer R51.1
- net D213_UART0_TX: now also R55.1, TP42.1, U20.85 (PA0), U21.6 (1Y), J8.1, J9.2; no longer R52.1, TP41.1, U20.6 (1Y)
- net D213_USB0_DM: now also U20.79 (PU0)
- net D213_USB0_DP: now also U20.80 (PU1)
- net D213_VCC30: now also C98.1, U20.84 (VCC30_ANA); no longer C95.1
- net D213_XI: now also C99.1, U20.78 (PLL_XI), TP43.1; no longer C96.1, TP42.1
- net D213_XO: now also R51.1, U20.77 (PLL_XO)
- net D213_XO_X: now also C100.1, R51.2; no longer C97.1
- net FPGA45_DONE: now also U20.91 (PA6)
- net FPGA45_INITN: now also U20.90 (PA5)
- net FPGA45_MISO: now also U20.48 (PB9)
- net FPGA45_MOSI_D: now also U20.49 (PB10)
- net FPGA45_PROGRAMN_D: now also U20.89 (PA4)
- net FPGA45_PWR_EN_D: now also U20.87 (PA2)
- net FPGA45_SCK_D: now also U20.51 (PB11)
- net FPGA45_SS_N_D: now also U20.47 (PB8)
- net FPGA45_VCC_PG: now also U20.88 (PA3)
- net GND: now also U20.129 (GND), U21.2 (GND), C101.2, C102.2, C103.2, J7.2, J8.2, J9.1, U22.10 (GND); no longer U20.2 (GND), U21.10 (GND)
- net G_CLKIN: now also U20.55 (PE3)
- net G_RXCK: now also U20.67 (PE13)
- net G_RXCTL: now also U20.54 (PE2)
- net G_RXD0: now also U20.53 (PE1)
- net G_RXD1: now also U20.52 (PE0)
- net G_RXD2: now also U20.66 (PE12)
- net G_RXD3: now also U20.65 (PE11)
- net G_TXCK_D: now also U20.60 (PE6)
- net G_TXCTL_D: now also U20.61 (PE7)
- net G_TXD0_D: now also U20.59 (PE5)
- net G_TXD1_D: now also U20.58 (PE4)
- net G_TXD2_D: now also U20.69 (PE15)
- net G_TXD3_D: now also U20.68 (PE14)
- net HDMI_HPD: now also U20.95 (PA10)
- net LCD_D0: now also U20.18 (PD0)
- net LCD_D1: now also U20.17 (PD1)
- net LCD_D10: now also U20.8 (PD10)
- net LCD_D11: now also U20.7 (PD11)
- net LCD_D12: now also U20.6 (PD12)
- net LCD_D13: now also U20.5 (PD13)
- net LCD_D14: now also U20.4 (PD14)
- net LCD_D15: now also U20.3 (PD15)
- net LCD_D16: now also U20.2 (PD16)
- net LCD_D17: now also U20.1 (PD17)
- net LCD_D18: now also U20.127 (PD18)
- net LCD_D19: now also U20.126 (PD19)
- net LCD_D2: now also U20.16 (PD2)
- net LCD_D20: now also U20.125 (PD20)
- net LCD_D21: now also U20.124 (PD21)
- net LCD_D22: now also U20.123 (PD22)
- net LCD_D23: now also U20.122 (PD23)
- net LCD_D3: now also U20.15 (PD3)
- net LCD_D4: now also U20.14 (PD4)
- net LCD_D5: now also U20.13 (PD5)
- net LCD_D6: now also U20.12 (PD6)
- net LCD_D7: now also U20.11 (PD7)
- net LCD_D8: now also U20.10 (PD8)
- net LCD_D9: now also U20.9 (PD9)
- net LCD_DCLK_D: now also U20.121 (PD24)
- net LCD_DE_D: now also U20.118 (PD27)
- net LCD_HS_D: now also U20.120 (PD25)
- net LCD_VS_D: now also U20.119 (PD26)
- new net HDMI_I2C_SCL: U20.93 (PA8)
- new net HDMI_I2C_SDA: U20.94 (PA9)
- new net HDMI_INT: U20.92 (PA7)
- new net HDMI_PD: U20.96 (PA11)
Other:
- moved on the sheet: C100, C75, C76, C77, C78, C79, C80, C81, C82, C83, C84, C85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
