File: hardware/arc1-compact/R10_WORK/cad/power.kicad_sch (KiCad schematic)
At the start: 122 parts, among them J2 F45 power override, J3 F12 power override, SW1 F133 RESET, U10 D213_DRAM, U11 F45_VCC, U12 3V3_F45 switch, U13 2V5_F45, U14 F12_VCC, U15 3V3_F12 switch, U16 2V5_F12, U3 3V3, U4 TPS3808G33, U5 F133_CORE, U6 F133_DRAM, U7 1V8_AN, U8 TPS3808G09, U9 D213_CORE

Commit message: R10 change order rev 1.1: HDMI audio (ADV7513), USB0 role mux + hub + 2x front USB-A, eMMC, buttonless board
Owner handoff ARC1_R10_Handoff rev 1.1 (spec/, SHA-256 recorded) implemented in the generated schematic:
- D8 ADV7513BSWZ replaces the TFP410 (supersedes D6): D213 RGB888 video, D213 I2C2 init,
  F133 I2S2 -> HDMI embedded audio; own 1.8 V buck + 3 filtered domains; R_EXT 887R.
  D[23:0] pin order verified from the datasheet glyph coordinates.
- D9 F133 USB0 -> TS3USB221A (default rear USB-C device/FEL) or USB2422 hub -> two
  TPS2051C-switched front USB-A ports; F133 USB1 remains the internal D213 link; the D213
  recovery USB-C becomes internal fixture pads.
- D10 Samsung KLMAG1JETD-B041 16 GB eMMC on F133 SMHC0 (CONDITIONAL: SMHC0 documented for SD).
- D11 no switches: fixture pad pairs; game buttons, microSD and speakers removed.
- crosscheck_r10 section I (handoff go/no-go: 4 exterior connectors, 0 switches, I2S wired
  to the HDMI transmitter, USB0/USB1 roles, eMMC wiring) PASS; ERC 0/0; pin review PASS.
Sources: ADV7513 DS Rev B (LCSC copy), ADI AN-1270, Linux adv7511 driver, USB2422
DS00001726A, TPS20xxC SLVSAU6I, Samsung eMMC DS (not committed: vendor-confidential mark).

Co-Authored-By: Claude Opus 5.5 <noreply@anthropic.com>
Claude-Session: https://claude.ai/code/session_01UkiuLdbjDvK75uDzAPKsGs
Parts:
- removed SW1: F133 RESET, Button_Switch_SMD:SW_SPST_B3U-1000P, symbol ARC1_R10:SW_B3U
- added C41: 10uF, Capacitor_SMD:C_0603_1608Metric, symbol ARC1_R10:C0603
- added C42, C43: 1uF, Capacitor_SMD:C_0402_1005Metric, symbol ARC1_R10:C0402
- added J4: F12 power override, Connector_PinHeader_2.54mm:PinHeader_1x03_P2.54mm_Vertical, symbol ARC1_R10:HDR_1x3
- added L8: 2.2uH, ARC1_R10:SLIM4_FP_L2_ASWPA4035, symbol ARC1_R10:L4035
- added R39: 1k, Resistor_SMD:R_0402_1005Metric, symbol ARC1_R10:R0402
- added R40, R41: 100k, Resistor_SMD:R_0402_1005Metric, symbol ARC1_R10:R0402
- added TP26: GND, TestPoint:TestPoint_Pad_D1.0mm, symbol ARC1_R10:TP
- added U17: 2V5_F12, Package_TO_SOT_SMD:SOT-23-5, symbol ARC1_R10:TLV75525P
- C28, C36: value 1nF -> 10uF; footprint Capacitor_SMD:C_0402_1005Metric -> Capacitor_SMD:C_0805_2012Metric; symbol ARC1_R10:C0402 -> ARC1_R10:C0805; LCSC (none) -> C15850; MPN (none) -> CL21A106KAYNNNE; Manufacturer (none) -> Samsung; Reuse (none) -> SLIM4_R26_BOM_LINE (re-validate)
- C29, C37: value 1uF -> 22uF; footprint Capacitor_SMD:C_0402_1005Metric -> Capacitor_SMD:C_0805_2012Metric; symbol ARC1_R10:C0402 -> ARC1_R10:C0805; LCSC C52923 -> C5674; MPN CL05A105KA5NQNC -> CL21A226MQQNNNE
- C30, C38: value 10uF -> 22uF; footprint Capacitor_SMD:C_0603_1608Metric -> Capacitor_SMD:C_0805_2012Metric; symbol ARC1_R10:C0603 -> ARC1_R10:C0805; LCSC C19702 -> C5674; MPN CL10A106KP8NNNC -> CL21A226MQQNNNE
- C31, C39: value 1uF -> 1nF; LCSC C52923 -> (none); MPN CL05A105KA5NQNC -> (none); Manufacturer Samsung -> (none); Reuse SLIM4_R26_BOM_LINE (re-validate) -> (none)
- C33: footprint Capacitor_SMD:C_0805_2012Metric -> Capacitor_SMD:C_0603_1608Metric; symbol ARC1_R10:C0805 -> ARC1_R10:C0603; LCSC C15850 -> C19702; MPN CL21A106KAYNNNE -> CL10A106KP8NNNC
- C34, C35: value 22uF -> 1uF; footprint Capacitor_SMD:C_0805_2012Metric -> Capacitor_SMD:C_0402_1005Metric; symbol ARC1_R10:C0805 -> ARC1_R10:C0402; LCSC C5674 -> C52923; MPN CL21A226MQQNNNE -> CL05A105KA5NQNC
- J2: value F45 power override -> F133 RESET pads; footprint Connector_PinHeader_2.54mm:PinHeader_1x03_P2.54mm_Vertical -> TestPoint:TestPoint_2Pads_Pitch2.54mm_Drill0.8mm; symbol ARC1_R10:HDR_1x3 -> ARC1_R10:PADS_1x2; MPN header 1x3 2.54 (DNP-able) -> internal service pad pair; Note JTAG service without firmware: jumper 1-2 powers the FPGA r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 -> internal fixture pads (handoff: no exterior controls); soft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; now not fitted
- J3: value F12 power override -> F45 power override; Note JTAG service without firmware: jumper 1-2 powers the FPGA r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 -> internal fixture: JTAG service without firmware, jumper 1-2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; now not fitted
- R27: value 82.5k -> 200k
- R30: value 1k -> 82.5k; LCSC C11702 -> (none); MPN 0402WGF1001TCE -> (none); Manufacturer UNI-ROYAL -> (none); Note D213 PA2 drive; jumper override below -> 1 % E96; Reuse SLIM4_R26_BOM_LINE (re-validate) -> (none)
- R31, R37: Note FPGA unpowered until its owner enables it -> 1 %
- R32, R38: value 100k -> 0R; footprint Resistor_SMD:R_0402_1005Metric -> Resistor_SMD:R_0603_1608Metric; symbol ARC1_R10:R0402 -> ARC1_R10:R0603; LCSC C25741 -> (none); MPN 0402WGF1003TCE -> (none); Manufacturer UNI-ROYAL -> (none); Note PG pulled to the switched VCCIO rail: high only with VCC an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 -> staged power-on link / current measurement; Reuse SLIM4_R26_BOM_LINE (re-validate) -> (none)
- R33: value 82.5k -> 1k; LCSC (none) -> C11702; MPN (none) -> 0402WGF1001TCE; Manufacturer (none) -> UNI-ROYAL; Note 1 % E96 -> D213 PA2 drive; jumper override below; Reuse (none) -> SLIM4_R26_BOM_LINE (re-validate)
- R34: Note 1 % -> FPGA unpowered until its owner enables it
- R35: value 0R -> 100k; footprint Resistor_SMD:R_0603_1608Metric -> Resistor_SMD:R_0402_1005Metric; symbol ARC1_R10:R0603 -> ARC1_R10:R0402; LCSC (none) -> C25741; MPN (none) -> 0402WGF1003TCE; Manufacturer (none) -> UNI-ROYAL; Note staged power-on link / current measurement -> PG pulled to the switched VCCIO rail: high only with VCC an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; Reuse (none) -> SLIM4_R26_BOM_LINE (re-validate)
- R36: value 1k -> 82.5k; LCSC C11702 -> (none); MPN 0402WGF1001TCE -> (none); Manufacturer UNI-ROYAL -> (none); Note F133 PE0 drive; jumper override below -> 1 % E96; Reuse SLIM4_R26_BOM_LINE (re-validate) -> (none)
- TP12: value 1V1_F45 -> 1V8_HDMI
- TP13: value 3V3_F45 -> 1V1_F45
- TP14: value 2V5_F45 -> 3V3_F45
- TP15: value FPGA45_VCC_PG -> 2V5_F45
- TP16: value FPGA45_PWR_EN -> FPGA45_VCC_PG
- TP17: value 1V1_F12 -> FPGA45_PWR_EN
- TP18: value 3V3_F12 -> 1V1_F12
- TP19: value 2V5_F12 -> 3V3_F12
- TP20: value FPGA12_VCC_PG -> 2V5_F12
- TP21: value FPGA12_PWR_EN -> FPGA12_VCC_PG
- TP22: value GND -> FPGA12_PWR_EN
- U11: value F45_VCC -> HDMI_1V8; footprint Package_TO_SOT_SMD:SOT-23-6 -> Package_TO_SOT_SMD:SOT-23-5; symbol ARC1_R10:TLV62569P -> ARC1_R10:TLV62569; Evidence VERIFIED_BY_VENDOR_DOC (DDC is a thin SOT-23-6: confirm lan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 -> VERIFIED_BY_VENDOR_DOC; LCSC (none) -> C141836; MPN TLV62569PDDCR -> TLV62569DBVR; Note 0.6*(1+82.5k/100k)=1.095 V (ECP5 VCC 1.045/1.10/1.155) -> 0.6*(1+200k/100k)=1.80 V ADV7513 DVDD/AVDD/PVDD/BGVDD (1.71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
- U12: value 3V3_F45 switch -> F45_VCC; symbol ARC1_R10:TPS22918 -> ARC1_R10:TLV62569P; Evidence VERIFIED_BY_VENDOR_DOC -> VERIFIED_BY_VENDOR_DOC (DDC is a thin SOT-23-6: confirm lan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; MPN TPS22918DBVR -> TLV62569PDDCR; Note VCCIO with VCC (TN-02038 s.4); 1 nF CT -> ~1.9 ms ramp -> 0.6*(1+82.5k/100k)=1.095 V (ECP5 VCC 1.045/1.10/1.155); Source TPS22918 DS s.5 (sources/glue) -> TLV62569 DS s.5 (sources/glue)
- U13: value 2V5_F45 -> 3V3_F45 switch; footprint Package_TO_SOT_SMD:SOT-23-5 -> Package_TO_SOT_SMD:SOT-23-6; symbol ARC1_R10:TLV75525P -> ARC1_R10:TPS22918; Evidence CANDIDATE (pinout per TLV755P family DS; 2.5 V option order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 -> VERIFIED_BY_VENDOR_DOC; MPN TLV75525PDBVR -> TPS22918DBVR; Note ECP5 VCCAUX 2.375-2.625 V -> VCCIO with VCC (TN-02038 s.4); 1 nF CT -> ~1.9 ms ramp; Source TLV755P DS Table 4-1 (same DBV pinout for all fixed voltage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 -> TPS22918 DS s.5 (sources/glue)
- U14: value F12_VCC -> 2V5_F45; footprint Package_TO_SOT_SMD:SOT-23-6 -> Package_TO_SOT_SMD:SOT-23-5; symbol ARC1_R10:TLV62569P -> ARC1_R10:TLV75525P; Evidence VERIFIED_BY_VENDOR_DOC (DDC is a thin SOT-23-6: confirm lan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 -> CANDIDATE (pinout per TLV755P family DS; 2.5 V option order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; MPN TLV62569PDDCR -> TLV75525PDBVR; Note 0.6*(1+82.5k/100k)=1.095 V (ECP5 VCC 1.045/1.10/1.155) -> ECP5 VCCAUX 2.375-2.625 V; Source TLV62569 DS s.5 (sources/glue) -> TLV755P DS Table 4-1 (same DBV pinout for all fixed voltage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
- U15: value 3V3_F12 switch -> F12_VCC; symbol ARC1_R10:TPS22918 -> ARC1_R10:TLV62569P; Evidence VERIFIED_BY_VENDOR_DOC -> VERIFIED_BY_VENDOR_DOC (DDC is a thin SOT-23-6: confirm lan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; MPN TPS22918DBVR -> TLV62569PDDCR; Note VCCIO with VCC (TN-02038 s.4); 1 nF CT -> ~1.9 ms ramp -> 0.6*(1+82.5k/100k)=1.095 V (ECP5 VCC 1.045/1.10/1.155); Source TPS22918 DS s.5 (sources/glue) -> TLV62569 DS s.5 (sources/glue)
- U16: value 2V5_F12 -> 3V3_F12 switch; footprint Package_TO_SOT_SMD:SOT-23-5 -> Package_TO_SOT_SMD:SOT-23-6; symbol ARC1_R10:TLV75525P -> ARC1_R10:TPS22918; Evidence CANDIDATE (pinout per TLV755P family DS; 2.5 V option order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 -> VERIFIED_BY_VENDOR_DOC; MPN TLV75525PDBVR -> TPS22918DBVR; Note ECP5 VCCAUX 2.375-2.625 V -> VCCIO with VCC (TN-02038 s.4); 1 nF CT -> ~1.9 ms ramp; Source TLV755P DS Table 4-1 (same DBV pinout for all fixed voltage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 -> TPS22918 DS s.5 (sources/glue)
Connections:
- net 1V1_F12: now also R38.2, TP18.1; no longer R35.2, TP17.1
- net 1V1_F12_REG: now also C37.1, C38.1, R36.1, R38.1, L8.2; no longer C34.1, C35.1, L7.2, R33.1, R35.1
- net 1V1_F45: now also R32.2, TP13.1; no longer R29.2, TP12.1
- net 1V1_F45_REG: now also C29.1, C30.1, L7.2, R30.1, R32.1; no longer C26.1, C27.1, L6.2, R27.1, R29.1
- net 2V5_F12: now also TP20.1; no longer TP19.1
- net 2V5_F12_REG: now also C43.1, U17.5 (OUT); no longer C40.1, U16.5 (OUT)
- net 2V5_F45: now also TP15.1; no longer TP14.1
- net 2V5_F45_REG: now also C35.1, U14.5 (OUT); no longer C32.1, U13.5 (OUT)
- net 3V3: now also C32.1, C40.1, U13.1 (VIN), U16.1 (VIN), J4.1; no longer C29.1, C37.1, J2.1, U12.1 (VIN), U15.1 (VIN)
- net 3V3_F12: now also TP19.1, U16.5 (QOD), U16.6 (VOUT), C41.1, C42.1, R41.2, U17.1 (IN), U17.3 (EN); no longer C38.1, C39.1, R38.2, TP18.1, U15.5 (QOD), U15.6 (VOUT), U16.1 (IN), U16.3 (EN)
- net 3V3_F45: now also C33.1, C34.1, R35.2, TP14.1, U13.5 (QOD), U13.6 (VOUT), U14.1 (IN), U14.3 (EN); no longer C30.1, C31.1, R32.2, TP13.1, U12.5 (QOD), U12.6 (VOUT), U13.1 (IN), U13.3 (EN)
- net FB_F12_VCC: now also R36.2, R37.1, U15.6 (FB); no longer R33.2, R34.1, U14.6 (FB)
- net FB_F45_VCC: now also R30.2, R31.1, U12.6 (FB); no longer R27.2, R28.1, U11.6 (FB)
- net FPGA12_PWR_EN: now also TP22.1, U15.1 (EN), U16.3 (ON), J4.2, R39.2, R40.1; no longer J3.2, R36.2, R37.1, TP21.1, U14.1 (EN), U15.3 (ON)
- net FPGA12_PWR_EN_F: now also R39.1; no longer R36.1
- net FPGA12_VCC_PG: now also TP21.1, U15.5 (PG), R41.1; no longer R38.1, TP20.1, U14.5 (PG)
- net FPGA45_PWR_EN: now also J3.2, R33.2, R34.1, TP17.1, U12.1 (EN), U13.3 (ON); no longer J2.2, R30.2, R31.1, TP16.1, U11.1 (EN), U12.3 (ON)
- net FPGA45_PWR_EN_D: now also R33.1; no longer R30.1
- net FPGA45_VCC_PG: now also R35.1, TP16.1, U12.5 (PG); no longer R32.1, TP15.1, U11.5 (PG)
- net GND: now also J2.2, C41.2, C42.2, C43.2, J4.3, R40.2, TP26.1, U17.2 (GND); no longer J2.3, TP22.1
- net PG_3V3: now also U11.1 (EN)
- net RST_BTN_N: now also J2.1
- net SW_F12_CT: now also C39.1, U16.4 (CT); no longer C36.1, U15.4 (CT)
- net SW_F12_VCC: now also U15.3 (SW), L8.1; no longer L7.1, U14.3 (SW)
- net SW_F45_CT: now also C31.1, U13.4 (CT); no longer C28.1, U12.4 (CT)
- net SW_F45_VCC: now also L7.1, U12.3 (SW); no longer L6.1, U11.3 (SW)
- net VBUS_5V: now also C28.1, C36.1, U12.4 (VIN), U15.4 (VIN); no longer C33.1, U14.4 (VIN)
- new net 1V8_HDMI: R29.2, TP12.1
- new net 1V8_HDMI_REG: C26.1, C27.1, L6.2, R27.1, R29.1
- new net FB_HDMI_1V8: R27.2, R28.1, U11.5 (FB)
- new net SW_HDMI_1V8: L6.1, U11.3 (SW)
Other:
- moved on the sheet: C10, C11, C12, C13, C14, C15, C16, C17, C18, C19, C20, C21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
