File: hardware/arc1-compact/R10_WORK/cad/usb_link.kicad_sch (KiCad schematic)
At the start: 14 parts, among them J6 USB path select, J7 recovery USB-C, U22 TS3USB221A, U23 TPD2EUSB30

Commit message: R10 change order rev 1.1: HDMI audio (ADV7513), USB0 role mux + hub + 2x front USB-A, eMMC, buttonless board
Owner handoff ARC1_R10_Handoff rev 1.1 (spec/, SHA-256 recorded) implemented in the generated schematic:
- D8 ADV7513BSWZ replaces the TFP410 (supersedes D6): D213 RGB888 video, D213 I2C2 init,
  F133 I2S2 -> HDMI embedded audio; own 1.8 V buck + 3 filtered domains; R_EXT 887R.
  D[23:0] pin order verified from the datasheet glyph coordinates.
- D9 F133 USB0 -> TS3USB221A (default rear USB-C device/FEL) or USB2422 hub -> two
  TPS2051C-switched front USB-A ports; F133 USB1 remains the internal D213 link; the D213
  recovery USB-C becomes internal fixture pads.
- D10 Samsung KLMAG1JETD-B041 16 GB eMMC on F133 SMHC0 (CONDITIONAL: SMHC0 documented for SD).
- D11 no switches: fixture pad pairs; game buttons, microSD and speakers removed.
- crosscheck_r10 section I (handoff go/no-go: 4 exterior connectors, 0 switches, I2S wired
  to the HDMI transmitter, USB0/USB1 roles, eMMC wiring) PASS; ERC 0/0; pin review PASS.
Sources: ADV7513 DS Rev B (LCSC copy), ADI AN-1270, Linux adv7511 driver, USB2422
DS00001726A, TPS20xxC SLVSAU6I, Samsung eMMC DS (not committed: vendor-confidential mark).

Co-Authored-By: Claude Opus 5.5 <noreply@anthropic.com>
Claude-Session: https://claude.ai/code/session_01UkiuLdbjDvK75uDzAPKsGs
Parts:
- removed C101: 100nF, Capacitor_SMD:C_0402_1005Metric, symbol ARC1_R10:C0402
- removed D3: SMF5.0A, Diode_SMD:D_SMF, symbol ARC1_R10:TVS_SMF
- removed J6: USB path select, Connector_PinHeader_2.54mm:PinHeader_1x03_P2.54mm_Vertical, symbol ARC1_R10:HDR_1x3
- removed J7: recovery USB-C, Connector_USB:USB_C_Receptacle_GCT_USB4105-xx-A_16P_TopMnt_Horizontal, symbol ARC1_R10:USB_C
- removed R59, R60: 10k, Resistor_SMD:R_0402_1005Metric, symbol ARC1_R10:R0402
- removed R61: 5.1k, Resistor_SMD:R_0402_1005Metric, symbol ARC1_R10:R0402
- removed TP43: REC_VBUS, TestPoint:TestPoint_Pad_D1.0mm, symbol ARC1_R10:TP
- removed U22: TS3USB221A, Package_DFN_QFN:Texas_UQFN-10_1.5x2mm_P0.5mm, symbol ARC1_R10:TS3USB221A
- added C104: 100nF, Capacitor_SMD:C_0402_1005Metric, symbol ARC1_R10:C0402
- added J10: D213 USB path select, Connector_PinHeader_2.54mm:PinHeader_1x03_P2.54mm_Vertical, symbol ARC1_R10:HDR_1x3
- added J11: D213 recovery USB pads, Connector_PinHeader_2.54mm:PinHeader_1x04_P2.54mm_Vertical, symbol ARC1_R10:PADS_1x4
- added U24: TPD2EUSB30, ARC1_R10:SLIM4_FP_U11_TPD2EUSB30_DRT3, symbol ARC1_R10:TPD2EUSB30
- R62: value 5.1k -> 10k; LCSC (none) -> C25744; MPN (none) -> 0402WGF1002TCE; Manufacturer (none) -> UNI-ROYAL; Note (none) -> default: internal host link; Reuse (none) -> SLIM4_R26_BOM_LINE (re-validate)
- R63: value 100k -> 10k; LCSC C25741 -> C25744; MPN 0402WGF1003TCE -> 0402WGF1002TCE; Note defined level; VBUS only to a test point -> mux enabled
- U23: value TPD2EUSB30 -> TS3USB221A; footprint ARC1_R10:SLIM4_FP_U11_TPD2EUSB30_DRT3 -> Package_DFN_QFN:Texas_UQFN-10_1.5x2mm_P0.5mm; symbol ARC1_R10:TPD2EUSB30 -> ARC1_R10:TS3USB221A; Footprint_status SLIM4_CANDIDATE -> STD_LIB; LCSC C97502 -> (none); MPN TPD2EUSB30DRTR -> TS3USB221ARSER; Note (none) -> S=L (default): D213 USB0 <-> F133 USB1 host. S=H (internal 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; Source TPD2EUSB30 DS Table 5-1 (sources/glue) -> TI SCDS277C Table 4-1 / 7-1 (sources/ti)
Connections:
- net REC_CC2 is gone; now on net USBMUX_SEL: R62.1
- net REC_VBUS is gone; now on net USBMUX_OE_N: R63.1
- net 3V3: now also U23.10 (VCC), C104.1, J10.1
- net D213_USB0_DM: now also U23.7 (D-)
- net D213_USB0_DP: now also U23.8 (D+)
- net F133_USB1_DM: now also U23.2 (1D-)
- net F133_USB1_DP: now also U23.1 (1D+)
- net GND: now also U23.5 (GND), C104.2, J10.3, J11.1, J11.4, U24.3 (GND); no longer U23.3 (GND)
- net REC_USB_DM: now also U23.4 (2D-), J11.2, U24.2 (D-); no longer U23.2 (D-)
- net REC_USB_DP: now also U23.3 (2D+), J11.3, U24.1 (D+); no longer U23.1 (D+)
- net USBMUX_OE_N: now also U23.6 (~{OE})
- net USBMUX_SEL: now also U23.9 (S), J10.2
- no-connect marks 2 -> 0
Other:
- note added: "Internal: F133 USB1 host -> D213 USB0 device; service mux to internal D213 recovery pads Sheet generated from design.py; global labels carry every net."
- note removed: "F133 USB1 host -> D213 USB0 device; power-off service mux to recovery USB-C Sheet generated from design.py; global labels carry every net."
- title: ARC-1 Compact R10: F133 USB1 host -> D213 USB0 device; power-off service mux to recovery USB-C -> ARC-1 Compact R10: Internal: F133 USB1 host -> D213 USB0 device; service mux to internal D213 recovery pads
- moved on the sheet: R62, R63, TP44, TP45
