File: hardware/arc1-compact/R10_WORK/cad/ARC1_R10.kicad_sch (KiCad schematic)
At the start: 0 parts

Commit message: R10 change order rev 1.1: HDMI audio (ADV7513), USB0 role mux + hub + 2x front USB-A, eMMC, buttonless board
Owner handoff ARC1_R10_Handoff rev 1.1 (spec/, SHA-256 recorded) implemented in the generated schematic:
- D8 ADV7513BSWZ replaces the TFP410 (supersedes D6): D213 RGB888 video, D213 I2C2 init,
  F133 I2S2 -> HDMI embedded audio; own 1.8 V buck + 3 filtered domains; R_EXT 887R.
  D[23:0] pin order verified from the datasheet glyph coordinates.
- D9 F133 USB0 -> TS3USB221A (default rear USB-C device/FEL) or USB2422 hub -> two
  TPS2051C-switched front USB-A ports; F133 USB1 remains the internal D213 link; the D213
  recovery USB-C becomes internal fixture pads.
- D10 Samsung KLMAG1JETD-B041 16 GB eMMC on F133 SMHC0 (CONDITIONAL: SMHC0 documented for SD).
- D11 no switches: fixture pad pairs; game buttons, microSD and speakers removed.
- crosscheck_r10 section I (handoff go/no-go: 4 exterior connectors, 0 switches, I2S wired
  to the HDMI transmitter, USB0/USB1 roles, eMMC wiring) PASS; ERC 0/0; pin review PASS.
Sources: ADV7513 DS Rev B (LCSC copy), ADI AN-1270, Linux adv7511 driver, USB2422
DS00001726A, TPS20xxC SLVSAU6I, Samsung eMMC DS (not committed: vendor-confidential mark).

Co-Authored-By: Claude Opus 5.5 <noreply@anthropic.com>
Claude-Session: https://claude.ai/code/session_01UkiuLdbjDvK75uDzAPKsGs
Other:
- removed sheet controls
- removed sheet sd_audio
- added sheet debug (debug.kicad_sch)
- added sheet emmc (emmc.kicad_sch)
- added sheet usb_host (usb_host.kicad_sch)
- note added: "16 GB eMMC on F133 SMHC0 (4-bit, 3.3 V): installed games and saves"
- note added: "D213 RGB888 + F133 I2S -> ADV7513 HDMI transmitter (embedded audio) -> TPD12S016 -> HDMI-A"
- note added: "F133 USB0 role mux: rear USB-C (device/FEL, default) or USB2422 hub -> front USB-A Player 1 / Player 2"
- note added: "Internal: F133 USB1 host -> D213 USB0 device; service mux to internal D213 recovery pads"
- note added: "Internal: status LEDs, F133 UART0 fixture header"
- note added: "Rear USB-C: power input + F133 USB0 device/recovery path (via the USB0 role mux)"
- note removed: "D213 RGB888 -> TFP410 (DVI, strap mode) -> TPD12S016 -> HDMI type-A"
- note removed: "F133 USB1 host -> D213 USB0 device; power-off service mux to recovery USB-C"
- note removed: "Game buttons, LEDs, F133 debug UART"
- note removed: "USB-C sink, VBUS protection, F133 USB0 device / FEL"
- note removed: "microSD game media (not boot), 2x MAX98357A I2S speakers"

Commit message: R10 D12: top USB-A game cartridge, no eMMC; USB2514B 4-port hub (3 ports used)
Owner direction: games are played directly from a USB drive in a top USB-A "cartridge"
port; the two front USB-A ports are controller inputs; eMMC not needed.
- Schematic: eMMC sheet removed (F133 PF0-PF6 freed); USB2422 replaced by USB2514B-I/M2
  (strap mode CFG_SEL=00, port 4 disabled by strap, CRFILT/PLLFILT 0.1 uF per DS00001692C);
  third TPS2051C + ESD + TVS + vertical USB-A (Molex 105057) marked TOP.
- crosscheck I: five exterior connectors (rear USB-C + HDMI, 2x front USB-A, top USB-A),
  eMMC/USB2422 must be absent, all three ports on the hub. PASS. ERC 0/0, pin review and
  pin/function matrix PASS, R10_HOST_CHECKS_PASS.
- PCB regenerated: Ø 119.8 mm, DRC 0 errors (unrouted), top cartridge at (-9.3, 24.2) mm.
- DECISIONS D12 (supersedes D10 and the four-connector rule); change-order report sections
  1, 2, 4, 5, 6 and the mechanical note updated; CLAUDE.md topology line amended.

Co-Authored-By: Claude Opus 5.5 <noreply@anthropic.com>
Claude-Session: https://claude.ai/code/session_01UkiuLdbjDvK75uDzAPKsGs
Other:
- removed sheet emmc
- note added: "F133 USB0 role mux: rear USB-C (device/FEL, default) or USB2514B hub -> 2x front USB-A + top cartridge USB-A"
- note removed: "16 GB eMMC on F133 SMHC0 (4-bit, 3.3 V): installed games and saves"
- note removed: "F133 USB0 role mux: rear USB-C (device/FEL, default) or USB2422 hub -> front USB-A Player 1 / Player 2"
Changed lines of the file:
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@@
 (text "Internal: F133 USB1 host -> D213 USB0 device; service mux to internal D213 recovery pads" (exclude_from_sim no) (at 105.4 203.04 0) (effects (font (size 2 2)) (justify left)))
 (sheet (at 25.4 223.52) (size 76.2 20.32) (fields_autoplaced yes) (stroke (width 0.1524) (type solid)) (fill (color 0 0 0 0.0000)) (property "Sheetname" "usb_host" (at 25.4 222.8088 0) (effects (font (size 1.27 1.27)) (justify left bottom))) (property "Sheetfile" "usb_host.kicad_sch" (at 25.4 244.3988 0) (effects (font (size 1.27 1.27)) (justify left top))) (instances (project "ARC1_R10" (path "/08113eda-8d75-5ca0-b1cc-74f429d396dc" (page "8")))))
-(text "F133 USB0 role mux: rear USB-C (device/FEL, default) or USB2422 hub -> front USB-A Player 1 / Player 2" (exclude_from_sim no) (at 105.4 233.52 0) (effects (font (size 2 2)) (justify left)))
+(text "F133 USB0 role mux: rear USB-C (device/FEL, default) or USB2514B hub -> 2x front USB-A + top cartridge USB-A" (exclude_from_sim no) (at 105.4 233.52 0) (effects (font (size 2 2)) (justify left)))
 (sheet (at 225.4 40.64) (size 76.2 20.32) (fields_autoplaced yes) (stroke (width 0.1524) (type solid)) (fill (color 0 0 0 0.0000)) (property "Sheetname" "video" (at 225.4 39.9288 0) (effects (font (size 1.27 1.27)) (justify left bottom))) (property "Sheetfile" "video.kicad_sch" (at 225.4 61.5188 0) (effects (font (size 1.27 1.27)) (justify left top))) (instances (project "ARC1_R10" (path "/08113eda-8d75-5ca0-b1cc-74f429d396dc" (page "9")))))
 (text "D213 RGB888 + F133 I2S -> ADV7513 HDMI transmitter (embedded audio) -> TPD12S016 -> HDMI-A" (exclude_from_sim no) (at 305.4 50.64 0) (effects (font (size 2 2)) (justify left)))
@@
 (sheet (at 225.4 162.56) (size 76.2 20.32) (fields_autoplaced yes) (stroke (width 0.1524) (type solid)) (fill (color 0 0 0 0.0000)) (property "Sheetname" "psram12" (at 225.4 161.8488 0) (effects (font (size 1.27 1.27)) (justify left bottom))) (property "Sheetfile" "psram12.kicad_sch" (at 225.4 183.4388 0) (effects (font (size 1.27 1.27)) (justify left top))) (instances (project "ARC1_R10" (path "/08113eda-8d75-5ca0-b1cc-74f429d396dc" (page "13")))))
 (text "APS3204L 4 MiB QSPI PSRAM on the 12F (3V3_F12)" (exclude_from_sim no) (at 305.4 172.56 0) (effects (font (size 2 2)) (justify left)))
-(sheet (at 225.4 193.04) (size 76.2 20.32) (fields_autoplaced yes) (stroke (width 0.1524) (type solid)) (fill (color 0 0 0 0.0000)) (property "Sheetname" "emmc" (at 225.4 192.3288 0) (effects (font (size 1.27 1.27)) (justify left bottom))) (property "Sheetfile" "emmc.kicad_sch" (at 225.4 213.9188 0) (effects (font (size 1.27 1.27)) (justify left top))) (instances (project "ARC1_R10" (path "/08113eda-8d75-5ca0-b1cc-74f429d396dc" (page "14")))))
-(text "16 GB eMMC on F133 SMHC0 (4-bit, 3.3 V): installed games and saves" (exclude_from_sim no) (at 305.4 203.04 0) (effects (font (size 2 2)) (justify left)))
-(sheet (at 225.4 223.52) (size 76.2 20.32) (fields_autoplaced yes) (stroke (width 0.1524) (type solid)) (fill (color 0 0 0 0.0000)) (property "Sheetname" "debug" (at 225.4 222.8088 0) (effects (font (size 1.27 1.27)) (justify left bottom))) (property "Sheetfile" "debug.kicad_sch" (at 225.4 244.3988 0) (effects (font (size 1.27 1.27)) (justify left top))) (instances (project "ARC1_R10" (path "/08113eda-8d75-5ca0-b1cc-74f429d396dc" (page "15")))))
-(text "Internal: status LEDs, F133 UART0 fixture header" (exclude_from_sim no) (at 305.4 233.52 0) (effects (font (size 2 2)) (justify left)))
+(sheet (at 225.4 193.04) (size 76.2 20.32) (fields_autoplaced yes) (stroke (width 0.1524) (type solid)) (fill (color 0 0 0 0.0000)) (property "Sheetname" "debug" (at 225.4 192.3288 0) (effects (font (size 1.27 1.27)) (justify left bottom))) (property "Sheetfile" "debug.kicad_sch" (at 225.4 213.9188 0) (effects (font (size 1.27 1.27)) (justify left top))) (instances (project "ARC1_R10" (path "/08113eda-8d75-5ca0-b1cc-74f429d396dc" (page "14")))))
+(text "Internal: status LEDs, F133 UART0 fixture header" (exclude_from_sim no) (at 305.4 203.04 0) (effects (font (size 2 2)) (justify left)))
 (sheet_instances (path "/" (page "1")))
 )
