File: hardware/arc1-compact/R10_WORK/cad/debug.kicad_sch (KiCad schematic)
At the start: 7 parts, among them J17 F133 UART0

Commit message: R10 D12: top USB-A game cartridge, no eMMC; USB2514B 4-port hub (3 ports used)
Owner direction: games are played directly from a USB drive in a top USB-A "cartridge"
port; the two front USB-A ports are controller inputs; eMMC not needed.
- Schematic: eMMC sheet removed (F133 PF0-PF6 freed); USB2422 replaced by USB2514B-I/M2
  (strap mode CFG_SEL=00, port 4 disabled by strap, CRFILT/PLLFILT 0.1 uF per DS00001692C);
  third TPS2051C + ESD + TVS + vertical USB-A (Molex 105057) marked TOP.
- crosscheck I: five exterior connectors (rear USB-C + HDMI, 2x front USB-A, top USB-A),
  eMMC/USB2422 must be absent, all three ports on the hub. PASS. ERC 0/0, pin review and
  pin/function matrix PASS, R10_HOST_CHECKS_PASS.
- PCB regenerated: Ø 119.8 mm, DRC 0 errors (unrouted), top cartridge at (-9.3, 24.2) mm.
- DECISIONS D12 (supersedes D10 and the four-connector rule); change-order report sections
  1, 2, 4, 5, 6 and the mechanical note updated; CLAUDE.md topology line amended.

Co-Authored-By: Claude Opus 5.5 <noreply@anthropic.com>
Claude-Session: https://claude.ai/code/session_01UkiuLdbjDvK75uDzAPKsGs
Parts:
- removed D7: STATUS, LED_SMD:LED_0603_1608Metric, symbol ARC1_R10:LED
- removed J17: F133 UART0, Connector_PinHeader_2.54mm:PinHeader_1x03_P2.54mm_Vertical, symbol ARC1_R10:HDR_1x3
- removed R179: 1k, Resistor_SMD:R_0402_1005Metric, symbol ARC1_R10:R0402
- removed R180: 2k, Resistor_SMD:R_0402_1005Metric, symbol ARC1_R10:R0402
- added D10: 3V3, LED_SMD:LED_0603_1608Metric, symbol ARC1_R10:LED
- added J18: F133 UART0, Connector_PinHeader_2.54mm:PinHeader_1x03_P2.54mm_Vertical, symbol ARC1_R10:HDR_1x3
- added R176, R177: 1k, Resistor_SMD:R_0402_1005Metric, symbol ARC1_R10:R0402
- D8: value ERROR -> STATUS
- D9: value 3V3 -> ERROR
- R178: value 1k -> 2k; LCSC C11702 -> (none); MPN 0402WGF1001TCE -> (none); Manufacturer UNI-ROYAL -> (none); Reuse SLIM4_R26_BOM_LINE (re-validate) -> (none)
Connections:
- net 3V3: now also R178.1
- net GND: now also D10.1 (K), J18.1
- net LED_3V3_R: now also R178.2, D10.2 (A); no longer D9.2 (A)
- net LED_ERROR: now also R177.1
- net LED_ERROR_R: now also D9.2 (A), R177.2; no longer D8.2 (A)
- net LED_STATUS: now also R176.1; no longer R178.1
- net LED_STATUS_R: now also D8.2 (A), R176.2; no longer R178.2
- net UART0_RX: now also J18.3
- net UART0_TX: now also J18.2
Other:
- moved on the sheet: D8, D9, R178
