File: hardware/arc1-compact/R10_WORK/cad/fpga12.kicad_sch (KiCad schematic)
At the start: 77 parts, among them J16 12F JTAG, U38 LFE5U-12F-6TG144C, U39 iso SCK, U40 iso MOSI, U41 iso SS, U42 iso MISO, X4 25MHz

Commit message: R10 D12: top USB-A game cartridge, no eMMC; USB2514B 4-port hub (3 ports used)
Owner direction: games are played directly from a USB drive in a top USB-A "cartridge"
port; the two front USB-A ports are controller inputs; eMMC not needed.
- Schematic: eMMC sheet removed (F133 PF0-PF6 freed); USB2422 replaced by USB2514B-I/M2
  (strap mode CFG_SEL=00, port 4 disabled by strap, CRFILT/PLLFILT 0.1 uF per DS00001692C);
  third TPS2051C + ESD + TVS + vertical USB-A (Molex 105057) marked TOP.
- crosscheck I: five exterior connectors (rear USB-C + HDMI, 2x front USB-A, top USB-A),
  eMMC/USB2422 must be absent, all three ports on the hub. PASS. ERC 0/0, pin review and
  pin/function matrix PASS, R10_HOST_CHECKS_PASS.
- PCB regenerated: Ø 119.8 mm, DRC 0 errors (unrouted), top cartridge at (-9.3, 24.2) mm.
- DECISIONS D12 (supersedes D10 and the four-connector rule); change-order report sections
  1, 2, 4, 5, 6 and the mechanical note updated; CLAUDE.md topology line amended.

Co-Authored-By: Claude Opus 5.5 <noreply@anthropic.com>
Claude-Session: https://claude.ai/code/session_01UkiuLdbjDvK75uDzAPKsGs
Parts:
- removed C205, C206, C207, C208, C209, C210: 100nF, Capacitor_SMD:C_0402_1005Metric, symbol ARC1_R10:C0402
- removed C211, C212: 10uF, Capacitor_SMD:C_0603_1608Metric, symbol ARC1_R10:C0603
- removed D6: 12F LED, LED_SMD:LED_0603_1608Metric, symbol ARC1_R10:LED
- removed J16: 12F JTAG, Connector_PinHeader_1.27mm:PinHeader_2x05_P1.27mm_Vertical_SMD, symbol ARC1_R10:HDR_2x5_127
- removed R131, R132, R133, R134, R135: 22R, Resistor_SMD:R_0402_1005Metric, symbol ARC1_R10:R0402
- removed TP67: ETH_TXCK, TestPoint:TestPoint_Pad_D1.0mm, symbol ARC1_R10:TP
- removed U38: LFE5U-12F-6TG144C, Package_QFP:TQFP-144_20x20mm_P0.5mm, symbol ARC1_R10:ECP5_12F_TQ144
- removed U39: iso SCK, Package_TO_SOT_SMD:SOT-353_SC-70-5, symbol ARC1_R10:LVC1G125
- added C235, C236, C237: 10uF, Capacitor_SMD:C_0603_1608Metric, symbol ARC1_R10:C0603
- added C238, C239, C240, C241, C242: 100nF, Capacitor_SMD:C_0402_1005Metric, symbol ARC1_R10:C0402
- added D7: 12F LED, LED_SMD:LED_0603_1608Metric, symbol ARC1_R10:LED
- added J17: 12F JTAG, Connector_PinHeader_1.27mm:PinHeader_2x05_P1.27mm_Vertical_SMD, symbol ARC1_R10:HDR_2x5_127
- added R164, R165, R166: 4.7k, Resistor_SMD:R_0402_1005Metric, symbol ARC1_R10:R0402
- added R167: 33R, Resistor_SMD:R_0402_1005Metric, symbol ARC1_R10:R0402
- added R168: 1k, Resistor_SMD:R_0402_1005Metric, symbol ARC1_R10:R0402
- added TP73: FPGA12_SCK, TestPoint:TestPoint_Pad_D1.0mm, symbol ARC1_R10:TP
- added U43: iso SS, Package_TO_SOT_SMD:SOT-353_SC-70-5, symbol ARC1_R10:LVC1G125
- added U44: iso MISO, Package_TO_SOT_SMD:SOT-353_SC-70-5, symbol ARC1_R10:LVC1G125
- C217, C227, C228, C229: value 10uF -> 100nF; footprint Capacitor_SMD:C_0603_1608Metric -> Capacitor_SMD:C_0402_1005Metric; symbol ARC1_R10:C0603 -> ARC1_R10:C0402; LCSC C19702 -> C1525; MPN CL10A106KP8NNNC -> CL05B104KO5NNNC
- C219, C220, C225: value 100nF -> 10uF; footprint Capacitor_SMD:C_0402_1005Metric -> Capacitor_SMD:C_0603_1608Metric; symbol ARC1_R10:C0402 -> ARC1_R10:C0603; LCSC C1525 -> C19702; MPN CL05B104KO5NNNC -> CL10A106KP8NNNC
- R136: Note F133->12F series R at the F133 (TXCTL) -> F133->12F series R at the F133 (TXCK)
- R137: Note 12F->F133 series R at the 12F (RXCK) -> F133->12F series R at the F133 (TXD0)
- R138: Note 12F->F133 series R at the 12F (RXD0) -> F133->12F series R at the F133 (TXD1)
- R139: Note 12F->F133 series R at the 12F (RXD1) -> F133->12F series R at the F133 (TXD2)
- R140: Note 12F->F133 series R at the 12F (RXD2) -> F133->12F series R at the F133 (TXD3)
- R141: Note 12F->F133 series R at the 12F (RXD3) -> F133->12F series R at the F133 (TXCTL)
- R142: Note 12F->F133 series R at the 12F (RXCTL) -> 12F->F133 series R at the 12F (RXCK)
- R143: value 100k -> 22R; LCSC C25741 -> C25092; MPN 0402WGF1003TCE -> 0402WGF220JTCE; Note 12F RX idle while F133 PG12 is hi-Z -> 12F->F133 series R at the 12F (RXD0)
- R144: value 100k -> 22R; LCSC C25741 -> C25092; MPN 0402WGF1003TCE -> 0402WGF220JTCE; Note F133 EMAC RX idle while the 12F is off/unconfigured -> 12F->F133 series R at the 12F (RXD1)
- R145: value 33R -> 22R; LCSC C25105 -> C25092; MPN 0402WGF330JTCE -> 0402WGF220JTCE; Note CCLK series R -> 12F->F133 series R at the 12F (RXD2)
- R146: value 10k -> 22R; LCSC C25744 -> C25092; MPN 0402WGF1002TCE -> 0402WGF220JTCE; Note buffers disabled at reset -> 12F->F133 series R at the 12F (RXD3)
- R147: value 10k -> 22R; LCSC C25744 -> C25092; MPN 0402WGF1002TCE -> 0402WGF220JTCE; Note FPGA deselected, MISO buffer off at reset -> 12F->F133 series R at the 12F (RXCTL)
- R148: Note (none) -> 12F RX idle while F133 PG12 is hi-Z
- R149: Note (none) -> F133 EMAC RX idle while the 12F is off/unconfigured
- R150: value 4.7k -> 33R; LCSC C25900 -> C25105; MPN 0402WGF4701TCE -> 0402WGF330JTCE; Note (none) -> CCLK series R
- R151: value 470R -> 10k; LCSC (none) -> C25744; MPN (none) -> 0402WGF1002TCE; Manufacturer (none) -> UNI-ROYAL; Note F133 PE8 open-drain use -> buffers disabled at reset; Reuse (none) -> SLIM4_R26_BOM_LINE (re-validate)
- R152: value 4.7k -> 10k; LCSC C25900 -> C25744; MPN 0402WGF4701TCE -> 0402WGF1002TCE; Note (none) -> FPGA deselected, MISO buffer off at reset
- R153, R154: value 4.7k -> 100k; LCSC C25900 -> C25741; MPN 0402WGF4701TCE -> 0402WGF1003TCE
- R155: Note CFG[2:0] = 001 slave SPI -> (none)
- R156: value 1k -> 470R; LCSC C11702 -> (none); MPN 0402WGF1001TCE -> (none); Manufacturer UNI-ROYAL -> (none); Note (none) -> F133 PE8 open-drain use; Reuse SLIM4_R26_BOM_LINE (re-validate) -> (none)
- R160: Note (none) -> CFG[2:0] = 001 slave SPI
- R161: value 4.7k -> 1k; LCSC C25900 -> C11702; MPN 0402WGF4701TCE -> 0402WGF1001TCE; Note open drain to F133 PE5 -> (none)
- R162: value 33R -> 4.7k; LCSC C25105 -> C25900; MPN 0402WGF330JTCE -> 0402WGF4701TCE
- R163: value 1k -> 4.7k; LCSC C11702 -> C25900; MPN 0402WGF1001TCE -> 0402WGF4701TCE
- TP68: value ETH_RXCK -> ETH_TXCK
- TP69: value FPGA12_DONE -> ETH_RXCK
- TP70: value FPGA12_PROGRAMN -> FPGA12_DONE
- TP71: value FPGA12_INITN -> FPGA12_PROGRAMN
- TP72: value FPGA12_SCK -> FPGA12_INITN
- U40: value iso MOSI -> LFE5U-12F-6TG144C; footprint Package_TO_SOT_SMD:SOT-353_SC-70-5 -> Package_QFP:TQFP-144_20x20mm_P0.5mm; symbol ARC1_R10:LVC1G125 -> ARC1_R10:ECP5_12F_TQ144; MPN SN74LVC1G125DCKR -> LFE5U-12F-6TG144C; Manufacturer Texas Instruments -> Lattice; Note Ioff: powered with the FPGA it drives -> (none); Source SN74LVC1G125 DS pin functions (sources/glue) -> Lattice FPGA-DS-02012 v3.4 + pinout FPGA-SC-02032 v2.1 (arc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
- U41: value iso SS -> iso SCK
- U42: value iso MISO -> iso MOSI; Note drives PC5 only while the F133 selects the FPGA -> Ioff: powered with the FPGA it drives
Connections:
- net 1V1_F12: now also C213.1, C214.1, C215.1, C216.1, C217.1, C218.1, C219.1, C220.1, U40.130 (VCC), U40.20 (VCC), U40.29 (VCC), U40.38 (VCC), U40.66 (VCC), U40.83 (VCC)
- net 2V5_F12: now also C221.1, C222.1, C223.1, C224.1, C225.1, U40.132 (VCCAUX), U40.17 (VCCAUX), U40.53 (VCCAUX), U40.96 (VCCAUX); no longer C213.1, C214.1, C215.1, C216.1, C217.1
- net 3V3: now also R151.2, R152.2, C241.1, U44.5 (VCC); no longer C233.1, R146.2, R147.2, U42.5 (VCC)
- net 3V3_F12: now also C233.1, R157.2, R163.2, U40.100 (VCCIO2), U40.122 (VCCIO1), U40.137 (VCCIO0), U40.16 (VCCIO6), U40.36 (VCCIO6), U40.43 (VCCIO8), U40.70 (VCCIO3), U40.86 (VCCIO3), U40.9 (VCCIO7), U42.5 (VCC), C235.1, C236.1, C237.1, C238.1, C239.1, C240.1, C242.1, J17.1, R164.2, R165.2, R166.2, U43.5 (VCC); no longer C218.1, C219.1, C220.1, C221.1, C222.1, C223.1, C224.1, C225.1, R150.2, R152.2, R153.2, R154.2, R156.2, U40.5 (VCC)
- net ETH_RXCK: now also R142.2, TP69.1; no longer R137.2, TP68.1
- net ETH_RXCK_E: now also R142.1, U40.110 (PT67A); no longer R137.1
- net ETH_RXCTL: now also R147.2, R149.1; no longer R142.2, R144.1
- net ETH_RXCTL_E: now also R147.1, U40.115 (PT58B); no longer R142.1
- net ETH_RXD0: now also R143.2; no longer R138.2
- net ETH_RXD0_E: now also R143.1, U40.111 (PT62B); no longer R138.1
- net ETH_RXD1: now also R144.2; no longer R139.2
- net ETH_RXD1_E: now also R144.1, U40.112 (PT62A); no longer R139.1
- net ETH_RXD2: now also R145.2; no longer R140.2
- net ETH_RXD2_E: now also R145.1, U40.113 (PT60B); no longer R140.1
- net ETH_RXD3: now also R146.2; no longer R141.2
- net ETH_RXD3_E: now also R146.1, U40.114 (PT60A); no longer R141.1
- net ETH_TXCK: now also R136.2, TP68.1, U40.128 (PT29A/PCLKT0_0)
- net ETH_TXCK_F: now also R136.1
- net ETH_TXCTL: now also R141.2, R148.1, U40.139 (PT9B); no longer R136.2, R143.1
- net ETH_TXCTL_F: now also R141.1; no longer R136.1
- net ETH_TXD0: now also R137.2, U40.133 (PT15B)
- net ETH_TXD0_F: now also R137.1
- net ETH_TXD1: now also R138.2, U40.134 (PT15A)
- net ETH_TXD1_F: now also R138.1
- net ETH_TXD2: now also R139.2, U40.135 (PT13B)
- net ETH_TXD2_F: now also R139.1
- net ETH_TXD3: now also R140.2, U40.136 (PT13A)
- net ETH_TXD3_F: now also R140.1
- net F12_LED0: now also U40.121 (PT51A), R168.1; no longer R163.1
- net F12_LED0_R: now also D7.2 (A), R168.2; no longer R163.2
- net F12_OSC_25M: now also U40.37 (PL47C/LLC_GPLL0T_IN), R167.2; no longer R162.2
- net F12_OSC_25M_X: now also R167.1; no longer R162.1
- net FPGA12_BUS_EN_N: now also R151.1, U42.1 (~{OE}), U43.1 (~{OE}); no longer R146.1, U40.1 (~{OE})
- net FPGA12_CFG0: now also R160.1, U40.62 (CFG_0); no longer R155.1
- net FPGA12_DONE: now also R158.1, TP70.1, U40.56 (DONE); no longer R153.1, TP69.1
- net FPGA12_INITN: now also R157.1, TP72.1, U40.55 (INITN); no longer R152.1, TP71.1
- net FPGA12_IRQ_N: now also U40.124 (PT42B), R166.1; no longer R161.1
- net FPGA12_MISO: now also R154.1, U40.46 (PB11A/D1), U44.2 (A); no longer R149.1, U42.2 (A)
- net FPGA12_MOSI: now also R153.1, U40.47 (PB11B/D0), U42.4 (Y); no longer R148.1, U40.4 (Y)
- net FPGA12_PROGRAMN: now also R155.1, R156.2, TP71.1, U40.57 (PROGRAMN), J17.10; no longer R150.1, R151.2, TP70.1
- net FPGA12_PROGRAMN_F: now also R156.1; no longer R151.1
- net FPGA12_SCK: now also R150.2, R161.1, U40.54 (CCLK/MCLK), TP73.1; no longer R145.2, R156.1, TP72.1
- net FPGA12_SCK_B: now also R150.1, U41.4 (Y); no longer R145.1
- net FPGA12_SS_N: now also R159.1, U40.48 (PB13A/SN), U43.4 (Y); no longer R154.1, U41.4 (Y)
- net FPGA12_SS_N_F: now also R152.1, U43.2 (A), U44.1 (~{OE}); no longer R147.1, U41.2 (A), U42.1 (~{OE})
- net FPGA12_TCK: now also R162.1, U40.63 (TCK), J17.4; no longer R157.1
- net FPGA12_TDI: now also U40.61 (TDI), J17.8, R164.1; no longer R159.1
- net FPGA12_TDO: now also U40.60 (TDO), J17.6, R165.1; no longer R160.1
- net FPGA12_TMS: now also R163.1, U40.64 (TMS), J17.2; no longer R158.1
- net GND: now also R153.2, R154.2, R162.2, U40.101 (GND), U40.123 (GND), U40.129 (GND), U40.131 (GND), U40.138 (GND), U40.15 (GND), U40.21 (GND), U40.32 (GND), U40.42 (GND), U40.58 (CFG_2), U40.59 (CFG_1), U40.65 (GND), U40.75 (GND), U40.8 (GND), U40.85 (GND), U40.87 (GND), C235.2, C236.2, C237.2, C238.2, C239.2, C240.2, C241.2, C242.2, D7.1 (K), J17.3, J17.5, J17.9, U43.3 (GND), U44.3 (GND); no longer R143.2, R144.2, R157.2, U40.3 (GND)
- net PSRAM_CE_N: now also U40.72 (PR44C)
- net PSRAM_SCLK_F: now also U40.73 (PR41D)
- net PSRAM_SIO0: now also U40.74 (PR41C)
- net PSRAM_SIO1: now also U40.76 (PR41B)
- net PSRAM_SIO2: now also U40.77 (PR41A)
- net PSRAM_SIO3: now also U40.78 (PR35D)
- net SPI0_CLK: now also U41.2 (A)
- net SPI0_MISO: now also U44.4 (Y); no longer U42.4 (Y)
- net SPI0_MOSI: now also U42.2 (A); no longer U40.2 (A)
Other:
- moved on the sheet: C213, C214, C215, C216, C217, C218, C219, C220, C221, C222, C223, C224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
