File: hardware/arc1-compact/R10_WORK/cad/psram12.kicad_sch (KiCad schematic)
At the start: 10 parts, among them U36 APS3204L-3SQNA-SN

Commit message: R10 change order rev 1.1: HDMI audio (ADV7513), USB0 role mux + hub + 2x front USB-A, eMMC, buttonless board
Owner handoff ARC1_R10_Handoff rev 1.1 (spec/, SHA-256 recorded) implemented in the generated schematic:
- D8 ADV7513BSWZ replaces the TFP410 (supersedes D6): D213 RGB888 video, D213 I2C2 init,
  F133 I2S2 -> HDMI embedded audio; own 1.8 V buck + 3 filtered domains; R_EXT 887R.
  D[23:0] pin order verified from the datasheet glyph coordinates.
- D9 F133 USB0 -> TS3USB221A (default rear USB-C device/FEL) or USB2422 hub -> two
  TPS2051C-switched front USB-A ports; F133 USB1 remains the internal D213 link; the D213
  recovery USB-C becomes internal fixture pads.
- D10 Samsung KLMAG1JETD-B041 16 GB eMMC on F133 SMHC0 (CONDITIONAL: SMHC0 documented for SD).
- D11 no switches: fixture pad pairs; game buttons, microSD and speakers removed.
- crosscheck_r10 section I (handoff go/no-go: 4 exterior connectors, 0 switches, I2S wired
  to the HDMI transmitter, USB0/USB1 roles, eMMC wiring) PASS; ERC 0/0; pin review PASS.
Sources: ADV7513 DS Rev B (LCSC copy), ADI AN-1270, Linux adv7511 driver, USB2422
DS00001726A, TPS20xxC SLVSAU6I, Samsung eMMC DS (not committed: vendor-confidential mark).

Co-Authored-By: Claude Opus 5.5 <noreply@anthropic.com>
Claude-Session: https://claude.ai/code/session_01UkiuLdbjDvK75uDzAPKsGs
Parts:
- removed C213: 100nF, Capacitor_SMD:C_0402_1005Metric, symbol ARC1_R10:C0402
- removed C214: 1uF, Capacitor_SMD:C_0402_1005Metric, symbol ARC1_R10:C0402
- removed R158: 22R, Resistor_SMD:R_0402_1005Metric, symbol ARC1_R10:R0402
- removed R159: 10k, Resistor_SMD:R_0402_1005Metric, symbol ARC1_R10:R0402
- removed R160, R161, R162, R163: 100k, Resistor_SMD:R_0402_1005Metric, symbol ARC1_R10:R0402
- removed U36: APS3204L-3SQNA-SN, Package_SO:SOIC-8_3.9x4.9mm_P1.27mm, symbol ARC1_R10:APS3204L
- added C235: 100nF, Capacitor_SMD:C_0402_1005Metric, symbol ARC1_R10:C0402
- added C236: 1uF, Capacitor_SMD:C_0402_1005Metric, symbol ARC1_R10:C0402
- added R165: 10k, Resistor_SMD:R_0402_1005Metric, symbol ARC1_R10:R0402
- added R166, R167, R168, R169, R170: 100k, Resistor_SMD:R_0402_1005Metric, symbol ARC1_R10:R0402
- added U43: APS3204L-3SQNA-SN, Package_SO:SOIC-8_3.9x4.9mm_P1.27mm, symbol ARC1_R10:APS3204L
- R164: value 100k -> 22R; LCSC C25741 -> C25092; MPN 0402WGF1003TCE -> 0402WGF220JTCE; Note static idle level -> source termination near the FPGA
Connections:
- net 3V3_F12: now also C235.1, C236.1, R165.2, U43.8 (VDD)
- net GND: now also C235.2, C236.2, R166.2, R167.2, R168.2, R169.2, R170.2, U43.4 (VSS); no longer R164.2
- net PSRAM_CE_N: now also R165.1, U43.1 (~{CE})
- net PSRAM_SCLK: now also R164.2, R166.1, U43.6 (SCLK)
- net PSRAM_SCLK_F: now also R164.1
- net PSRAM_SIO0: now also R167.1, U43.5 (SI_SIO0)
- net PSRAM_SIO1: now also R168.1, U43.2 (SO_SIO1)
- net PSRAM_SIO2: now also R169.1, U43.3 (SIO2)
- net PSRAM_SIO3: now also R170.1, U43.7 (SIO3); no longer R164.1
Other:
- moved on the sheet: R164

Commit message: R10 D12: top USB-A game cartridge, no eMMC; USB2514B 4-port hub (3 ports used)
Owner direction: games are played directly from a USB drive in a top USB-A "cartridge"
port; the two front USB-A ports are controller inputs; eMMC not needed.
- Schematic: eMMC sheet removed (F133 PF0-PF6 freed); USB2422 replaced by USB2514B-I/M2
  (strap mode CFG_SEL=00, port 4 disabled by strap, CRFILT/PLLFILT 0.1 uF per DS00001692C);
  third TPS2051C + ESD + TVS + vertical USB-A (Molex 105057) marked TOP.
- crosscheck I: five exterior connectors (rear USB-C + HDMI, 2x front USB-A, top USB-A),
  eMMC/USB2422 must be absent, all three ports on the hub. PASS. ERC 0/0, pin review and
  pin/function matrix PASS, R10_HOST_CHECKS_PASS.
- PCB regenerated: Ø 119.8 mm, DRC 0 errors (unrouted), top cartridge at (-9.3, 24.2) mm.
- DECISIONS D12 (supersedes D10 and the four-connector rule); change-order report sections
  1, 2, 4, 5, 6 and the mechanical note updated; CLAUDE.md topology line amended.

Co-Authored-By: Claude Opus 5.5 <noreply@anthropic.com>
Claude-Session: https://claude.ai/code/session_01UkiuLdbjDvK75uDzAPKsGs
Parts:
- removed C235: 100nF, Capacitor_SMD:C_0402_1005Metric, symbol ARC1_R10:C0402
- removed C236: 1uF, Capacitor_SMD:C_0402_1005Metric, symbol ARC1_R10:C0402
- removed R164: 22R, Resistor_SMD:R_0402_1005Metric, symbol ARC1_R10:R0402
- removed R165: 10k, Resistor_SMD:R_0402_1005Metric, symbol ARC1_R10:R0402
- removed R166, R167, R168: 100k, Resistor_SMD:R_0402_1005Metric, symbol ARC1_R10:R0402
- removed U43: APS3204L-3SQNA-SN, Package_SO:SOIC-8_3.9x4.9mm_P1.27mm, symbol ARC1_R10:APS3204L
- added C243: 100nF, Capacitor_SMD:C_0402_1005Metric, symbol ARC1_R10:C0402
- added C244: 1uF, Capacitor_SMD:C_0402_1005Metric, symbol ARC1_R10:C0402
- added R171, R172, R173, R174, R175: 100k, Resistor_SMD:R_0402_1005Metric, symbol ARC1_R10:R0402
- added U45: APS3204L-3SQNA-SN, Package_SO:SOIC-8_3.9x4.9mm_P1.27mm, symbol ARC1_R10:APS3204L
- R169: value 100k -> 22R; LCSC C25741 -> C25092; MPN 0402WGF1003TCE -> 0402WGF220JTCE; Note static idle level -> source termination near the FPGA
- R170: value 100k -> 10k; LCSC C25741 -> C25744; MPN 0402WGF1003TCE -> 0402WGF1002TCE; Note static idle level -> CE# tracks VDD during power-up (APS3204L s8)
Connections:
- net 3V3_F12: now also R170.2, C243.1, C244.1, U45.8 (VDD)
- net GND: now also C243.2, C244.2, R171.2, R172.2, R173.2, R174.2, R175.2, U45.4 (VSS); no longer R169.2, R170.2
- net PSRAM_CE_N: now also R170.1, U45.1 (~{CE})
- net PSRAM_SCLK: now also R169.2, R171.1, U45.6 (SCLK)
- net PSRAM_SCLK_F: now also R169.1
- net PSRAM_SIO0: now also R172.1, U45.5 (SI_SIO0)
- net PSRAM_SIO1: now also R173.1, U45.2 (SO_SIO1)
- net PSRAM_SIO2: now also R174.1, U45.3 (SIO2); no longer R169.1
- net PSRAM_SIO3: now also R175.1, U45.7 (SIO3); no longer R170.1
Other:
- moved on the sheet: R169, R170
