File: hardware/arc1-compact/R10_WORK/cad/sdram45.kicad_sch (KiCad schematic)
At the start: 13 parts, among them U30 AS4C16M16SA-6TIN

Commit message: R10 schematic: SDRAM net rename (collision with microSD clock found by crosscheck), 12F config buffers on 3V3_F12, crosscheck_r10 (A-H) PASS, every-pin review tables
Co-Authored-By: Claude Opus 5.5 <noreply@anthropic.com>
Claude-Session: https://claude.ai/code/session_01UkiuLdbjDvK75uDzAPKsGs
Parts:
- TP58: value SD_CLK -> SDR_CLK
Connections:
- net SD_A0 renamed SDR_A0
- net SD_A1 renamed SDR_A1
- net SD_A10 renamed SDR_A10
- net SD_A11 renamed SDR_A11
- net SD_A12 renamed SDR_A12
- net SD_A2 renamed SDR_A2
- net SD_A3 renamed SDR_A3
- net SD_A4 renamed SDR_A4
- net SD_A5 renamed SDR_A5
- net SD_A6 renamed SDR_A6
- net SD_A7 renamed SDR_A7
- net SD_A8 renamed SDR_A8
- net SD_A9 renamed SDR_A9
- net SD_BA0 renamed SDR_BA0
- net SD_BA1 renamed SDR_BA1
- net SD_CAS_N renamed SDR_CAS_N
- net SD_CKE renamed SDR_CKE
- net SD_CLK renamed SDR_CLK
- net SD_CLK_F renamed SDR_CLK_F
- net SD_CS_N renamed SDR_CS_N
- net SD_DQ0 renamed SDR_DQ0
- net SD_DQ1 renamed SDR_DQ1
- net SD_DQ10 renamed SDR_DQ10
- net SD_DQ11 renamed SDR_DQ11
- net SD_DQ12 renamed SDR_DQ12
- net SD_DQ13 renamed SDR_DQ13
- net SD_DQ14 renamed SDR_DQ14
- net SD_DQ15 renamed SDR_DQ15
- net SD_DQ2 renamed SDR_DQ2
- net SD_DQ3 renamed SDR_DQ3
- net SD_DQ4 renamed SDR_DQ4
- net SD_DQ5 renamed SDR_DQ5
- net SD_DQ6 renamed SDR_DQ6
- net SD_DQ7 renamed SDR_DQ7
- net SD_DQ8 renamed SDR_DQ8
- net SD_DQ9 renamed SDR_DQ9
- net SD_DQM0 renamed SDR_DQM0
- net SD_DQM1 renamed SDR_DQM1
- net SD_RAS_N renamed SDR_RAS_N
- net SD_WE_N renamed SDR_WE_N

Commit message: R10 change order rev 1.1: HDMI audio (ADV7513), USB0 role mux + hub + 2x front USB-A, eMMC, buttonless board
Owner handoff ARC1_R10_Handoff rev 1.1 (spec/, SHA-256 recorded) implemented in the generated schematic:
- D8 ADV7513BSWZ replaces the TFP410 (supersedes D6): D213 RGB888 video, D213 I2C2 init,
  F133 I2S2 -> HDMI embedded audio; own 1.8 V buck + 3 filtered domains; R_EXT 887R.
  D[23:0] pin order verified from the datasheet glyph coordinates.
- D9 F133 USB0 -> TS3USB221A (default rear USB-C device/FEL) or USB2422 hub -> two
  TPS2051C-switched front USB-A ports; F133 USB1 remains the internal D213 link; the D213
  recovery USB-C becomes internal fixture pads.
- D10 Samsung KLMAG1JETD-B041 16 GB eMMC on F133 SMHC0 (CONDITIONAL: SMHC0 documented for SD).
- D11 no switches: fixture pad pairs; game buttons, microSD and speakers removed.
- crosscheck_r10 section I (handoff go/no-go: 4 exterior connectors, 0 switches, I2S wired
  to the HDMI transmitter, USB0/USB1 roles, eMMC wiring) PASS; ERC 0/0; pin review PASS.
Sources: ADV7513 DS Rev B (LCSC copy), ADI AN-1270, Linux adv7511 driver, USB2422
DS00001726A, TPS20xxC SLVSAU6I, Samsung eMMC DS (not committed: vendor-confidential mark).

Co-Authored-By: Claude Opus 5.5 <noreply@anthropic.com>
Claude-Session: https://claude.ai/code/session_01UkiuLdbjDvK75uDzAPKsGs
Parts:
- removed C174, C175, C176, C177, C178, C179, C180: 100nF, Capacitor_SMD:C_0402_1005Metric, symbol ARC1_R10:C0402
- removed C181, C182: 10uF, Capacitor_SMD:C_0603_1608Metric, symbol ARC1_R10:C0603
- removed R123: 22R, Resistor_SMD:R_0402_1005Metric, symbol ARC1_R10:R0402
- removed R124: 10k, Resistor_SMD:R_0402_1005Metric, symbol ARC1_R10:R0402
- removed TP58: SDR_CLK, TestPoint:TestPoint_Pad_D1.0mm, symbol ARC1_R10:TP
- removed U30: AS4C16M16SA-6TIN, Package_SO:TSOP-II-54_22.2x10.16mm_P0.8mm, symbol ARC1_R10:AS4C16M16SA
- added C196, C197, C198, C199, C200, C201, C202: 100nF, Capacitor_SMD:C_0402_1005Metric, symbol ARC1_R10:C0402
- added C203, C204: 10uF, Capacitor_SMD:C_0603_1608Metric, symbol ARC1_R10:C0603
- added R129: 22R, Resistor_SMD:R_0402_1005Metric, symbol ARC1_R10:R0402
- added R130: 10k, Resistor_SMD:R_0402_1005Metric, symbol ARC1_R10:R0402
- added TP66: SDR_CLK, TestPoint:TestPoint_Pad_D1.0mm, symbol ARC1_R10:TP
- added U37: AS4C16M16SA-6TIN, Package_SO:TSOP-II-54_22.2x10.16mm_P0.8mm, symbol ARC1_R10:AS4C16M16SA
Connections:
- net 3V3_F45: now also C196.1, C197.1, C198.1, C199.1, C200.1, C201.1, C202.1, C203.1, C204.1, U37.1 (VDD), U37.14 (VDD), U37.27 (VDD), U37.3 (VDDQ), U37.43 (VDDQ), U37.49 (VDDQ), U37.9 (VDDQ)
- net GND: now also C196.2, C197.2, C198.2, C199.2, C200.2, C201.2, C202.2, C203.2, C204.2, R130.2, U37.12 (VSSQ), U37.28 (VSS), U37.41 (VSS), U37.46 (VSSQ), U37.52 (VSSQ), U37.54 (VSS), U37.6 (VSSQ)
- net SDR_A0: now also U37.23 (A0)
- net SDR_A1: now also U37.24 (A1)
- net SDR_A10: now also U37.22 (A10)
- net SDR_A11: now also U37.35 (A11)
- net SDR_A12: now also U37.36 (A12)
- net SDR_A2: now also U37.25 (A2)
- net SDR_A3: now also U37.26 (A3)
- net SDR_A4: now also U37.29 (A4)
- net SDR_A5: now also U37.30 (A5)
- net SDR_A6: now also U37.31 (A6)
- net SDR_A7: now also U37.32 (A7)
- net SDR_A8: now also U37.33 (A8)
- net SDR_A9: now also U37.34 (A9)
- net SDR_BA0: now also U37.20 (BA0)
- net SDR_BA1: now also U37.21 (BA1)
- net SDR_CAS_N: now also U37.17 (~{CAS})
- net SDR_CKE: now also R130.1, U37.37 (CKE)
- net SDR_CLK: now also R129.2, TP66.1, U37.38 (CLK)
- net SDR_CLK_F: now also R129.1
- net SDR_CS_N: now also U37.19 (~{CS})
- net SDR_DQ0: now also U37.2 (DQ0)
- net SDR_DQ1: now also U37.4 (DQ1)
- net SDR_DQ10: now also U37.45 (DQ10)
- net SDR_DQ11: now also U37.47 (DQ11)
- net SDR_DQ12: now also U37.48 (DQ12)
- net SDR_DQ13: now also U37.50 (DQ13)
- net SDR_DQ14: now also U37.51 (DQ14)
- net SDR_DQ15: now also U37.53 (DQ15)
- net SDR_DQ2: now also U37.5 (DQ2)
- net SDR_DQ3: now also U37.7 (DQ3)
- net SDR_DQ4: now also U37.8 (DQ4)
- net SDR_DQ5: now also U37.10 (DQ5)
- net SDR_DQ6: now also U37.11 (DQ6)
- net SDR_DQ7: now also U37.13 (DQ7)
- net SDR_DQ8: now also U37.42 (DQ8)
- net SDR_DQ9: now also U37.44 (DQ9)
- net SDR_DQM0: now also U37.15 (LDQM)
- net SDR_DQM1: now also U37.39 (UDQM)
- net SDR_RAS_N: now also U37.18 (~{RAS})
- net SDR_WE_N: now also U37.16 (~{WE})

Commit message: R10 D12: top USB-A game cartridge, no eMMC; USB2514B 4-port hub (3 ports used)
Owner direction: games are played directly from a USB drive in a top USB-A "cartridge"
port; the two front USB-A ports are controller inputs; eMMC not needed.
- Schematic: eMMC sheet removed (F133 PF0-PF6 freed); USB2422 replaced by USB2514B-I/M2
  (strap mode CFG_SEL=00, port 4 disabled by strap, CRFILT/PLLFILT 0.1 uF per DS00001692C);
  third TPS2051C + ESD + TVS + vertical USB-A (Molex 105057) marked TOP.
- crosscheck I: five exterior connectors (rear USB-C + HDMI, 2x front USB-A, top USB-A),
  eMMC/USB2422 must be absent, all three ports on the hub. PASS. ERC 0/0, pin review and
  pin/function matrix PASS, R10_HOST_CHECKS_PASS.
- PCB regenerated: Ø 119.8 mm, DRC 0 errors (unrouted), top cartridge at (-9.3, 24.2) mm.
- DECISIONS D12 (supersedes D10 and the four-connector rule); change-order report sections
  1, 2, 4, 5, 6 and the mechanical note updated; CLAUDE.md topology line amended.

Co-Authored-By: Claude Opus 5.5 <noreply@anthropic.com>
Claude-Session: https://claude.ai/code/session_01UkiuLdbjDvK75uDzAPKsGs
Parts:
- removed C196, C197, C198, C199, C200, C201, C202: 100nF, Capacitor_SMD:C_0402_1005Metric, symbol ARC1_R10:C0402
- removed C203: 10uF, Capacitor_SMD:C_0603_1608Metric, symbol ARC1_R10:C0603
- removed R129: 22R, Resistor_SMD:R_0402_1005Metric, symbol ARC1_R10:R0402
- removed R130: 10k, Resistor_SMD:R_0402_1005Metric, symbol ARC1_R10:R0402
- removed TP66: SDR_CLK, TestPoint:TestPoint_Pad_D1.0mm, symbol ARC1_R10:TP
- removed U37: AS4C16M16SA-6TIN, Package_SO:TSOP-II-54_22.2x10.16mm_P0.8mm, symbol ARC1_R10:AS4C16M16SA
- added C205, C206, C207, C208, C209, C210: 100nF, Capacitor_SMD:C_0402_1005Metric, symbol ARC1_R10:C0402
- added C211, C212: 10uF, Capacitor_SMD:C_0603_1608Metric, symbol ARC1_R10:C0603
- added R134: 22R, Resistor_SMD:R_0402_1005Metric, symbol ARC1_R10:R0402
- added R135: 10k, Resistor_SMD:R_0402_1005Metric, symbol ARC1_R10:R0402
- added TP67: SDR_CLK, TestPoint:TestPoint_Pad_D1.0mm, symbol ARC1_R10:TP
- added U39: AS4C16M16SA-6TIN, Package_SO:TSOP-II-54_22.2x10.16mm_P0.8mm, symbol ARC1_R10:AS4C16M16SA
- C204: value 10uF -> 100nF; footprint Capacitor_SMD:C_0603_1608Metric -> Capacitor_SMD:C_0402_1005Metric; symbol ARC1_R10:C0603 -> ARC1_R10:C0402; LCSC C19702 -> C1525; MPN CL10A106KP8NNNC -> CL05B104KO5NNNC
Connections:
- net 3V3_F45: now also C205.1, C206.1, C207.1, C208.1, C209.1, C210.1, C211.1, C212.1, U39.1 (VDD), U39.14 (VDD), U39.27 (VDD), U39.3 (VDDQ), U39.43 (VDDQ), U39.49 (VDDQ), U39.9 (VDDQ)
- net GND: now also C205.2, C206.2, C207.2, C208.2, C209.2, C210.2, C211.2, C212.2, R135.2, U39.12 (VSSQ), U39.28 (VSS), U39.41 (VSS), U39.46 (VSSQ), U39.52 (VSSQ), U39.54 (VSS), U39.6 (VSSQ)
- net SDR_A0: now also U39.23 (A0)
- net SDR_A1: now also U39.24 (A1)
- net SDR_A10: now also U39.22 (A10)
- net SDR_A11: now also U39.35 (A11)
- net SDR_A12: now also U39.36 (A12)
- net SDR_A2: now also U39.25 (A2)
- net SDR_A3: now also U39.26 (A3)
- net SDR_A4: now also U39.29 (A4)
- net SDR_A5: now also U39.30 (A5)
- net SDR_A6: now also U39.31 (A6)
- net SDR_A7: now also U39.32 (A7)
- net SDR_A8: now also U39.33 (A8)
- net SDR_A9: now also U39.34 (A9)
- net SDR_BA0: now also U39.20 (BA0)
- net SDR_BA1: now also U39.21 (BA1)
- net SDR_CAS_N: now also U39.17 (~{CAS})
- net SDR_CKE: now also R135.1, U39.37 (CKE)
- net SDR_CLK: now also R134.2, TP67.1, U39.38 (CLK)
- net SDR_CLK_F: now also R134.1
- net SDR_CS_N: now also U39.19 (~{CS})
- net SDR_DQ0: now also U39.2 (DQ0)
- net SDR_DQ1: now also U39.4 (DQ1)
- net SDR_DQ10: now also U39.45 (DQ10)
- net SDR_DQ11: now also U39.47 (DQ11)
- net SDR_DQ12: now also U39.48 (DQ12)
- net SDR_DQ13: now also U39.50 (DQ13)
- net SDR_DQ14: now also U39.51 (DQ14)
- net SDR_DQ15: now also U39.53 (DQ15)
- net SDR_DQ2: now also U39.5 (DQ2)
- net SDR_DQ3: now also U39.7 (DQ3)
- net SDR_DQ4: now also U39.8 (DQ4)
- net SDR_DQ5: now also U39.10 (DQ5)
- net SDR_DQ6: now also U39.11 (DQ6)
- net SDR_DQ7: now also U39.13 (DQ7)
- net SDR_DQ8: now also U39.42 (DQ8)
- net SDR_DQ9: now also U39.44 (DQ9)
- net SDR_DQM0: now also U39.15 (LDQM)
- net SDR_DQM1: now also U39.39 (UDQM)
- net SDR_RAS_N: now also U39.18 (~{RAS})
- net SDR_WE_N: now also U39.16 (~{WE})
Other:
- moved on the sheet: C204
