File: hardware/arc1-compact/R10_WORK/cad/usb_host.kicad_sch (KiCad schematic)
At the start: 44 parts, among them J12 USB-A Player 1, J13 USB-A Player 2 / game load, U25 TS3USB221A, U26 USB2422-I/MJ, U27 USB-A1 power, U28 TPD2EUSB30, U29 USB-A2 power, U30 TPD2EUSB30, Y3 24MHz +-50ppm

Commit message: R10 D12: top USB-A game cartridge, no eMMC; USB2514B 4-port hub (3 ports used)
Owner direction: games are played directly from a USB drive in a top USB-A "cartridge"
port; the two front USB-A ports are controller inputs; eMMC not needed.
- Schematic: eMMC sheet removed (F133 PF0-PF6 freed); USB2422 replaced by USB2514B-I/M2
  (strap mode CFG_SEL=00, port 4 disabled by strap, CRFILT/PLLFILT 0.1 uF per DS00001692C);
  third TPS2051C + ESD + TVS + vertical USB-A (Molex 105057) marked TOP.
- crosscheck I: five exterior connectors (rear USB-C + HDMI, 2x front USB-A, top USB-A),
  eMMC/USB2422 must be absent, all three ports on the hub. PASS. ERC 0/0, pin review and
  pin/function matrix PASS, R10_HOST_CHECKS_PASS.
- PCB regenerated: Ø 119.8 mm, DRC 0 errors (unrouted), top cartridge at (-9.3, 24.2) mm.
- DECISIONS D12 (supersedes D10 and the four-connector rule); change-order report sections
  1, 2, 4, 5, 6 and the mechanical note updated; CLAUDE.md topology line amended.

Co-Authored-By: Claude Opus 5.5 <noreply@anthropic.com>
Claude-Session: https://claude.ai/code/session_01UkiuLdbjDvK75uDzAPKsGs
Parts:
- added C121, C125: 1uF, Capacitor_SMD:C_0402_1005Metric, symbol ARC1_R10:C0402
- added C122, C126: 100uF, Capacitor_SMD:C_1210_3225Metric, symbol ARC1_R10:C1210
- added C123, C127: 22uF, Capacitor_SMD:C_0805_2012Metric, symbol ARC1_R10:C0805
- added C124, C128: 100nF, Capacitor_SMD:C_0402_1005Metric, symbol ARC1_R10:C0402
- added D5: SMF5.0A, Diode_SMD:D_SMF, symbol ARC1_R10:TVS_SMF
- added J14: USB-A game cartridge, Connector_USB:USB_A_Molex_105057_Vertical, symbol ARC1_R10:USB_A_V
- added R75, R76: 100k, Resistor_SMD:R_0402_1005Metric, symbol ARC1_R10:R0402
- added R77, R78, R79: 10k, Resistor_SMD:R_0402_1005Metric, symbol ARC1_R10:R0402
- added TP52: HUB_UP_DM, TestPoint:TestPoint_Pad_D1.0mm, symbol ARC1_R10:TP
- added U31: USB-A3 power, Package_TO_SOT_SMD:SOT-23-5, symbol ARC1_R10:TPS2051C
- added U32: TPD2EUSB30, ARC1_R10:SLIM4_FP_U11_TPD2EUSB30_DRT3, symbol ARC1_R10:TPD2EUSB30
- C106: Note pin 1 (DS 2.3) -> (none)
- C107: value 1uF -> 100nF; LCSC C52923 -> C1525; MPN CL05A105KA5NQNC -> CL05B104KO5NNNC; Note pin 9 (DS 2.3) -> (none)
- C108: Note pin 18 -> (none)
- C109: value 1uF -> 100nF; LCSC C52923 -> C1525; MPN CL05A105KA5NQNC -> CL05B104KO5NNNC; Note core regulator filter, low ESR -> (none)
- C110: Note <= 0.1 uF -> (none)
- C111: value 18pF -> 100nF; LCSC (none) -> C1525; MPN (none) -> CL05B104KO5NNNC; Manufacturer (none) -> Samsung; Note ~18 pF each (DS Note 6.2); match to crystal CL -> (none); Reuse (none) -> SLIM4_R26_BOM_LINE (re-validate)
- C112: value 18pF -> 4.7uF; footprint Capacitor_SMD:C_0402_1005Metric -> Capacitor_SMD:C_0603_1608Metric; symbol ARC1_R10:C0402 -> ARC1_R10:C0603; LCSC (none) -> C19666; MPN (none) -> CL10A475KO8NNNC; Manufacturer (none) -> Samsung; Reuse (none) -> SLIM4_R26_BOM_LINE (re-validate)
- C113: value 1uF -> 100nF; LCSC C52923 -> C1525; MPN CL05A105KA5NQNC -> CL05B104KO5NNNC; Note IN cap (>= 0.1 uF, DS) -> <= 0.1 uF low ESR (DS 3.2)
- C114: value 100uF -> 100nF; footprint Capacitor_SMD:C_1210_3225Metric -> Capacitor_SMD:C_0402_1005Metric; symbol ARC1_R10:C1210 -> ARC1_R10:C0402; LCSC (none) -> C1525; MPN (none) -> CL05B104KO5NNNC; Manufacturer (none) -> Samsung; Note downstream VBUS bulk (USB 2.0: >= 120 uF per hub port incl.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 -> <= 0.1 uF; Reuse (none) -> SLIM4_R26_BOM_LINE (re-validate)
- C115: value 22uF -> 18pF; footprint Capacitor_SMD:C_0805_2012Metric -> Capacitor_SMD:C_0402_1005Metric; symbol ARC1_R10:C0805 -> ARC1_R10:C0402; LCSC C5674 -> (none); MPN CL21A226MQQNNNE -> (none); Manufacturer Samsung -> (none); Note (none) -> match to crystal CL; Reuse SLIM4_R26_BOM_LINE (re-validate) -> (none)
- C116: value 100nF -> 18pF; LCSC C1525 -> (none); MPN CL05B104KO5NNNC -> (none); Manufacturer Samsung -> (none); Reuse SLIM4_R26_BOM_LINE (re-validate) -> (none)
- C118: Note downstream VBUS bulk (USB 2.0: >= 120 uF per hub port incl.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 -> downstream VBUS bulk (USB 2.0: >= 120 uF per port incl. the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
- J12: Note FRONT. Through-hole shell -> FRONT. Controller port (handoff s1)
- J13: value USB-A Player 2 / game load -> USB-A Player 2; Note FRONT. Through-hole shell -- reinforced: shell tabs soldere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 -> FRONT. Controller port (handoff s1)
- R66: Note 12.0k 1 % (DS 2.3) -> 12.0k 1 % (DS 3.2)
- R67: Note CFG_SEL = 0: default configuration, straps enabled (Table 4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 -> CFG_SEL0 = 0
- R68: value 10k -> 100k; LCSC C25744 -> C25741; MPN 0402WGF1002TCE -> 0402WGF1003TCE; Note NON_REM[1:0] = 00: both ports removable -> CFG_SEL1 = 0 (HS_IND pin: 47-100k strap, Table 3-3)
- R69: value 10k -> 100k; LCSC C25744 -> C25741; MPN 0402WGF1002TCE -> 0402WGF1003TCE; Note (none) -> NON_REM[1:0] = 00: all ports removable (47-100k)
- R70: value 10k -> 100k; LCSC C25744 -> C25741; MPN 0402WGF1002TCE -> 0402WGF1003TCE; Note hub in reset until F133 PD3 releases it (>= 1 us pulse) -> (none)
- R71: value 100k -> 10k; LCSC C25741 -> C25744; MPN 0402WGF1003TCE -> 0402WGF1002TCE; Note BC_EN1 strap = 0 (no battery charging) and switch off in re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 -> port 4 disable strap: both DN4 pins pulled up (DS 3.2)
- R72: value 100k -> 10k; LCSC C25741 -> C25744; MPN 0402WGF1003TCE -> 0402WGF1002TCE; Note switch off in reset -> unused over-current input held inactive
- R73: Note FLT open drain (hub also has an internal pull-up) -> hub in reset until F133 PD3 releases it
- R74: value 10k -> 100k; LCSC C25744 -> C25741; MPN 0402WGF1002TCE -> 0402WGF1003TCE; Note FLT open drain (hub also has an internal pull-up) -> BC_EN strap = 0 and port power off in reset
- TP48: value USB0_SEL -> USBA3_VBUS
- TP49: value HUB_RESET_N -> USB0_SEL
- TP50: value HUB_UP_DP -> HUB_RESET_N
- TP51: value HUB_UP_DM -> HUB_UP_DP
- U26: value USB2422-I/MJ -> USB2514B-I/M2; footprint Package_DFN_QFN:QFN-24-1EP_4x4mm_P0.5mm_EP2.6x2.6mm_ThermalVias -> Package_DFN_QFN:QFN-36-1EP_6x6mm_P0.5mm_EP3.7x3.7mm_ThermalVias; symbol ARC1_R10:USB2422 -> ARC1_R10:USB2514B; MPN USB2422-I/MJ -> USB2514B-I/M2; Note strap mode (CFG_SEL=0): self-powered, both ports removable,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 -> D12. Strap mode CFG_SEL[1:0]=00 (Table 5-1): self-powered, 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; Source Microchip DS00001726A Figure 2.1 / Table 2.2 (sources/micro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 -> Microchip DS00001692C Table 3-1 (USB2514B column) / Table 5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
- U27, U29: Note 0.5 A current limit, fault -> hub OCS (port power budgeted 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 -> 0.5 A current limit, fault -> hub OCS
- Y3: Note fundamental, parallel resonant, +-350 ppm max (DS 6) -> 24 MHz fundamental; load caps per crystal CL
Connections:
- net 3V3: now also C109.1, C110.1, C111.1, C112.1, R71.2, R72.2, U26.10 (VDDA33), U26.15 (VDD33), U26.23 (VDD33), U26.27 (VBUS_DET), U26.29 (VDDA33), U26.36 (VDDA33), U26.5 (VDDA33), R77.2, R78.2, R79.2; no longer R73.2, R74.2, U26.1 (VDD33), U26.16 (VBUS_DET), U26.18 (VDD33), U26.9 (VDD33)
- net GND: now also R73.2, R74.2, U26.11 (TEST), U26.37 (VSS_EP), C121.2, C122.2, C123.2, C124.2, C125.2, C126.2, C127.2, C128.2, D5.2 (A), J14.4 (GND), J14.5 (SHIELD), R75.2, R76.2, U31.2 (GND), U32.3 (GND); no longer R71.2, R72.2, U26.25 (VSS_EP)
- net HUB_CRFILT: now also C113.1, U26.14 (CRFILT); no longer C109.1, U26.10 (CRFILT)
- net HUB_NON_REM0: now also R70.1, U26.28 (SUSP_IND/NON_REM0); no longer R69.1, U26.17 (SUSP_IND/NON_REM0)
- net HUB_NON_REM1: now also R69.1, U26.22 (SDA/NON_REM1); no longer R68.1, U26.13 (SMBDATA/NON_REM1)
- net HUB_OCS1_N: now also U26.13 (OCS_N1), R77.1; no longer R73.1, U26.8 (OCS1_N)
- net HUB_OCS2_N: now also U26.17 (OCS_N2), R78.1; no longer R74.1, U26.12 (OCS2_N)
- net HUB_PLLFILT: now also C114.1, U26.34 (PLLFILT); no longer C110.1, U26.23 (PLLFILT)
- net HUB_PRTPWR1: now also R74.1, U26.12 (PRTPWR1/BC_EN1); no longer R71.1, U26.7 (PRTPWR1/BC_EN1)
- net HUB_PRTPWR2: now also U26.16 (PRTPWR2/BC_EN2), R75.1; no longer R72.1, U26.11 (PRTPWR2)
- net HUB_RBIAS: now also U26.35 (RBIAS); no longer U26.24 (RBIAS)
- net HUB_RESET_N: now also R73.1, TP50.1, U26.26 (RESET_N); no longer R70.1, TP49.1, U26.15 (RESET_N)
- net HUB_UP_DM: now also U26.30 (USBDM_UP), TP52.1; no longer TP51.1, U26.19 (USBDM_UP)
- net HUB_UP_DP: now also TP51.1, U26.31 (USBDP_UP); no longer TP50.1, U26.20 (USBDP_UP)
- net HUB_XI: now also C115.1, U26.33 (XTALIN/CLKIN); no longer C111.1, U26.22 (XTALIN)
- net HUB_XO: now also C116.1, U26.32 (XTALOUT); no longer C112.1, U26.21 (XTALOUT)
- net USB0_SEL: now also TP49.1; no longer TP48.1
- net USBA1_DM: now also U26.1 (USBDM_DN1); no longer U26.2 (USBDM_DN1)
- net USBA1_DP: now also U26.2 (USBDP_DN1); no longer U26.3 (USBDP_DN1)
- net USBA1_VBUS: now also C118.1, C119.1, C120.1; no longer C114.1, C115.1, C116.1
- net USBA2_DM: now also U26.3 (USBDM_DN2); no longer U26.4 (USBDM_DN2)
- net USBA2_DP: now also U26.4 (USBDP_DN2); no longer U26.5 (USBDP_DN2)
- net USBA2_VBUS: now also C122.1, C123.1, C124.1; no longer C118.1, C119.1, C120.1
- net VBUS_5V: now also C121.1, C125.1, U31.5 (IN); no longer C113.1
- net USBA3_DM: now reaches U26.6 (USBDM_DN3)
- net USBA3_DM: now also J14.2 (D-), U32.2 (D-)
- net HUB_CFG_SEL renamed HUB_CFG_SEL0
- net HUB_CFG_SEL0: now also U26.24 (SCL/CFG_SEL0); no longer U26.14 (SMBCLK/CFG_SEL0)
- new net HUB_CFG_SEL1: R68.1, U26.25 (HS_IND/CFG_SEL1)
- new net HUB_DN4_DIS: R71.1, U26.8 (USBDM_DN4/PRT_DIS_M4), U26.9 (USBDP_DN4/PRT_DIS_P4)
- new net HUB_OCS3_N: R79.1, U26.19 (OCS_N3), U31.3 (~{FLT})
- new net HUB_OCS4_N: R72.1, U26.21 (OCS_N4)
- new net HUB_PRTPWR3: R76.1, U26.18 (PRTPWR3/BC_EN3), U31.4 (EN)
- new net USBA3_DP: J14.3 (D+), U26.7 (USBDP_DN3), U32.1 (D+)
- new net USBA3_VBUS: C126.1, C127.1, C128.1, D5.1 (K), J14.1 (VBUS), TP48.1, U31.1 (OUT)
Other:
- note added: "F133 USB0 role mux: rear USB-C (device/FEL, default) or USB2514B hub -> 2x front USB-A + top cartridge USB-A Sheet generated from design.py; global labels carry every net."
- note removed: "F133 USB0 role mux: rear USB-C (device/FEL, default) or USB2422 hub -> front USB-A Player 1 / Player 2 Sheet generated from design.py; global labels carry every net."
- title: ARC-1 Compact R10: F133 USB0 role mux: rear USB-C (device/FEL, default) or USB2422 hub -> front USB-A Player 1 / Player 2 -> ARC-1 Compact R10: F133 USB0 role mux: rear USB-C (device/FEL, default) or USB2514B hub -> 2x front USB-A + top cartridge USB-A
- moved on the sheet: C105, C106, C107, C108, C109, C110, C111, C112, C113, C114, C115, C116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
