File: hardware/arc1-compact/R10_WORK/cad/ARC1_R10.kicad_pcb (KiCad board)
At the start: 6 copper layers, 119.6 x 109.7 mm, 597 parts, among them J1 USB-C receptacle, J10 D213 USB path select, J11 D213 recovery USB pads, J12 USB-A Player 1, J13 USB-A Player 2 / game load, J14 HDMI type-A, J15 45F JTAG, J16 12F JTAG, J17 F133 UART0, J2 F133 RESET pads, J3 F45 power override, J4 F12 power override, J5 FEL pads (NOR reset), J6 LA SPI0, J7 D213 RESET pads, J8 D213 BOOT pads (PA0), J9 D213 UART0, U1 TUSB320LAI, U10 D213_DRAM, U11 HDMI_1V8, U12 F45_VCC, U13 3V3_F45 switch, U14 2V5_F45, U15 F12_VCC, U16 3V3_F12 switch, U17 2V5_F12, U18 F133-B, U19 W25Q512JVFIQ, U2 TPD2EUSB30, U20 D213ECV, U21 D213 ctl OD, U22 W25Q512JVFIQ, U23 TS3USB221A, U24 TPD2EUSB30, U25 TS3USB221A, U26 USB2422-I/MJ, U27 USB-A1 power, U28 TPD2EUSB30, U29 USB-A2 power, U3 3V3, U30 TPD2EUSB30, U31 ADV7513BSWZ, U32 TPD12S016, U33 LFE5U-45F-6BG381C, U34 iso FPGA45_SCK_B, U35 iso FPGA45_MOSI, U36 iso FPGA45_SS_N, U37 AS4C16M16SA-6TIN, U38 LFE5U-12F-6TG144C, U39 iso SCK, U4 TPS3808G33, U40 iso MOSI, U41 iso SS, U42 iso MISO, U43 APS3204L-3SQNA-SN, U44 KLMAG1JETD-B041, U5 F133_CORE, U6 F133_DRAM, U7 1V8_AN, U8 TPS3808G09, U9 D213_CORE, X1 12MHz, X2 125MHz, X3 25MHz, X4 25MHz, Y1 24MHz, Y2 24MHz +-20ppm, Y3 24MHz +-50ppm

Commit message: R10 D12: top USB-A game cartridge, no eMMC; USB2514B 4-port hub (3 ports used)
Owner direction: games are played directly from a USB drive in a top USB-A "cartridge"
port; the two front USB-A ports are controller inputs; eMMC not needed.
- Schematic: eMMC sheet removed (F133 PF0-PF6 freed); USB2422 replaced by USB2514B-I/M2
  (strap mode CFG_SEL=00, port 4 disabled by strap, CRFILT/PLLFILT 0.1 uF per DS00001692C);
  third TPS2051C + ESD + TVS + vertical USB-A (Molex 105057) marked TOP.
- crosscheck I: five exterior connectors (rear USB-C + HDMI, 2x front USB-A, top USB-A),
  eMMC/USB2422 must be absent, all three ports on the hub. PASS. ERC 0/0, pin review and
  pin/function matrix PASS, R10_HOST_CHECKS_PASS.
- PCB regenerated: Ø 119.8 mm, DRC 0 errors (unrouted), top cartridge at (-9.3, 24.2) mm.
- DECISIONS D12 (supersedes D10 and the four-connector rule); change-order report sections
  1, 2, 4, 5, 6 and the mechanical note updated; CLAUDE.md topology line amended.

Co-Authored-By: Claude Opus 5.5 <noreply@anthropic.com>
Claude-Session: https://claude.ai/code/session_01UkiuLdbjDvK75uDzAPKsGs
Parts:
- removed R179: 1k, Resistor_SMD:R_0402_1005Metric
- removed R180: 2k, Resistor_SMD:R_0402_1005Metric
- removed TP74: EMMC_CMD, TestPoint:TestPoint_Pad_D1.0mm
- removed TP75: EMMC_D0, TestPoint:TestPoint_Pad_D1.0mm
- added D10: 3V3, LED_SMD:LED_0603_1608Metric, F.Cu at (130.7, 133.6)
- added J18: F133 UART0, Connector_PinHeader_2.54mm:PinHeader_1x03_P2.54mm_Vertical, F.Cu at (127.6, 125.5)
- added U45: APS3204L-3SQNA-SN, Package_SO:SOIC-8_3.9x4.9mm_P1.27mm, F.Cu at (120.3, 124.0)
- C107, C109, C113, C243: value 1uF -> 100nF
- C111: value 18pF -> 100nF
- C112: value 18pF -> 4.7uF; footprint Capacitor_SMD:C_0402_1005Metric -> Capacitor_SMD:C_0603_1608Metric
- C114: value 100uF -> 100nF; footprint Capacitor_SMD:C_1210_3225Metric -> Capacitor_SMD:C_0402_1005Metric; moved to B.Cu
- C115: value 22uF -> 18pF; footprint Capacitor_SMD:C_0805_2012Metric -> Capacitor_SMD:C_0402_1005Metric; moved to B.Cu
- C116: value 100nF -> 18pF
- C121: value 10pF -> 1uF
- C122: value 10uF -> 100uF; footprint Capacitor_SMD:C_0603_1608Metric -> Capacitor_SMD:C_1210_3225Metric; moved to F.Cu
- C123: value 100nF -> 22uF; footprint Capacitor_SMD:C_0402_1005Metric -> Capacitor_SMD:C_0805_2012Metric; moved to F.Cu
- C125, C143, C244: value 100nF -> 1uF
- C126: value 100nF -> 100uF; footprint Capacitor_SMD:C_0402_1005Metric -> Capacitor_SMD:C_1210_3225Metric; moved to F.Cu
- C127: value 10uF -> 22uF; footprint Capacitor_SMD:C_0603_1608Metric -> Capacitor_SMD:C_0805_2012Metric; moved to F.Cu
- C129: value 100nF -> 10pF
- C130, C139, C167, C168, C169, C174, C193, C194, C195, C196, C197, C198, C199, C219, C220, C225, C235, C237: value 100nF -> 10uF; footprint Capacitor_SMD:C_0402_1005Metric -> Capacitor_SMD:C_0603_1608Metric
- C131, C159, C160, C161, C166, C185, C186, C187, C188, C189, C190, C191, C203, C204, C217, C227, C228, C229, C241: value 10uF -> 100nF; footprint Capacitor_SMD:C_0603_1608Metric -> Capacitor_SMD:C_0402_1005Metric
- C135, C236: value 1uF -> 10uF; footprint Capacitor_SMD:C_0402_1005Metric -> Capacitor_SMD:C_0603_1608Metric
- C242: value 4.7uF -> 100nF; footprint Capacitor_SMD:C_0603_1608Metric -> Capacitor_SMD:C_0402_1005Metric
- D5: value 45F LED -> SMF5.0A; footprint LED_SMD:LED_0603_1608Metric -> Diode_SMD:D_SMF
- D6: value 12F LED -> 45F LED
- D7: value STATUS -> 12F LED
- D8: value ERROR -> STATUS
- D9: value 3V3 -> ERROR
- J13: value USB-A Player 2 / game load -> USB-A Player 2
- J14: value HDMI type-A -> USB-A game cartridge; footprint Connector_Video:HDMI_A_Molex_208658-1001_Horizontal -> Connector_USB:USB_A_Molex_105057_Vertical
- J15: value 45F JTAG -> HDMI type-A; footprint Connector_PinHeader_1.27mm:PinHeader_2x05_P1.27mm_Vertical_SMD -> Connector_Video:HDMI_A_Molex_208658-1001_Horizontal
- J16: value 12F JTAG -> 45F JTAG
- J17: value F133 UART0 -> 12F JTAG; footprint Connector_PinHeader_2.54mm:PinHeader_1x03_P2.54mm_Vertical -> Connector_PinHeader_1.27mm:PinHeader_2x05_P1.27mm_Vertical_SMD
- R106, R107, R143, R144, R169: value 100k -> 22R
- R108, R109: value 0R -> 22R
- R110, R145: value 33R -> 22R
- R111, R172, R68, R69, R70, R74: value 10k -> 100k
- R113, R114: value 100k -> 0R
- R115, R150: value 4.7k -> 33R
- R116, R151: value 470R -> 10k
- R117, R118, R119, R153, R154: value 4.7k -> 100k
- R121: value 10k -> 470R
- R122, R128, R163: value 1k -> 4.7k
- R126, R152: value 4.7k -> 10k
- R127: value 33R -> 1k
- R129, R131, R164: value 22R -> 4.7k
- R130, R165: value 10k -> 4.7k
- R132: value 22R -> 33R
- R133: value 22R -> 1k
- R135, R77, R78, R93, R96, R97: value 22R -> 10k
- R146, R147, R80, R81, R82, R83: value 10k -> 22R
- R156: value 1k -> 470R
- R161: value 4.7k -> 1k
- R162: value 33R -> 4.7k
- R166: value 100k -> 4.7k
- R167: value 100k -> 33R
- R168: value 100k -> 1k
- R170, R71, R72: value 100k -> 10k
- R171: value 33R -> 100k
- R173, R174, R175: value 47k -> 100k
- R176: value 47k -> 1k
- R177: value 10k -> 1k
- R178: value 1k -> 2k
- R75, R76: value 22R -> 100k
- R79: value 887R -> 10k
- R84: value 10k -> 887R
- R86: value 0R -> 10k
- R89, R90: value 2.2k -> 10k
- R91: value 10k -> 0R
- R94, R95: value 22R -> 2.2k
- TP48: value USB0_SEL -> USBA3_VBUS
- TP49: value HUB_RESET_N -> USB0_SEL
- TP50: value HUB_UP_DP -> HUB_RESET_N
- TP51: value HUB_UP_DM -> HUB_UP_DP
- TP52: value LCD_DCLK -> HUB_UP_DM
- TP53: value HDMI_HPD -> LCD_DCLK
- TP54: value HDMI_INT -> HDMI_HPD
- TP55: value HDMI_5V -> HDMI_INT
- TP56: value I2S_BCLK -> HDMI_5V
- TP57: value I2S_LRCK -> I2S_BCLK
- TP58: value G_TXCK -> I2S_LRCK
- TP59: value G_RXCK -> G_TXCK
- TP60: value G_CLKIN -> G_RXCK
- TP61: value FPGA45_DONE -> G_CLKIN
- TP62: value FPGA45_PROGRAMN -> FPGA45_DONE
- TP63: value FPGA45_INITN -> FPGA45_PROGRAMN
- TP64: value FPGA45_SCK -> FPGA45_INITN
- TP65: value F45_OSC_25M -> FPGA45_SCK
- TP66: value SDR_CLK -> F45_OSC_25M
- TP67: value ETH_TXCK -> SDR_CLK
- TP68: value ETH_RXCK -> ETH_TXCK
- TP69: value FPGA12_DONE -> ETH_RXCK
- TP70: value FPGA12_PROGRAMN -> FPGA12_DONE
- TP71: value FPGA12_INITN -> FPGA12_PROGRAMN
- TP72: value FPGA12_SCK -> FPGA12_INITN
- TP73: value EMMC_CLK -> FPGA12_SCK
- U26: value USB2422-I/MJ -> USB2514B-I/M2; footprint Package_DFN_QFN:QFN-24-1EP_4x4mm_P0.5mm_EP2.6x2.6mm_ThermalVias -> Package_DFN_QFN:QFN-36-1EP_6x6mm_P0.5mm_EP3.7x3.7mm_ThermalVias
- U31: value ADV7513BSWZ -> USB-A3 power; footprint Package_QFP:LQFP-64-1EP_10x10mm_P0.5mm_EP5x5mm_ThermalVias -> Package_TO_SOT_SMD:SOT-23-5
- U32: value TPD12S016 -> TPD2EUSB30; footprint Package_SO:TSSOP-24_4.4x7.8mm_P0.65mm -> ARC1_R10:SLIM4_FP_U11_TPD2EUSB30_DRT3
- U33: value LFE5U-45F-6BG381C -> ADV7513BSWZ; footprint Package_BGA:Lattice_caBGA-381_17x17mm_Layout20x20_P0.8mm -> Package_QFP:LQFP-64-1EP_10x10mm_P0.5mm_EP5x5mm_ThermalVias
- U34: value iso FPGA45_SCK_B -> TPD12S016; footprint Package_TO_SOT_SMD:SOT-353_SC-70-5 -> Package_SO:TSSOP-24_4.4x7.8mm_P0.65mm
- U35: value iso FPGA45_MOSI -> LFE5U-45F-6BG381C; footprint Package_TO_SOT_SMD:SOT-353_SC-70-5 -> Package_BGA:Lattice_caBGA-381_17x17mm_Layout20x20_P0.8mm
- U36: value iso FPGA45_SS_N -> iso FPGA45_SCK_B
- U37: value AS4C16M16SA-6TIN -> iso FPGA45_MOSI; footprint Package_SO:TSOP-II-54_22.2x10.16mm_P0.8mm -> Package_TO_SOT_SMD:SOT-353_SC-70-5
- U38: value LFE5U-12F-6TG144C -> iso FPGA45_SS_N; footprint Package_QFP:TQFP-144_20x20mm_P0.5mm -> Package_TO_SOT_SMD:SOT-353_SC-70-5
- U39: value iso SCK -> AS4C16M16SA-6TIN; footprint Package_TO_SOT_SMD:SOT-353_SC-70-5 -> Package_SO:TSOP-II-54_22.2x10.16mm_P0.8mm
- U40: value iso MOSI -> LFE5U-12F-6TG144C; footprint Package_TO_SOT_SMD:SOT-353_SC-70-5 -> Package_QFP:TQFP-144_20x20mm_P0.5mm
- U41: value iso SS -> iso SCK
- U42: value iso MISO -> iso MOSI
- U43: value APS3204L-3SQNA-SN -> iso SS; footprint Package_SO:SOIC-8_3.9x4.9mm_P1.27mm -> Package_TO_SOT_SMD:SOT-353_SC-70-5
- U44: value KLMAG1JETD-B041 -> iso MISO; footprint Package_BGA:LFBGA-153_11.5x13mm_Layout14x14_P0.5mm -> Package_TO_SOT_SMD:SOT-353_SC-70-5
- moved J14 71.0 mm to (139.2, 129.2), turned to 0 degrees
- moved C112 70.8 mm to (136.2, 133.6)
- moved C113 70.3 mm to (137.9, 131.9)
- moved C111 68.4 mm to (135.6, 131.9)
- moved C69 67.5 mm to (201.4, 103.6)
- moved C114 66.7 mm to (140.3, 131.9), turned to 180 degrees
- moved TP51 66.6 mm to (135.7, 138.3)
- moved D9 66.4 mm to (127.3, 133.6)
- moved U29 65.8 mm to (136.8, 136.9)
- moved C121 65.2 mm to (151.8, 131.9)
- moved U32 64.7 mm to (151.4, 139.7)
- moved R64 64.7 mm to (139.1, 133.3)
- moved R65 64.7 mm to (141.5, 133.3)
- moved R66 64.7 mm to (143.8, 133.3)
- moved R74 64.3 mm to (135.7, 135.3)
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Connections:
- C109 pad 1: HUB_CRFILT -> 3V3
- C110 pad 1: HUB_PLLFILT -> 3V3
- C111 pad 1: HUB_XI -> 3V3
- C112 pad 1: HUB_XO -> 3V3
- C113 pad 1: VBUS_5V -> HUB_CRFILT
- C114 pad 1: USBA1_VBUS -> HUB_PLLFILT
- C115 pad 1: USBA1_VBUS -> HUB_XI
- C116 pad 1: USBA1_VBUS -> HUB_XO
- C118 pad 1: USBA2_VBUS -> USBA1_VBUS
- C119 pad 1: USBA2_VBUS -> USBA1_VBUS
- C120 pad 1: USBA2_VBUS -> USBA1_VBUS
- C121 pad 1: LCD_DCLK -> VBUS_5V
- C122 pad 1: 1V8_ADV_D -> USBA2_VBUS
- C123 pad 1: 1V8_ADV_D -> USBA2_VBUS
- C124 pad 1: 1V8_ADV_D -> USBA2_VBUS
- C125 pad 1: 1V8_ADV_D -> VBUS_5V
- C126 pad 1: 1V8_ADV_D -> USBA3_VBUS
- C127 pad 1: 1V8_ADV_A -> USBA3_VBUS
- C128 pad 1: 1V8_ADV_A -> USBA3_VBUS
- C129 pad 1: 1V8_ADV_A -> LCD_DCLK
- C130 pad 1: 1V8_ADV_A -> 1V8_ADV_D
- C131 pad 1: 1V8_ADV_P -> 1V8_ADV_D
- C132 pad 1: 1V8_ADV_P -> 1V8_ADV_D
- C133 pad 1: 1V8_ADV_P -> 1V8_ADV_D
- C134 pad 1: 3V3 -> 1V8_ADV_D
- C135 pad 1: 3V3 -> 1V8_ADV_A
- C136 pad 1: 3V3 -> 1V8_ADV_A
- C137 pad 1: VBUS_5V -> 1V8_ADV_A
- C138 pad 1: HDMI_5V -> 1V8_ADV_A
- C139 pad 1: 1V1_F45 -> 1V8_ADV_P
- C140 pad 1: 1V1_F45 -> 1V8_ADV_P
- C141 pad 1: 1V1_F45 -> 1V8_ADV_P
- C142 pad 1: 1V1_F45 -> 3V3
- C143 pad 1: 1V1_F45 -> 3V3
- C144 pad 1: 1V1_F45 -> 3V3
- C145 pad 1: 1V1_F45 -> VBUS_5V
- C146 pad 1: 1V1_F45 -> HDMI_5V
- C162 pad 1: 2V5_F45 -> 1V1_F45
- C163 pad 1: 2V5_F45 -> 1V1_F45
- C164 pad 1: 2V5_F45 -> 1V1_F45
- C165 pad 1: 2V5_F45 -> 1V1_F45
- C166 pad 1: 2V5_F45 -> 1V1_F45
- C167 pad 1: 3V3_F45 -> 1V1_F45
- C168 pad 1: 3V3_F45 -> 1V1_F45
- C169 pad 1: 3V3_F45 -> 1V1_F45
- C170 pad 1: 3V3_F45 -> 2V5_F45
- C171 pad 1: 3V3_F45 -> 2V5_F45
- C172 pad 1: 3V3_F45 -> 2V5_F45
- C173 pad 1: 3V3_F45 -> 2V5_F45
- C174 pad 1: 3V3_F45 -> 2V5_F45
- C205 pad 1: 1V1_F12 -> 3V3_F45
- C206 pad 1: 1V1_F12 -> 3V3_F45
- C207 pad 1: 1V1_F12 -> 3V3_F45
- C208 pad 1: 1V1_F12 -> 3V3_F45
- C209 pad 1: 1V1_F12 -> 3V3_F45
- C210 pad 1: 1V1_F12 -> 3V3_F45
- C211 pad 1: 1V1_F12 -> 3V3_F45
- C212 pad 1: 1V1_F12 -> 3V3_F45
- C213 pad 1: 2V5_F12 -> 1V1_F12
- C214 pad 1: 2V5_F12 -> 1V1_F12
- C215 pad 1: 2V5_F12 -> 1V1_F12
- C216 pad 1: 2V5_F12 -> 1V1_F12
- C217 pad 1: 2V5_F12 -> 1V1_F12
- C218 pad 1: 3V3_F12 -> 1V1_F12
- C219 pad 1: 3V3_F12 -> 1V1_F12
- C220 pad 1: 3V3_F12 -> 1V1_F12
- C221 pad 1: 3V3_F12 -> 2V5_F12
- C222 pad 1: 3V3_F12 -> 2V5_F12
- C223 pad 1: 3V3_F12 -> 2V5_F12
- C224 pad 1: 3V3_F12 -> 2V5_F12
- C225 pad 1: 3V3_F12 -> 2V5_F12
- C233 pad 1: 3V3 -> 3V3_F12
- C237 pad 1: 3V3 -> 3V3_F12
- C238 pad 1: 3V3 -> 3V3_F12
- C239 pad 1: 3V3 -> 3V3_F12
- C240 pad 1: 3V3 -> 3V3_F12
- C242 pad 1: 3V3 -> 3V3_F12
- C243 pad 1: EMMC_VDDI -> 3V3_F12
- C244 pad 1: EMMC_VDDI -> 3V3_F12
- D5 pad 1: GND -> USBA3_VBUS
- D5 pad 2: F45_LED0_R -> GND
- D6 pad 2: F12_LED0_R -> F45_LED0_R
- D7 pad 2: LED_STATUS_R -> F12_LED0_R
- D8 pad 2: LED_ERROR_R -> LED_STATUS_R
- D9 pad 2: LED_3V3_R -> LED_ERROR_R
- J14 pad 1: TMDS_D2_P -> USBA3_VBUS
- J14 pad 2: GND -> USBA3_DM
- J14 pad 3: TMDS_D2_N -> USBA3_DP
- J14 pad 4: TMDS_D1_P -> GND
- J15 pad 1: 3V3_F45 -> TMDS_D2_P
- J15 pad 10: FPGA45_PROGRAMN -> TMDS_CK_P
- J15 pad 2: FPGA45_TMS -> GND
- J15 pad 3: GND -> TMDS_D2_N
- J15 pad 4: FPGA45_TCK -> TMDS_D1_P
- J15 pad 6: FPGA45_TDO -> TMDS_D1_N
- J15 pad 7: (no net) -> TMDS_D0_P
- J15 pad 8: FPGA45_TDI -> GND
- J15 pad 9: GND -> TMDS_D0_N
- J16 pad 1: 3V3_F12 -> 3V3_F45
- J16 pad 10: FPGA12_PROGRAMN -> FPGA45_PROGRAMN
- J16 pad 2: FPGA12_TMS -> FPGA45_TMS
- J16 pad 4: FPGA12_TCK -> FPGA45_TCK
- J16 pad 6: FPGA12_TDO -> FPGA45_TDO
- J16 pad 8: FPGA12_TDI -> FPGA45_TDI
- J17 pad 1: GND -> 3V3_F12
- J17 pad 2: UART0_TX -> FPGA12_TMS
- J17 pad 3: UART0_RX -> GND
- R100 pad 1: G_RXD0_F -> G_TXD1_D
- R100 pad 2: G_RXD0 -> G_TXD1
- R101 pad 1: G_RXD1_F -> G_TXD2_D
- R101 pad 2: G_RXD1 -> G_TXD2
- R102 pad 1: G_RXD2_F -> G_TXD3_D
- R102 pad 2: G_RXD2 -> G_TXD3
- R103 pad 1: G_RXD3_F -> G_TXCTL_D
- R103 pad 2: G_RXD3 -> G_TXCTL
- R104 pad 1: G_RXCTL_F -> G_RXCK_F
- R104 pad 2: G_RXCTL -> G_RXCK
- R105 pad 1: G_CLKIN_F -> G_RXD0_F
- R105 pad 2: G_CLKIN -> G_RXD0
- R106 pad 1: G_TXCTL -> G_RXD1_F
- R106 pad 2: GND -> G_RXD1
- R107 pad 1: G_RXCTL -> G_RXD2_F
- R107 pad 2: GND -> G_RXD2
- R108 pad 1: G_RXCK -> G_RXD3_F
- R108 pad 2: G_CLKIN -> G_RXD3
- R109 pad 1: G_CLKIN_OSC -> G_RXCTL_F
- R109 pad 2: G_CLKIN -> G_RXCTL
- R110 pad 1: FPGA45_SCK_B -> G_CLKIN_F
- R110 pad 2: FPGA45_SCK -> G_CLKIN
- R111 pad 1: FPGA45_SS_N_D -> G_TXCTL
- R111 pad 2: 3V3 -> GND
- R112 pad 1: FPGA45_SCK_D -> G_RXCTL
- R113 pad 1: FPGA45_MOSI_D -> G_RXCK
- R113 pad 2: GND -> G_CLKIN
- R114 pad 1: FPGA45_MISO -> G_CLKIN_OSC
- R114 pad 2: GND -> G_CLKIN
- R115 pad 1: FPGA45_PROGRAMN -> FPGA45_SCK_B
- R115 pad 2: 3V3_F45 -> FPGA45_SCK
- R116 pad 1: FPGA45_PROGRAMN_D -> FPGA45_SS_N_D
- R116 pad 2: FPGA45_PROGRAMN -> 3V3
- R117 pad 1: FPGA45_INITN -> FPGA45_SCK_D
- R117 pad 2: 3V3_F45 -> GND
- R118 pad 1: FPGA45_DONE -> FPGA45_MOSI_D
- R118 pad 2: 3V3_F45 -> GND
- R119 pad 1: FPGA45_SS_N -> FPGA45_MISO
- R119 pad 2: 3V3_F45 -> GND
- R120 pad 1: FPGA45_CFG0 -> FPGA45_PROGRAMN
- R121 pad 1: FPGA45_HOLDN -> FPGA45_PROGRAMN_D
- R121 pad 2: 3V3_F45 -> FPGA45_PROGRAMN
- R122 pad 1: FPGA45_SCK -> FPGA45_INITN
- R123 pad 1: FPGA45_TCK -> FPGA45_DONE
- R123 pad 2: GND -> 3V3_F45
- R124 pad 1: FPGA45_TMS -> FPGA45_SS_N
- R125 pad 1: FPGA45_TDI -> FPGA45_CFG0
- R126 pad 1: FPGA45_TDO -> FPGA45_HOLDN
- R127 pad 1: F45_OSC_25M_X -> FPGA45_SCK
- R127 pad 2: F45_OSC_25M -> 3V3_F45
- R128 pad 1: F45_LED0 -> FPGA45_TCK
- R128 pad 2: F45_LED0_R -> GND
- R129 pad 1: SDR_CLK_F -> FPGA45_TMS
- R129 pad 2: SDR_CLK -> 3V3_F45
- R130 pad 1: SDR_CKE -> FPGA45_TDI
- R130 pad 2: GND -> 3V3_F45
- R131 pad 1: ETH_TXCK_F -> FPGA45_TDO
- R131 pad 2: ETH_TXCK -> 3V3_F45
- R132 pad 1: ETH_TXD0_F -> F45_OSC_25M_X
- R132 pad 2: ETH_TXD0 -> F45_OSC_25M
- R133 pad 1: ETH_TXD1_F -> F45_LED0
- R133 pad 2: ETH_TXD1 -> F45_LED0_R
- R134 pad 1: ETH_TXD2_F -> SDR_CLK_F
- R134 pad 2: ETH_TXD2 -> SDR_CLK
- R135 pad 1: ETH_TXD3_F -> SDR_CKE
- R135 pad 2: ETH_TXD3 -> GND
- R136 pad 1: ETH_TXCTL_F -> ETH_TXCK_F
- R136 pad 2: ETH_TXCTL -> ETH_TXCK
- R137 pad 1: ETH_RXCK_E -> ETH_TXD0_F
- R137 pad 2: ETH_RXCK -> ETH_TXD0
- R138 pad 1: ETH_RXD0_E -> ETH_TXD1_F
- R138 pad 2: ETH_RXD0 -> ETH_TXD1
- R139 pad 1: ETH_RXD1_E -> ETH_TXD2_F
- R139 pad 2: ETH_RXD1 -> ETH_TXD2
- R140 pad 1: ETH_RXD2_E -> ETH_TXD3_F
- R140 pad 2: ETH_RXD2 -> ETH_TXD3
- R141 pad 1: ETH_RXD3_E -> ETH_TXCTL_F
- R141 pad 2: ETH_RXD3 -> ETH_TXCTL
- R142 pad 1: ETH_RXCTL_E -> ETH_RXCK_E
- R142 pad 2: ETH_RXCTL -> ETH_RXCK
- R143 pad 1: ETH_TXCTL -> ETH_RXD0_E
- R143 pad 2: GND -> ETH_RXD0
- R144 pad 1: ETH_RXCTL -> ETH_RXD1_E
- R144 pad 2: GND -> ETH_RXD1
- R145 pad 1: FPGA12_SCK_B -> ETH_RXD2_E
- R145 pad 2: FPGA12_SCK -> ETH_RXD2
- R146 pad 1: FPGA12_BUS_EN_N -> ETH_RXD3_E
- R146 pad 2: 3V3 -> ETH_RXD3
- R147 pad 1: FPGA12_SS_N_F -> ETH_RXCTL_E
- R147 pad 2: 3V3 -> ETH_RXCTL
- R148 pad 1: FPGA12_MOSI -> ETH_TXCTL
- R149 pad 1: FPGA12_MISO -> ETH_RXCTL
- R150 pad 1: FPGA12_PROGRAMN -> FPGA12_SCK_B
- R150 pad 2: 3V3_F12 -> FPGA12_SCK
- R151 pad 1: FPGA12_PROGRAMN_F -> FPGA12_BUS_EN_N
- R151 pad 2: FPGA12_PROGRAMN -> 3V3
- R152 pad 1: FPGA12_INITN -> FPGA12_SS_N_F
- R152 pad 2: 3V3_F12 -> 3V3
- R153 pad 1: FPGA12_DONE -> FPGA12_MOSI
- R153 pad 2: 3V3_F12 -> GND
- R154 pad 1: FPGA12_SS_N -> FPGA12_MISO
- R154 pad 2: 3V3_F12 -> GND
- R155 pad 1: FPGA12_CFG0 -> FPGA12_PROGRAMN
- R156 pad 1: FPGA12_SCK -> FPGA12_PROGRAMN_F
- R156 pad 2: 3V3_F12 -> FPGA12_PROGRAMN
- R157 pad 1: FPGA12_TCK -> FPGA12_INITN
- R157 pad 2: GND -> 3V3_F12
- R158 pad 1: FPGA12_TMS -> FPGA12_DONE
- R159 pad 1: FPGA12_TDI -> FPGA12_SS_N
- R160 pad 1: FPGA12_TDO -> FPGA12_CFG0
- R161 pad 1: FPGA12_IRQ_N -> FPGA12_SCK
- R162 pad 1: F12_OSC_25M_X -> FPGA12_TCK
- R162 pad 2: F12_OSC_25M -> GND
- R163 pad 1: F12_LED0 -> FPGA12_TMS
- R163 pad 2: F12_LED0_R -> 3V3_F12
- R164 pad 1: PSRAM_SCLK_F -> FPGA12_TDI
- R164 pad 2: PSRAM_SCLK -> 3V3_F12
- R165 pad 1: PSRAM_CE_N -> FPGA12_TDO
- R166 pad 1: PSRAM_SCLK -> FPGA12_IRQ_N
- R166 pad 2: GND -> 3V3_F12
- R167 pad 1: PSRAM_SIO0 -> F12_OSC_25M_X
- R167 pad 2: GND -> F12_OSC_25M
- R168 pad 1: PSRAM_SIO1 -> F12_LED0
- R168 pad 2: GND -> F12_LED0_R
- R169 pad 1: PSRAM_SIO2 -> PSRAM_SCLK_F
- R169 pad 2: GND -> PSRAM_SCLK
- R170 pad 1: PSRAM_SIO3 -> PSRAM_CE_N
- R170 pad 2: GND -> 3V3_F12
- R171 pad 1: EMMC_CLK_F -> PSRAM_SCLK
- R171 pad 2: EMMC_CLK -> GND
- R172 pad 1: EMMC_CMD -> PSRAM_SIO0
- R172 pad 2: 3V3 -> GND
- R173 pad 1: EMMC_D0 -> PSRAM_SIO1
- R173 pad 2: 3V3 -> GND
- R174 pad 1: EMMC_D1 -> PSRAM_SIO2
- R174 pad 2: 3V3 -> GND
- R175 pad 1: EMMC_D2 -> PSRAM_SIO3
- R175 pad 2: 3V3 -> GND
- R176 pad 1: EMMC_D3 -> LED_STATUS
- R176 pad 2: 3V3 -> LED_STATUS_R
- R177 pad 1: EMMC_RST_N -> LED_ERROR
- R177 pad 2: 3V3 -> LED_ERROR_R
- R178 pad 1: LED_STATUS -> 3V3
- R178 pad 2: LED_STATUS_R -> LED_3V3_R
- R67 pad 1: HUB_CFG_SEL -> HUB_CFG_SEL0
- R68 pad 1: HUB_NON_REM1 -> HUB_CFG_SEL1
- R69 pad 1: HUB_NON_REM0 -> HUB_NON_REM1
- R70 pad 1: HUB_RESET_N -> HUB_NON_REM0
- R71 pad 1: HUB_PRTPWR1 -> HUB_DN4_DIS
- R71 pad 2: GND -> 3V3
- R72 pad 1: HUB_PRTPWR2 -> HUB_OCS4_N
- R72 pad 2: GND -> 3V3
- R73 pad 1: HUB_OCS1_N -> HUB_RESET_N
- R73 pad 2: 3V3 -> GND
- R74 pad 1: HUB_OCS2_N -> HUB_PRTPWR1
- R74 pad 2: 3V3 -> GND
- R75 pad 1: LCD_DCLK_D -> HUB_PRTPWR2
- R75 pad 2: LCD_DCLK -> GND
- R76 pad 1: LCD_HS_D -> HUB_PRTPWR3
- R76 pad 2: LCD_HS -> GND
- R77 pad 1: LCD_VS_D -> HUB_OCS1_N
- R77 pad 2: LCD_VS -> 3V3
- R78 pad 1: LCD_DE_D -> HUB_OCS2_N
- R78 pad 2: LCD_DE -> 3V3
- R79 pad 1: ADV_REXT -> HUB_OCS3_N
- R79 pad 2: GND -> 3V3
- R80 pad 1: ADV_SPDIF -> LCD_DCLK_D
- R80 pad 2: GND -> LCD_DCLK
- R81 pad 1: ADV_MCLK -> LCD_HS_D
- R81 pad 2: GND -> LCD_HS
- R82 pad 1: ADV_I2S1 -> LCD_VS_D
- R82 pad 2: GND -> LCD_VS
- R83 pad 1: ADV_I2S2 -> LCD_DE_D
- R83 pad 2: GND -> LCD_DE
- R84 pad 1: ADV_I2S3 -> ADV_REXT
- R85 pad 1: ADV_CEC_CLK -> ADV_SPDIF
- R86 pad 1: ADV_CEC_CLK_X -> ADV_MCLK
- R86 pad 2: ADV_CEC_CLK -> GND
- R87 pad 1: HDMI_PD -> ADV_I2S1
- R88 pad 1: HDMI_INT -> ADV_I2S2
- R88 pad 2: 3V3 -> GND
- R89 pad 1: HDMI_I2C_SCL -> ADV_I2S3
- R89 pad 2: 3V3 -> GND
- R90 pad 1: HDMI_I2C_SDA -> ADV_CEC_CLK
- R90 pad 2: 3V3 -> GND
- R91 pad 1: TPD_LS_OE -> ADV_CEC_CLK_X
- R91 pad 2: 3V3 -> ADV_CEC_CLK
- R92 pad 1: TPD_CT_HPD -> HDMI_PD
- R92 pad 2: 3V3 -> GND
- R93 pad 1: G_TXCK_D -> HDMI_INT
- R93 pad 2: G_TXCK -> 3V3
- R94 pad 1: G_TXD0_D -> HDMI_I2C_SCL
- R94 pad 2: G_TXD0 -> 3V3
- R95 pad 1: G_TXD1_D -> HDMI_I2C_SDA
- R95 pad 2: G_TXD1 -> 3V3
- R96 pad 1: G_TXD2_D -> TPD_LS_OE
- R96 pad 2: G_TXD2 -> 3V3
- R97 pad 1: G_TXD3_D -> TPD_CT_HPD
- R97 pad 2: G_TXD3 -> 3V3
- R98 pad 1: G_TXCTL_D -> G_TXCK_D
- R98 pad 2: G_TXCTL -> G_TXCK
- R99 pad 1: G_RXCK_F -> G_TXD0_D
- R99 pad 2: G_RXCK -> G_TXD0
- TP48 pad 1: USB0_SEL -> USBA3_VBUS
- TP49 pad 1: HUB_RESET_N -> USB0_SEL
- TP50 pad 1: HUB_UP_DP -> HUB_RESET_N
- TP51 pad 1: HUB_UP_DM -> HUB_UP_DP
- TP52 pad 1: LCD_DCLK -> HUB_UP_DM
- TP53 pad 1: HDMI_HPD -> LCD_DCLK
- TP54 pad 1: HDMI_INT -> HDMI_HPD
- TP55 pad 1: HDMI_5V -> HDMI_INT
- TP56 pad 1: I2S_BCLK -> HDMI_5V
- TP57 pad 1: I2S_LRCK -> I2S_BCLK
- TP58 pad 1: G_TXCK -> I2S_LRCK
- TP59 pad 1: G_RXCK -> G_TXCK
- TP60 pad 1: G_CLKIN -> G_RXCK
- TP61 pad 1: FPGA45_DONE -> G_CLKIN
- TP62 pad 1: FPGA45_PROGRAMN -> FPGA45_DONE
- TP63 pad 1: FPGA45_INITN -> FPGA45_PROGRAMN
- TP64 pad 1: FPGA45_SCK -> FPGA45_INITN
- TP65 pad 1: F45_OSC_25M -> FPGA45_SCK
- TP66 pad 1: SDR_CLK -> F45_OSC_25M
- TP67 pad 1: ETH_TXCK -> SDR_CLK
- TP68 pad 1: ETH_RXCK -> ETH_TXCK
- TP69 pad 1: FPGA12_DONE -> ETH_RXCK
- TP70 pad 1: FPGA12_PROGRAMN -> FPGA12_DONE
- TP71 pad 1: FPGA12_INITN -> FPGA12_PROGRAMN
- TP72 pad 1: FPGA12_SCK -> FPGA12_INITN
- TP73 pad 1: EMMC_CLK -> FPGA12_SCK
- U18 pad 10: EMMC_CMD -> (no net)
- U18 pad 11: EMMC_D3 -> (no net)
- U18 pad 12: EMMC_D2 -> (no net)
- U18 pad 13: EMMC_RST_N -> (no net)
- U18 pad 7: EMMC_D1 -> (no net)
- U18 pad 8: EMMC_D0 -> (no net)
- U18 pad 9: EMMC_CLK_F -> (no net)
- U26 pad 1: 3V3 -> USBA1_DM
- U26 pad 10: HUB_CRFILT -> 3V3
- U26 pad 11: HUB_PRTPWR2 -> GND
- U26 pad 12: HUB_OCS2_N -> HUB_PRTPWR1
- U26 pad 13: HUB_NON_REM1 -> HUB_OCS1_N
- U26 pad 14: HUB_CFG_SEL -> HUB_CRFILT
- U26 pad 15: HUB_RESET_N -> 3V3
- U26 pad 16: 3V3 -> HUB_PRTPWR2
- U26 pad 17: HUB_NON_REM0 -> HUB_OCS2_N
- U26 pad 18: 3V3 -> HUB_PRTPWR3
- U26 pad 19: HUB_UP_DM -> HUB_OCS3_N
- U26 pad 2: USBA1_DM -> USBA1_DP
- U26 pad 20: HUB_UP_DP -> (no net)
- U26 pad 21: HUB_XO -> HUB_OCS4_N
- U26 pad 22: HUB_XI -> HUB_NON_REM1
- U26 pad 23: HUB_PLLFILT -> 3V3
- U26 pad 24: HUB_RBIAS -> HUB_CFG_SEL0
- U26 pad 25: GND -> HUB_CFG_SEL1
- U26 pad 3: USBA1_DP -> USBA2_DM
- U26 pad 4: USBA2_DM -> USBA2_DP
- U26 pad 5: USBA2_DP -> 3V3
- U26 pad 6: (no net) -> USBA3_DM
- U26 pad 7: HUB_PRTPWR1 -> USBA3_DP
- U26 pad 8: HUB_OCS1_N -> HUB_DN4_DIS
- U26 pad 9: 3V3 -> HUB_DN4_DIS
- U31 pad 1: 1V8_ADV_D -> USBA3_VBUS
- U31 pad 2: LCD_VS -> GND
- U31 pad 3: ADV_SPDIF -> HUB_OCS3_N
- U31 pad 4: ADV_MCLK -> HUB_PRTPWR3
- U31 pad 5: I2S_DOUT -> VBUS_5V
- U32 pad 1: HDMI_CEC_A -> USBA3_DP
- U32 pad 2: HDMI_DDC_SCL -> USBA3_DM
- U32 pad 3: HDMI_DDC_SDA -> GND
- U34 pad 1: GND -> HDMI_CEC_A
- U34 pad 2: FPGA45_SCK_D -> HDMI_DDC_SCL
- U34 pad 3: GND -> HDMI_DDC_SDA
- U34 pad 4: FPGA45_SCK_B -> HDMI_HPD
- U34 pad 5: 3V3_F45 -> TPD_LS_OE
- U36 pad 2: FPGA45_SS_N_D -> FPGA45_SCK_D
- U36 pad 4: FPGA45_SS_N -> FPGA45_SCK_B
- U37 pad 1: 3V3_F45 -> GND
- U37 pad 2: SDR_DQ0 -> FPGA45_MOSI_D
- U37 pad 3: 3V3_F45 -> GND
- U37 pad 4: SDR_DQ1 -> FPGA45_MOSI
- U37 pad 5: SDR_DQ2 -> 3V3_F45
- U38 pad 1: (no net) -> GND
- U38 pad 2: (no net) -> FPGA45_SS_N_D
- U38 pad 3: (no net) -> GND
- U38 pad 4: (no net) -> FPGA45_SS_N
- U38 pad 5: (no net) -> 3V3_F45
- U39 pad 1: FPGA12_BUS_EN_N -> 3V3_F45
- U39 pad 2: SPI0_CLK -> SDR_DQ0
- U39 pad 3: GND -> 3V3_F45
- U39 pad 4: FPGA12_SCK_B -> SDR_DQ1
- U39 pad 5: 3V3_F12 -> SDR_DQ2
- U40 pad 1: FPGA12_BUS_EN_N -> (no net)
- U40 pad 2: SPI0_MOSI -> (no net)
- U40 pad 3: GND -> (no net)
- U40 pad 4: FPGA12_MOSI -> (no net)
- U40 pad 5: 3V3_F12 -> (no net)
- U41 pad 2: FPGA12_SS_N_F -> SPI0_CLK
- U41 pad 4: FPGA12_SS_N -> FPGA12_SCK_B
- U42 pad 1: FPGA12_SS_N_F -> FPGA12_BUS_EN_N
- U42 pad 2: FPGA12_MISO -> SPI0_MOSI
- U42 pad 4: SPI0_MISO -> FPGA12_MOSI
- U42 pad 5: 3V3 -> 3V3_F12
- U43 pad 1: PSRAM_CE_N -> FPGA12_BUS_EN_N
- U43 pad 2: PSRAM_SIO1 -> FPGA12_SS_N_F
- U43 pad 3: PSRAM_SIO2 -> GND
- U43 pad 4: GND -> FPGA12_SS_N
- U43 pad 5: PSRAM_SIO0 -> 3V3_F12
Other:
- board size 119.6 x 109.7 mm -> 119.8 x 110 mm
- board text added: "J15 HDMI_A REAR: plug insertion envelope keep-out in front of this face"
- board text removed: "J14 HDMI_A REAR: plug insertion envelope keep-out in front of this face"
