File: hardware/arc1-compact/R10_WORK/cad/video.kicad_sch (KiCad schematic)
At the start: 48 parts, among them J8 HDMI type-A, U24 TFP410PAP, U25 TPD12S016

Commit message: R10 change order rev 1.1: HDMI audio (ADV7513), USB0 role mux + hub + 2x front USB-A, eMMC, buttonless board
Owner handoff ARC1_R10_Handoff rev 1.1 (spec/, SHA-256 recorded) implemented in the generated schematic:
- D8 ADV7513BSWZ replaces the TFP410 (supersedes D6): D213 RGB888 video, D213 I2C2 init,
  F133 I2S2 -> HDMI embedded audio; own 1.8 V buck + 3 filtered domains; R_EXT 887R.
  D[23:0] pin order verified from the datasheet glyph coordinates.
- D9 F133 USB0 -> TS3USB221A (default rear USB-C device/FEL) or USB2422 hub -> two
  TPS2051C-switched front USB-A ports; F133 USB1 remains the internal D213 link; the D213
  recovery USB-C becomes internal fixture pads.
- D10 Samsung KLMAG1JETD-B041 16 GB eMMC on F133 SMHC0 (CONDITIONAL: SMHC0 documented for SD).
- D11 no switches: fixture pad pairs; game buttons, microSD and speakers removed.
- crosscheck_r10 section I (handoff go/no-go: 4 exterior connectors, 0 switches, I2S wired
  to the HDMI transmitter, USB0/USB1 roles, eMMC wiring) PASS; ERC 0/0; pin review PASS.
Sources: ADV7513 DS Rev B (LCSC copy), ADI AN-1270, Linux adv7511 driver, USB2422
DS00001726A, TPS20xxC SLVSAU6I, Samsung eMMC DS (not committed: vendor-confidential mark).

Co-Authored-By: Claude Opus 5.5 <noreply@anthropic.com>
Claude-Session: https://claude.ai/code/session_01UkiuLdbjDvK75uDzAPKsGs
Parts:
- removed C102: 10pF, Capacitor_SMD:C_0402_1005Metric, symbol ARC1_R10:C0402
- removed C103, C107, C110: 22uF, Capacitor_SMD:C_0805_2012Metric, symbol ARC1_R10:C0805
- removed C104, C105, C106, C108, C109, C111, C112, C113: 10nF, Capacitor_SMD:C_0402_1005Metric, symbol ARC1_R10:C0402
- removed C114, C115, C116: 100nF, Capacitor_SMD:C_0402_1005Metric, symbol ARC1_R10:C0402
- removed J8: HDMI type-A, Connector_Video:HDMI_A_Molex_208658-1001_Horizontal, symbol ARC1_R10:HDMI_A
- removed R64, R65, R66, R67: 22R, Resistor_SMD:R_0402_1005Metric, symbol ARC1_R10:R0402
- removed R68, R69, R70, R71, R72, R73, R74: 10k, Resistor_SMD:R_0402_1005Metric, symbol ARC1_R10:R0402
- removed TP46: LCD_DCLK, TestPoint:TestPoint_Pad_D1.0mm, symbol ARC1_R10:TP
- removed TP47: HDMI_HPD, TestPoint:TestPoint_Pad_D1.0mm, symbol ARC1_R10:TP
- removed TP48: TFP_MSEN, TestPoint:TestPoint_Pad_D1.0mm, symbol ARC1_R10:TP
- removed TP49: HDMI_5V, TestPoint:TestPoint_Pad_D1.0mm, symbol ARC1_R10:TP
- removed U24: TFP410PAP, Package_QFP:Texas_TQFP-64-1EP_10x10mm_P0.5mm_EP8x8mm_Mask4.44x4.44mm_ThermalVias, symbol ARC1_R10:TFP410
- removed U25: TPD12S016, Package_SO:TSSOP-24_4.4x7.8mm_P0.65mm, symbol ARC1_R10:TPD12S016
- added C121: 10pF, Capacitor_SMD:C_0402_1005Metric, symbol ARC1_R10:C0402
- added C122, C127, C131: 10uF, Capacitor_SMD:C_0603_1608Metric, symbol ARC1_R10:C0603
- added C123, C124, C125, C126, C128, C129, C130, C132, C133, C134, C136, C137, C138: 100nF, Capacitor_SMD:C_0402_1005Metric, symbol ARC1_R10:C0402
- added C135: 1uF, Capacitor_SMD:C_0402_1005Metric, symbol ARC1_R10:C0402
- added J14: HDMI type-A, Connector_Video:HDMI_A_Molex_208658-1001_Horizontal, symbol ARC1_R10:HDMI_A
- added R87, R88, R91, R92: 10k, Resistor_SMD:R_0402_1005Metric, symbol ARC1_R10:R0402
- added R89, R90: 2.2k, Resistor_SMD:R_0402_1005Metric, symbol ARC1_R10:R0402
- added TP52: LCD_DCLK, TestPoint:TestPoint_Pad_D1.0mm, symbol ARC1_R10:TP
- added TP53: HDMI_HPD, TestPoint:TestPoint_Pad_D1.0mm, symbol ARC1_R10:TP
- added TP54: HDMI_INT, TestPoint:TestPoint_Pad_D1.0mm, symbol ARC1_R10:TP
- added TP55: HDMI_5V, TestPoint:TestPoint_Pad_D1.0mm, symbol ARC1_R10:TP
- added TP56: I2S_BCLK, TestPoint:TestPoint_Pad_D1.0mm, symbol ARC1_R10:TP
- added TP57: I2S_LRCK, TestPoint:TestPoint_Pad_D1.0mm, symbol ARC1_R10:TP
- added U31: ADV7513BSWZ, Package_QFP:LQFP-64-1EP_10x10mm_P0.5mm_EP5x5mm_ThermalVias, symbol ARC1_R10:ADV7513
- added U32: TPD12S016, Package_SO:TSSOP-24_4.4x7.8mm_P0.65mm, symbol ARC1_R10:TPD12S016
- added X1: 12MHz, Oscillator:Oscillator_SMD_Abracon_ASE-4Pin_3.2x2.5mm, symbol ARC1_R10:OSC_3225
- FB3, FB4, FB5: Note (none) -> separate quiet 1.8 V domains (DS: DVDD 'filtered and as qui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
- R75, R77: value 10k -> 22R; LCSC C25744 -> C25092; MPN 0402WGF1002TCE -> 0402WGF220JTCE; Note DK step 000 (fitted) -> series R at the D213 (HW guide 4.7 item 3)
- R76, R78: value 10k -> 22R; LCSC C25744 -> C25092; MPN 0402WGF1002TCE -> 0402WGF220JTCE; Note trim option -> series R at the D213 (HW guide 4.7 item 3); now fitted
- R79: value 10k -> 887R; LCSC C25744 -> (none); MPN 0402WGF1002TCE -> (none); Manufacturer UNI-ROYAL -> (none); Note DK step 000 (fitted) -> 887 ohm 1 % close to pin 14 (ADV7513 HW user guide, quoted;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; Reuse SLIM4_R26_BOM_LINE (re-validate) -> (none)
- R80: Note trim option -> unused audio input held low; now fitted
- R81: Note TFP410 on by default (display works before any GPIO setup);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 -> unused audio input held low
- R82: value 4.7k -> 10k; LCSC C25900 -> C25744; MPN 0402WGF4701TCE -> 0402WGF1002TCE; Note SLDS145D: 5k pull-up required on MSEN (open drain); 4.7k E12 -> unused audio input held low
- R83: value 510R -> 10k; LCSC (none) -> C25744; MPN (none) -> 0402WGF1002TCE; Manufacturer (none) -> UNI-ROYAL; Note RTFADJ 510 ohm 1 %: DVI-compliant swing (SLDS145D 5.3) -> unused audio input held low; Reuse (none) -> SLIM4_R26_BOM_LINE (re-validate)
- R84: Note level shifters on -> unused audio input held low
- R85: Note load switch + HPD on -> CEC unused: clock input held low (OPEN: confirm with the HW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
- R86: value 10k -> 0R; LCSC C25744 -> C17168; MPN 0402WGF1002TCE -> 0402WGF0000TCE; Note CEC unused at the D213; internal 10k pull-up suffices -> (none)
Connections:
- net 3V3: now also C134.1, C135.1, C136.1, R88.2, R89.2, R90.2, R91.2, R92.2, U31.29 (DVDD_3V), U32.24 (VCCA), X1.1 (OE), X1.4 (VDD); no longer FB3.1, FB4.1, FB5.1, R81.2, R84.2, R85.2, R86.2
- net GND: now also R80.2, R81.2, R82.2, R83.2, R84.2, R85.2, C121.2, C122.2, C123.2, C124.2, C125.2, C126.2, C127.2, C128.2, C129.2, C130.2, C131.2, C132.2, C133.2, C134.2, C135.2, C136.2, C137.2, C138.2, J14.11 (CKS), J14.17 (DDC_GND), J14.2 (D2S), J14.5 (D1S), J14.8 (D0S), J14.SH (SHIELD), R87.2, U31.65 (EPAD_GND), U32.14 (GND), U32.19 (GND), U32.6 (GND), X1.2 (GND); no longer R75.2, R77.2
- net HDMI_5V: now also C138.1, J14.18 (+5V), TP55.1, U32.13 (5V_OUT)
- net HDMI_CEC: now also J14.13 (CEC), U32.7 (CEC_B)
- net HDMI_HPD: now also TP53.1, U31.16 (HPD), U32.4 (HPD_A)
- net HDMI_HPD_5V: now also J14.19 (HPD), U32.10 (HPD_B)
- net HDMI_SCL_5V: now also J14.15 (SCL), U32.8 (SCL_B)
- net HDMI_SDA_5V: now also J14.16 (SDA), U32.9 (SDA_B)
- net LCD_D0: now also U31.62 (D0)
- net LCD_D1: now also U31.61 (D1)
- net LCD_D10: now also U31.50 (D10)
- net LCD_D11: now also U31.49 (D11)
- net LCD_D12: now also U31.48 (D12)
- net LCD_D13: now also U31.47 (D13)
- net LCD_D14: now also U31.46 (D14)
- net LCD_D15: now also U31.45 (D15)
- net LCD_D16: now also U31.44 (D16)
- net LCD_D17: now also U31.43 (D17)
- net LCD_D18: now also U31.42 (D18)
- net LCD_D19: now also U31.41 (D19)
- net LCD_D2: now also U31.60 (D2)
- net LCD_D20: now also U31.40 (D20)
- net LCD_D21: now also U31.39 (D21)
- net LCD_D22: now also U31.38 (D22)
- net LCD_D23: now also U31.37 (D23)
- net LCD_D3: now also U31.59 (D3)
- net LCD_D4: now also U31.58 (D4)
- net LCD_D5: now also U31.57 (D5)
- net LCD_D6: now also U31.56 (D6)
- net LCD_D7: now also U31.55 (D7)
- net LCD_D8: now also U31.54 (D8)
- net LCD_D9: now also U31.52 (D9)
- net LCD_DCLK: now also R75.2, C121.1, TP52.1, U31.53 (CLK)
- net LCD_DCLK_D: now also R75.1
- net LCD_DE: now also R78.2, U31.63 (DE)
- net LCD_DE_D: now also R78.1
- net LCD_HS: now also R76.2, U31.64 (HSYNC)
- net LCD_HS_D: now also R76.1
- net LCD_VS: now also R77.2, U31.2 (VSYNC)
- net LCD_VS_D: now also R77.1
- net TMDS_CK_N: now also J14.12 (CK-), U31.17 (TXC-), U32.15 (CLK-)
- net TMDS_CK_P: now also J14.10 (CK+), U31.18 (TXC+), U32.16 (CLK+)
- net TMDS_D0_N: now also J14.9 (D0-), U31.20 (TX0-), U32.17 (D0-)
- net TMDS_D0_P: now also J14.7 (D0+), U31.21 (TX0+), U32.18 (D0+)
- net TMDS_D1_N: now also J14.6 (D1-), U31.23 (TX1-), U32.20 (D1-)
- net TMDS_D1_P: now also J14.4 (D1+), U31.24 (TX1+), U32.21 (D1+)
- net TMDS_D2_N: now also J14.3 (D2-), U31.26 (TX2-), U32.22 (D2-)
- net TMDS_D2_P: now also J14.1 (D2+), U31.27 (TX2+), U32.23 (D2+)
- net TPD_CT_HPD: now also R92.1, U32.12 (CT_HPD); no longer R85.1
- net TPD_LS_OE: now also R91.1, U32.5 (LS_OE); no longer R84.1
- net VBUS_5V: now also C137.1, U32.11 (VCC5V)
- removed net 3V3_TFP_D: FB3.2, R76.2, R78.2, R80.2, R82.2
- net 3V3_TFP_P renamed 1V8_ADV_P
- net 1V8_ADV_P: now also C131.1, C132.1, C133.1, U31.12 (PVDD), U31.13 (BGVDD)
- net 3V3_TFP_T renamed 1V8_ADV_A
- net 1V8_ADV_A: now also C127.1, C128.1, C129.1, C130.1, U31.15 (AVDD), U31.19 (AVDD), U31.25 (AVDD); no longer R83.2
- net TFP_DK1 renamed ADV_REXT
- net ADV_REXT: now also U31.14 (R_EXT); no longer R80.1
- removed net TFP_DK2: R77.1, R78.1
- removed net TFP_DK3: R75.1, R76.1
- net TFP_MSEN renamed ADV_I2S1
- net ADV_I2S1: now also U31.6 (I2S1)
- net TFP_PD_N renamed ADV_MCLK
- net ADV_MCLK: now also U31.4 (MCLK)
- net TFP_TFADJ renamed ADV_I2S2
- net ADV_I2S2: now also U31.7 (I2S2)
- net TPD_CEC_A renamed ADV_CEC_CLK_X
- net ADV_CEC_CLK_X: now also X1.3 (OUT)
- new net 1V8_ADV_D: C122.1, C123.1, C124.1, C125.1, C126.1, FB3.2, U31.1 (DVDD), U31.11 (DVDD), U31.31 (DVDD), U31.51 (DVDD)
- new net 1V8_HDMI: FB3.1, FB4.1, FB5.1
- new net ADV_CEC_CLK: R85.1, R86.2, U31.32 (CEC_CLK)
- new net ADV_I2S3: R84.1, U31.8 (I2S3)
- new net ADV_SPDIF: R80.1, U31.3 (SPDIF)
- new net HDMI_CEC_A: U31.30 (CEC), U32.1 (CEC_A)
- new net HDMI_DDC_SCL: U31.33 (DDCSCL), U32.2 (SCL_A)
- new net HDMI_DDC_SDA: U31.34 (DDCSDA), U32.3 (SDA_A)
- new net HDMI_I2C_SCL: R89.1, U31.35 (SCL)
- new net HDMI_I2C_SDA: R90.1, U31.36 (SDA)
- new net HDMI_INT: R88.1, TP54.1, U31.28 (INT)
- new net HDMI_PD: R87.1, U31.22 (PD)
- new net I2S_BCLK: TP56.1, U31.9 (SCLK)
- new net I2S_DOUT: U31.5 (I2S0)
- new net I2S_LRCK: TP57.1, U31.10 (LRCLK)
- no-connect marks 2 -> 1
Other:
- note added: "D213 RGB888 + F133 I2S -> ADV7513 HDMI transmitter (embedded audio) -> TPD12S016 -> HDMI-A Sheet generated from design.py; global labels carry every net."
- note removed: "D213 RGB888 -> TFP410 (DVI, strap mode) -> TPD12S016 -> HDMI type-A Sheet generated from design.py; global labels carry every net."
- title: ARC-1 Compact R10: D213 RGB888 -> TFP410 (DVI, strap mode) -> TPD12S016 -> HDMI type-A -> ARC-1 Compact R10: D213 RGB888 + F133 I2S -> ADV7513 HDMI transmitter (embedded audio) -> TPD12S016 -> HDMI-A
- moved on the sheet: FB3, FB4, FB5, R75, R77, R79, R81, R82, R83, R84, R85, R86

Commit message: R10 D12: top USB-A game cartridge, no eMMC; USB2514B 4-port hub (3 ports used)
Owner direction: games are played directly from a USB drive in a top USB-A "cartridge"
port; the two front USB-A ports are controller inputs; eMMC not needed.
- Schematic: eMMC sheet removed (F133 PF0-PF6 freed); USB2422 replaced by USB2514B-I/M2
  (strap mode CFG_SEL=00, port 4 disabled by strap, CRFILT/PLLFILT 0.1 uF per DS00001692C);
  third TPS2051C + ESD + TVS + vertical USB-A (Molex 105057) marked TOP.
- crosscheck I: five exterior connectors (rear USB-C + HDMI, 2x front USB-A, top USB-A),
  eMMC/USB2422 must be absent, all three ports on the hub. PASS. ERC 0/0, pin review and
  pin/function matrix PASS, R10_HOST_CHECKS_PASS.
- PCB regenerated: Ø 119.8 mm, DRC 0 errors (unrouted), top cartridge at (-9.3, 24.2) mm.
- DECISIONS D12 (supersedes D10 and the four-connector rule); change-order report sections
  1, 2, 4, 5, 6 and the mechanical note updated; CLAUDE.md topology line amended.

Co-Authored-By: Claude Opus 5.5 <noreply@anthropic.com>
Claude-Session: https://claude.ai/code/session_01UkiuLdbjDvK75uDzAPKsGs
Parts:
- removed C121: 10pF, Capacitor_SMD:C_0402_1005Metric, symbol ARC1_R10:C0402
- removed C122, C127: 10uF, Capacitor_SMD:C_0603_1608Metric, symbol ARC1_R10:C0603
- removed C123, C124, C125, C126, C128: 100nF, Capacitor_SMD:C_0402_1005Metric, symbol ARC1_R10:C0402
- removed J14: HDMI type-A, Connector_Video:HDMI_A_Molex_208658-1001_Horizontal, symbol ARC1_R10:HDMI_A
- removed R75, R76, R77, R78: 22R, Resistor_SMD:R_0402_1005Metric, symbol ARC1_R10:R0402
- removed R79: 887R, Resistor_SMD:R_0402_1005Metric, symbol ARC1_R10:R0402
- removed TP52: LCD_DCLK, TestPoint:TestPoint_Pad_D1.0mm, symbol ARC1_R10:TP
- removed U31: ADV7513BSWZ, Package_QFP:LQFP-64-1EP_10x10mm_P0.5mm_EP5x5mm_ThermalVias, symbol ARC1_R10:ADV7513
- removed U32: TPD12S016, Package_SO:TSSOP-24_4.4x7.8mm_P0.65mm, symbol ARC1_R10:TPD12S016
- added C139: 10uF, Capacitor_SMD:C_0603_1608Metric, symbol ARC1_R10:C0603
- added C140, C141, C142, C144, C145, C146: 100nF, Capacitor_SMD:C_0402_1005Metric, symbol ARC1_R10:C0402
- added C143: 1uF, Capacitor_SMD:C_0402_1005Metric, symbol ARC1_R10:C0402
- added J15: HDMI type-A, Connector_Video:HDMI_A_Molex_208658-1001_Horizontal, symbol ARC1_R10:HDMI_A
- added R93, R96, R97: 10k, Resistor_SMD:R_0402_1005Metric, symbol ARC1_R10:R0402
- added R94, R95: 2.2k, Resistor_SMD:R_0402_1005Metric, symbol ARC1_R10:R0402
- added TP58: I2S_LRCK, TestPoint:TestPoint_Pad_D1.0mm, symbol ARC1_R10:TP
- added U33: ADV7513BSWZ, Package_QFP:LQFP-64-1EP_10x10mm_P0.5mm_EP5x5mm_ThermalVias, symbol ARC1_R10:ADV7513
- added U34: TPD12S016, Package_SO:TSSOP-24_4.4x7.8mm_P0.65mm, symbol ARC1_R10:TPD12S016
- C129: value 100nF -> 10pF; LCSC C1525 -> (none); MPN CL05B104KO5NNNC -> (none); Manufacturer Samsung -> (none); Note (none) -> DNP RC filter footprint on the pixel clock; Reuse SLIM4_R26_BOM_LINE (re-validate) -> (none); now not fitted
- C130: value 100nF -> 10uF; footprint Capacitor_SMD:C_0402_1005Metric -> Capacitor_SMD:C_0603_1608Metric; symbol ARC1_R10:C0402 -> ARC1_R10:C0603; LCSC C1525 -> C19702; MPN CL05B104KO5NNNC -> CL10A106KP8NNNC
- C131: value 10uF -> 100nF; footprint Capacitor_SMD:C_0603_1608Metric -> Capacitor_SMD:C_0402_1005Metric; symbol ARC1_R10:C0603 -> ARC1_R10:C0402; LCSC C19702 -> C1525; MPN CL10A106KP8NNNC -> CL05B104KO5NNNC
- C135: value 1uF -> 10uF; footprint Capacitor_SMD:C_0402_1005Metric -> Capacitor_SMD:C_0603_1608Metric; symbol ARC1_R10:C0402 -> ARC1_R10:C0603; LCSC C52923 -> C19702; MPN CL05A105KA5NQNC -> CL10A106KP8NNNC; Note DVDD_3V -> (none)
- R80, R81, R82, R83: value 10k -> 22R; LCSC C25744 -> C25092; MPN 0402WGF1002TCE -> 0402WGF220JTCE; Note unused audio input held low -> series R at the D213 (HW guide 4.7 item 3)
- R84: value 10k -> 887R; LCSC C25744 -> (none); MPN 0402WGF1002TCE -> (none); Manufacturer UNI-ROYAL -> (none); Note unused audio input held low -> 887 ohm 1 % close to pin 14 (ADV7513 HW user guide, quoted;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; Reuse SLIM4_R26_BOM_LINE (re-validate) -> (none)
- R85: Note CEC unused: clock input held low (OPEN: confirm with the HW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 -> unused audio input held low
- R86: value 0R -> 10k; LCSC C17168 -> C25744; MPN 0402WGF0000TCE -> 0402WGF1002TCE; Note (none) -> unused audio input held low; now fitted
- R87: Note PD low at power-up: device active, I2C main map 0x72/0x39 (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 -> unused audio input held low
- R88: Note INT pull-up (OPEN: output type per HW user guide; D213 may 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 -> unused audio input held low
- R89: value 2.2k -> 10k; LCSC (none) -> C25744; MPN (none) -> 0402WGF1002TCE; Manufacturer (none) -> UNI-ROYAL; Note D213 I2C2 -> ADV7513 (5 V tolerant, 400 kHz max) -> unused audio input held low; Reuse (none) -> SLIM4_R26_BOM_LINE (re-validate)
- R90: value 2.2k -> 10k; LCSC (none) -> C25744; MPN (none) -> 0402WGF1002TCE; Manufacturer (none) -> UNI-ROYAL; Note (none) -> CEC unused: clock input held low (OPEN: confirm with the HW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; Reuse (none) -> SLIM4_R26_BOM_LINE (re-validate)
- R91: value 10k -> 0R; LCSC C25744 -> C17168; MPN 0402WGF1002TCE -> 0402WGF0000TCE; Note level shifters on -> (none); now not fitted
- R92: Note load switch + HPD on -> PD low at power-up: device active, I2C main map 0x72/0x39 (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
- TP53: value HDMI_HPD -> LCD_DCLK
- TP54: value HDMI_INT -> HDMI_HPD
- TP55: value HDMI_5V -> HDMI_INT
- TP56: value I2S_BCLK -> HDMI_5V
- TP57: value I2S_LRCK -> I2S_BCLK
Connections:
- net 1V8_ADV_A: now also C135.1, C136.1, C137.1, C138.1, U33.15 (AVDD), U33.19 (AVDD), U33.25 (AVDD); no longer C129.1, C130.1
- net 1V8_ADV_D: now also C130.1, C131.1, C132.1, C133.1, C134.1, U33.1 (DVDD), U33.11 (DVDD), U33.31 (DVDD), U33.51 (DVDD)
- net 1V8_ADV_P: now also C139.1, C140.1, C141.1, U33.12 (PVDD), U33.13 (BGVDD); no longer C131.1, C132.1, C133.1
- net 3V3: now also C142.1, C143.1, C144.1, R93.2, R94.2, R95.2, R96.2, R97.2, U33.29 (DVDD_3V), U34.24 (VCCA); no longer C134.1, C135.1, C136.1, R88.2, R89.2, R90.2, R91.2, R92.2
- net ADV_CEC_CLK: now also R90.1, R91.2, U33.32 (CEC_CLK); no longer R85.1, R86.2
- net ADV_CEC_CLK_X: now also R91.1; no longer R86.1
- net ADV_I2S1: now also R87.1, U33.6 (I2S1); no longer R82.1
- net ADV_I2S2: now also R88.1, U33.7 (I2S2); no longer R83.1
- net ADV_I2S3: now also R89.1, U33.8 (I2S3); no longer R84.1
- net ADV_MCLK: now also R86.1, U33.4 (MCLK); no longer R81.1
- net ADV_REXT: now also R84.1, U33.14 (R_EXT)
- net ADV_SPDIF: now also R85.1, U33.3 (SPDIF); no longer R80.1
- net GND: now also R86.2, R88.2, R89.2, R90.2, R92.2, C139.2, C140.2, C141.2, C142.2, C143.2, C144.2, C145.2, C146.2, J15.11 (CKS), J15.17 (DDC_GND), J15.2 (D2S), J15.5 (D1S), J15.8 (D0S), J15.SH (SHIELD), U33.65 (EPAD_GND), U34.14 (GND), U34.19 (GND), U34.6 (GND); no longer R80.2, R81.2, R82.2, R83.2
- net HDMI_5V: now also TP56.1, C146.1, J15.18 (+5V), U34.13 (5V_OUT); no longer C138.1, TP55.1
- net HDMI_CEC: now also J15.13 (CEC), U34.7 (CEC_B)
- net HDMI_CEC_A: now also U33.30 (CEC), U34.1 (CEC_A)
- net HDMI_DDC_SCL: now also U33.33 (DDCSCL), U34.2 (SCL_A)
- net HDMI_DDC_SDA: now also U33.34 (DDCSDA), U34.3 (SDA_A)
- net HDMI_HPD: now also TP54.1, U33.16 (HPD), U34.4 (HPD_A); no longer TP53.1
- net HDMI_HPD_5V: now also J15.19 (HPD), U34.10 (HPD_B)
- net HDMI_I2C_SCL: now also R94.1, U33.35 (SCL); no longer R89.1
- net HDMI_I2C_SDA: now also R95.1, U33.36 (SDA); no longer R90.1
- net HDMI_INT: now also TP55.1, R93.1, U33.28 (INT); no longer R88.1, TP54.1
- net HDMI_PD: now also R92.1, U33.22 (PD); no longer R87.1
- net HDMI_SCL_5V: now also J15.15 (SCL), U34.8 (SCL_B)
- net HDMI_SDA_5V: now also J15.16 (SDA), U34.9 (SDA_B)
- net I2S_BCLK: now also TP57.1, U33.9 (SCLK); no longer TP56.1
- net I2S_DOUT: now also U33.5 (I2S0)
- net I2S_LRCK: now also TP58.1, U33.10 (LRCLK); no longer TP57.1
- net LCD_D0: now also U33.62 (D0)
- net LCD_D1: now also U33.61 (D1)
- net LCD_D10: now also U33.50 (D10)
- net LCD_D11: now also U33.49 (D11)
- net LCD_D12: now also U33.48 (D12)
- net LCD_D13: now also U33.47 (D13)
- net LCD_D14: now also U33.46 (D14)
- net LCD_D15: now also U33.45 (D15)
- net LCD_D16: now also U33.44 (D16)
- net LCD_D17: now also U33.43 (D17)
- net LCD_D18: now also U33.42 (D18)
- net LCD_D19: now also U33.41 (D19)
- net LCD_D2: now also U33.60 (D2)
- net LCD_D20: now also U33.40 (D20)
- net LCD_D21: now also U33.39 (D21)
- net LCD_D22: now also U33.38 (D22)
- net LCD_D23: now also U33.37 (D23)
- net LCD_D3: now also U33.59 (D3)
- net LCD_D4: now also U33.58 (D4)
- net LCD_D5: now also U33.57 (D5)
- net LCD_D6: now also U33.56 (D6)
- net LCD_D7: now also U33.55 (D7)
- net LCD_D8: now also U33.54 (D8)
- net LCD_D9: now also U33.52 (D9)
- net LCD_DCLK: now also C129.1, R80.2, TP53.1, U33.53 (CLK)
- net LCD_DCLK_D: now also R80.1
- net LCD_DE: now also R83.2, U33.63 (DE)
- net LCD_DE_D: now also R83.1
- net LCD_HS: now also R81.2, U33.64 (HSYNC)
- net LCD_HS_D: now also R81.1
- net LCD_VS: now also R82.2, U33.2 (VSYNC)
- net LCD_VS_D: now also R82.1
- net TMDS_CK_N: now also J15.12 (CK-), U33.17 (TXC-), U34.15 (CLK-)
- net TMDS_CK_P: now also J15.10 (CK+), U33.18 (TXC+), U34.16 (CLK+)
- net TMDS_D0_N: now also J15.9 (D0-), U33.20 (TX0-), U34.17 (D0-)
- net TMDS_D0_P: now also J15.7 (D0+), U33.21 (TX0+), U34.18 (D0+)
- net TMDS_D1_N: now also J15.6 (D1-), U33.23 (TX1-), U34.20 (D1-)
- net TMDS_D1_P: now also J15.4 (D1+), U33.24 (TX1+), U34.21 (D1+)
- net TMDS_D2_N: now also J15.3 (D2-), U33.26 (TX2-), U34.22 (D2-)
- net TMDS_D2_P: now also J15.1 (D2+), U33.27 (TX2+), U34.23 (D2+)
- net TPD_CT_HPD: now also R97.1, U34.12 (CT_HPD); no longer R92.1
- net TPD_LS_OE: now also R96.1, U34.5 (LS_OE); no longer R91.1
- net VBUS_5V: now also C145.1, U34.11 (VCC5V); no longer C137.1
Other:
- moved on the sheet: C130, C131, C132, C133, C134, C135, C136, C137, C138, R80, R81, R82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

Commit message: R10: keep ADV7513; close INT/CEC_CLK electrical type from the ADI IBIS model
Owner asked for an HDMI audio transmitter whose documentation is fully
available. Re-checked the alternatives: Lontium LT8618SX (3-page confidential
brief only), NXP TDA19988 (EOL), ITE IT66121 (NDA register docs). The ADV7513
remains the best-documented candidate (public DS, AN-1270, Linux driver, IBIS).

- sources/adi: add adv7513.ibs record (sha 9626...). INT = OUTPUT0 Open_drain,
  no power clamp, characterised to 3.6 V; CEC_CLK = INPUT0, VIL 0.7 V.
- design.py notes updated; schematic/PCB regenerated; ERC 0 errors.
- D8 and change order: INT/CEC_CLK DERIVED; R_EXT 887 ohm and layout rules
  stay OPEN (HW user guide public but unreachable from this environment).

Co-Authored-By: Claude Opus 5.5 <noreply@anthropic.com>
Claude-Session: https://claude.ai/code/session_01UkiuLdbjDvK75uDzAPKsGs
Parts:
- R84: Note 887 ohm 1 % close to pin 14 (ADV7513 HW user guide, quoted;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 -> 887 ohm 1 % close to pin 14 (HW user guide, quoted only; DS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
- R90: Note CEC unused: clock input held low (OPEN: confirm with the HW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 -> CEC unused: clock input held low (IBIS INPUT0, VIL 0.7 V; L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
- R93: Note INT pull-up (OPEN: output type per HW user guide; D213 may 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 -> INT pull-up: INT is open drain (ADV7513 IBIS OUTPUT0, no po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
